File: hardware/ether.kicad_pcb (KiCad board)
At the start: 6 copper layers, 244 x 90 mm, 36 parts, among them J301 SS-74500-022, J401 SS-74500-022, U101 ECP5U_85_CABGA756, U102 TXB0108DQSR, U103 TCA9535RTWR, U104 TCA9535RTWR, U201 TLV62569DRL, U202 TLV62569DRL, U203 TLV62569DRL, U204 TLV62569DRL

Commit message: Save
Parts:
- added C215: 4.7u, passive:C_0603, F.Cu at (84.3, 87.8)
- added C216: 22p, passive:C_0402, F.Cu at (87.7, 70.0)
- added C217: 22u, passive:C_0603, F.Cu at (84.3, 90.0)
- added L201: 2.2u, Inductor_SMD:L_Abracon_ASPI-3012S, F.Cu at (80.2, 71.3)
- added L202: 2.2u, Inductor_SMD:L_Abracon_ASPI-3012S, F.Cu at (80.2, 76.0)
- added L203: 2.2u, Inductor_SMD:L_Abracon_ASPI-3012S, F.Cu at (80.2, 80.7)
- added L204: 2.2u, Inductor_SMD:L_Abracon_ASPI-3012S, F.Cu at (80.2, 85.3)
- added L205: 2.2u, Inductor_SMD:L_Abracon_ASPI-3012S, F.Cu at (80.2, 90.0)
- added R209: ~, passive:R_0402, F.Cu at (87.7, 71.8)
- added R210: ~, passive:R_0402, F.Cu at (87.7, 73.7)
- added U201: TPS62290, Package_SON:WSON-6-1EP_2x2mm_P0.65mm_EP1x1.6mm, F.Cu at (84.5, 70.8)
- added U202: TPS62290, Package_SON:WSON-6-1EP_2x2mm_P0.65mm_EP1x1.6mm, F.Cu at (84.5, 74.3)
- added U203: TPS62290, Package_SON:WSON-6-1EP_2x2mm_P0.65mm_EP1x1.6mm, F.Cu at (84.5, 77.9)
- added U204: TPS62290, Package_SON:WSON-6-1EP_2x2mm_P0.65mm_EP1x1.6mm, F.Cu at (84.5, 81.5)
- added U206: TPS62290, Package_SON:WSON-6-1EP_2x2mm_P0.65mm_EP1x1.6mm, F.Cu at (84.5, 85.0)
- added U301: NUF8401MNT4G, dfn:DFN-16-1EP_1.6x4mm_P0.5mm, F.Cu at (158.0, 122.0)
- added U302: NUF8401MNT4G, dfn:DFN-16-1EP_1.6x4mm_P0.5mm, F.Cu at (221.1, 109.2)
- added U303: NUF8401MNT4G, dfn:DFN-16-1EP_1.6x4mm_P0.5mm, F.Cu at (224.9, 109.2)
- added U304: NUF8401MNT4G, dfn:DFN-16-1EP_1.6x4mm_P0.5mm, F.Cu at (228.8, 109.2)
- added U305: NUF8401MNT4G, dfn:DFN-16-1EP_1.6x4mm_P0.5mm, F.Cu at (232.6, 109.2)
- added U306: NUF8401MNT4G, dfn:DFN-16-1EP_1.6x4mm_P0.5mm, F.Cu at (236.5, 109.2)
- added U307: NUF8401MNT4G, dfn:DFN-16-1EP_1.6x4mm_P0.5mm, F.Cu at (240.3, 109.2)
- added U308: NUF8401MNT4G, dfn:DFN-16-1EP_1.6x4mm_P0.5mm, F.Cu at (244.2, 109.2)
- C205, C206, C207, C208: value 10p -> 22p
- R201, R204: value 100k -> ~
- R202: value 120k -> ~
- R203: value 150k -> ~
- R205: value 261k -> ~
- R206, R208: value 82k -> ~
- R207: value 365k -> ~
Connections:
- net /Input Port/LED_G_1 renamed /Input Port/LED_Y0
- net /Input Port/LED_G_10 renamed /Input Port/LED_Y9
- net /Input Port/LED_G_11 renamed /Input Port/LED_Y10
- net /Input Port/LED_G_12 renamed /Input Port/LED_Y11
- net /Input Port/LED_G_13 renamed /Input Port/LED_Y12
- net /Input Port/LED_G_14 renamed /Input Port/LED_Y13
- net /Input Port/LED_G_15 renamed /Input Port/LED_Y14
- net /Input Port/LED_G_16 renamed /Input Port/LED_Y15
- net /Input Port/LED_G_2 renamed /Input Port/LED_Y1
- net /Input Port/LED_G_3 renamed /Input Port/LED_Y2
- net /Input Port/LED_G_4 renamed /Input Port/LED_Y3
- net /Input Port/LED_G_5 renamed /Input Port/LED_Y4
- net /Input Port/LED_G_6 renamed /Input Port/LED_Y5
- net /Input Port/LED_G_7 renamed /Input Port/LED_Y6
- net /Input Port/LED_G_8 renamed /Input Port/LED_Y7
- net /Input Port/LED_G_9 renamed /Input Port/LED_Y8
- net /Input Port/LED_Y_1 renamed /Input Port/LED_G0
- net /Input Port/LED_Y_10 renamed /Input Port/LED_G9
- net /Input Port/LED_Y_11 renamed /Input Port/LED_G10
- net /Input Port/LED_Y_12 renamed /Input Port/LED_G11
- net /Input Port/LED_Y_13 renamed /Input Port/LED_G12
- net /Input Port/LED_Y_14 renamed /Input Port/LED_G13
- net /Input Port/LED_Y_15 renamed /Input Port/LED_G14
- net /Input Port/LED_Y_16 renamed /Input Port/LED_G15
- net /Input Port/LED_Y_2 renamed /Input Port/LED_G1
- net /Input Port/LED_Y_3 renamed /Input Port/LED_G2
- net /Input Port/LED_Y_4 renamed /Input Port/LED_G3
- net /Input Port/LED_Y_5 renamed /Input Port/LED_G4
- net /Input Port/LED_Y_6 renamed /Input Port/LED_G5
- net /Input Port/LED_Y_7 renamed /Input Port/LED_G6
- net /Input Port/LED_Y_8 renamed /Input Port/LED_G7
- net /Input Port/LED_Y_9 renamed /Input Port/LED_G8
- J301 pad 11_1: unconnected-(J301-Pad11_1) -> /Input Port/LED_Y0S
- J301 pad 11_10: unconnected-(J301-Pad11_10) -> /Input Port/LED_Y9S
- J301 pad 11_11: unconnected-(J301-Pad11_11) -> /Input Port/LED_Y10S
- J301 pad 11_12: unconnected-(J301-Pad11_12) -> /Input Port/LED_Y11S
- J301 pad 11_13: unconnected-(J301-Pad11_13) -> /Input Port/LED_Y12S
- J301 pad 11_14: unconnected-(J301-Pad11_14) -> /Input Port/LED_Y13S
- J301 pad 11_15: unconnected-(J301-Pad11_15) -> /Input Port/LED_Y14S
- J301 pad 11_16: unconnected-(J301-Pad11_16) -> /Input Port/LED_Y15S
- J301 pad 11_2: unconnected-(J301-Pad11_2) -> /Input Port/LED_Y1S
- J301 pad 11_3: unconnected-(J301-Pad11_3) -> /Input Port/LED_Y2S
- J301 pad 11_4: unconnected-(J301-Pad11_4) -> /Input Port/LED_Y3S
- J301 pad 11_5: unconnected-(J301-Pad11_5) -> /Input Port/LED_Y4S
- J301 pad 11_6: unconnected-(J301-Pad11_6) -> /Input Port/LED_Y5S
- J301 pad 11_7: unconnected-(J301-Pad11_7) -> /Input Port/LED_Y6S
- J301 pad 11_8: unconnected-(J301-Pad11_8) -> /Input Port/LED_Y7S
- J301 pad 11_9: unconnected-(J301-Pad11_9) -> /Input Port/LED_Y8S
- J301 pad 1_1: unconnected-(J301-Pad1_1) -> Net-(U301-1A)
- J301 pad 1_10: unconnected-(J301-Pad1_10) -> Net-(U305-5A)
- J301 pad 1_11: unconnected-(J301-Pad1_11) -> Net-(U306-1A)
- J301 pad 1_12: unconnected-(J301-Pad1_12) -> Net-(U306-5A)
- J301 pad 1_13: unconnected-(J301-Pad1_13) -> Net-(U307-1A)
- J301 pad 1_14: unconnected-(J301-Pad1_14) -> Net-(U307-5A)
- J301 pad 1_15: unconnected-(J301-Pad1_15) -> Net-(U308-1A)
- J301 pad 1_16: unconnected-(J301-Pad1_16) -> Net-(U308-5A)
- J301 pad 1_2: unconnected-(J301-Pad1_2) -> Net-(U301-5A)
- J301 pad 1_3: unconnected-(J301-Pad1_3) -> Net-(U302-1A)
- J301 pad 1_4: unconnected-(J301-Pad1_4) -> Net-(U302-5A)
- J301 pad 1_5: unconnected-(J301-Pad1_5) -> Net-(U304-1A)
- J301 pad 1_6: unconnected-(J301-Pad1_6) -> Net-(U304-5A)
- J301 pad 1_7: unconnected-(J301-Pad1_7) -> Net-(U303-1A)
- J301 pad 1_8: unconnected-(J301-Pad1_8) -> Net-(U303-5A)
- J301 pad 1_9: unconnected-(J301-Pad1_9) -> Net-(U305-1A)
- J301 pad 2_1: unconnected-(J301-Pad2_1) -> GND
- J301 pad 2_10: unconnected-(J301-Pad2_10) -> GND
- J301 pad 2_11: unconnected-(J301-Pad2_11) -> GND
- J301 pad 2_12: unconnected-(J301-Pad2_12) -> GND
- J301 pad 2_13: unconnected-(J301-Pad2_13) -> GND
- J301 pad 2_14: unconnected-(J301-Pad2_14) -> GND
- J301 pad 2_15: unconnected-(J301-Pad2_15) -> GND
- J301 pad 2_16: unconnected-(J301-Pad2_16) -> GND
- J301 pad 2_2: unconnected-(J301-Pad2_2) -> GND
- J301 pad 2_3: unconnected-(J301-Pad2_3) -> GND
- J301 pad 2_4: unconnected-(J301-Pad2_4) -> GND
- J301 pad 2_5: unconnected-(J301-Pad2_5) -> GND
- J301 pad 2_6: unconnected-(J301-Pad2_6) -> GND
- J301 pad 2_7: unconnected-(J301-Pad2_7) -> GND
- J301 pad 2_8: unconnected-(J301-Pad2_8) -> GND
- J301 pad 2_9: unconnected-(J301-Pad2_9) -> GND
- J301 pad 3_1: unconnected-(J301-Pad3_1) -> Net-(U301-2A)
- J301 pad 3_10: unconnected-(J301-Pad3_10) -> Net-(U305-6A)
- J301 pad 3_11: unconnected-(J301-Pad3_11) -> Net-(U306-2A)
- J301 pad 3_12: unconnected-(J301-Pad3_12) -> Net-(U306-6A)
- J301 pad 3_13: unconnected-(J301-Pad3_13) -> Net-(U307-2A)
- J301 pad 3_14: unconnected-(J301-Pad3_14) -> Net-(U307-6A)
- J301 pad 3_15: unconnected-(J301-Pad3_15) -> Net-(U308-2A)
- J301 pad 3_16: unconnected-(J301-Pad3_16) -> Net-(U308-6A)
- J301 pad 3_2: unconnected-(J301-Pad3_2) -> Net-(U301-6A)
- J301 pad 3_3: unconnected-(J301-Pad3_3) -> Net-(U302-2A)
- J301 pad 3_4: unconnected-(J301-Pad3_4) -> Net-(U302-6A)
- J301 pad 3_5: unconnected-(J301-Pad3_5) -> Net-(U304-2A)
- J301 pad 3_6: unconnected-(J301-Pad3_6) -> Net-(U304-6A)
- J301 pad 3_7: unconnected-(J301-Pad3_7) -> Net-(U303-2A)
- J301 pad 3_8: unconnected-(J301-Pad3_8) -> Net-(U303-6A)
- J301 pad 3_9: unconnected-(J301-Pad3_9) -> Net-(U305-2A)
- J301 pad 4_1: unconnected-(J301-Pad4_1) -> GND
- J301 pad 4_10: unconnected-(J301-Pad4_10) -> GND
- J301 pad 4_11: unconnected-(J301-Pad4_11) -> GND
- J301 pad 4_12: unconnected-(J301-Pad4_12) -> GND
- J301 pad 4_13: unconnected-(J301-Pad4_13) -> GND
- J301 pad 4_14: unconnected-(J301-Pad4_14) -> GND
- J301 pad 4_15: unconnected-(J301-Pad4_15) -> GND
- J301 pad 4_16: unconnected-(J301-Pad4_16) -> GND
- J301 pad 4_2: unconnected-(J301-Pad4_2) -> GND
- J301 pad 4_3: unconnected-(J301-Pad4_3) -> GND
- J301 pad 4_4: unconnected-(J301-Pad4_4) -> GND
- J301 pad 4_5: unconnected-(J301-Pad4_5) -> GND
- J301 pad 4_6: unconnected-(J301-Pad4_6) -> GND
- J301 pad 4_7: unconnected-(J301-Pad4_7) -> GND
- J301 pad 4_8: unconnected-(J301-Pad4_8) -> GND
- J301 pad 4_9: unconnected-(J301-Pad4_9) -> GND
- J301 pad 5_1: unconnected-(J301-Pad5_1) -> Net-(U301-3A)
- J301 pad 5_10: unconnected-(J301-Pad5_10) -> Net-(U305-7A)
- J301 pad 5_11: unconnected-(J301-Pad5_11) -> Net-(U306-3A)
- J301 pad 5_12: unconnected-(J301-Pad5_12) -> Net-(U306-7A)
- J301 pad 5_13: unconnected-(J301-Pad5_13) -> Net-(U307-3A)
- J301 pad 5_14: unconnected-(J301-Pad5_14) -> Net-(U307-7A)
- J301 pad 5_15: unconnected-(J301-Pad5_15) -> Net-(U308-3A)
- J301 pad 5_16: unconnected-(J301-Pad5_16) -> Net-(U308-7A)
- J301 pad 5_2: unconnected-(J301-Pad5_2) -> Net-(U301-7A)
- J301 pad 5_3: unconnected-(J301-Pad5_3) -> Net-(U302-3A)
- J301 pad 5_4: unconnected-(J301-Pad5_4) -> Net-(U302-7A)
- J301 pad 5_5: unconnected-(J301-Pad5_5) -> Net-(U304-3A)
- J301 pad 5_6: unconnected-(J301-Pad5_6) -> Net-(U304-7A)
- J301 pad 5_7: unconnected-(J301-Pad5_7) -> Net-(U303-3A)
- J301 pad 5_8: unconnected-(J301-Pad5_8) -> Net-(U303-7A)
- J301 pad 5_9: unconnected-(J301-Pad5_9) -> Net-(U305-3A)
- J301 pad 6_1: unconnected-(J301-Pad6_1) -> GND
- J301 pad 6_10: unconnected-(J301-Pad6_10) -> GND
- J301 pad 6_11: unconnected-(J301-Pad6_11) -> GND
- J301 pad 6_12: unconnected-(J301-Pad6_12) -> GND
- J301 pad 6_13: unconnected-(J301-Pad6_13) -> GND
- J301 pad 6_14: unconnected-(J301-Pad6_14) -> GND
- J301 pad 6_15: unconnected-(J301-Pad6_15) -> GND
- J301 pad 6_16: unconnected-(J301-Pad6_16) -> GND
- J301 pad 6_2: unconnected-(J301-Pad6_2) -> GND
- J301 pad 6_3: unconnected-(J301-Pad6_3) -> GND
- J301 pad 6_4: unconnected-(J301-Pad6_4) -> GND
- J301 pad 6_5: unconnected-(J301-Pad6_5) -> GND
- J301 pad 6_6: unconnected-(J301-Pad6_6) -> GND
- J301 pad 6_7: unconnected-(J301-Pad6_7) -> GND
- J301 pad 6_8: unconnected-(J301-Pad6_8) -> GND
- J301 pad 6_9: unconnected-(J301-Pad6_9) -> GND
- J301 pad 7_1: unconnected-(J301-Pad7_1) -> Net-(U301-4A)
- J301 pad 7_10: unconnected-(J301-Pad7_10) -> Net-(U305-8A)
- J301 pad 7_11: unconnected-(J301-Pad7_11) -> Net-(U306-4A)
- J301 pad 7_12: unconnected-(J301-Pad7_12) -> Net-(U306-8A)
- J301 pad 7_13: unconnected-(J301-Pad7_13) -> Net-(U307-4A)
- J301 pad 7_14: unconnected-(J301-Pad7_14) -> Net-(U307-8A)
- J301 pad 7_15: unconnected-(J301-Pad7_15) -> Net-(U308-4A)
- J301 pad 7_16: unconnected-(J301-Pad7_16) -> Net-(U308-8A)
- J301 pad 7_2: unconnected-(J301-Pad7_2) -> Net-(U301-8A)
- J301 pad 7_3: unconnected-(J301-Pad7_3) -> Net-(U302-4A)
- J301 pad 7_4: unconnected-(J301-Pad7_4) -> Net-(U302-8A)
- J301 pad 7_5: unconnected-(J301-Pad7_5) -> Net-(U304-4A)
- J301 pad 7_6: unconnected-(J301-Pad7_6) -> Net-(U304-8A)
- J301 pad 7_7: unconnected-(J301-Pad7_7) -> Net-(U303-4A)
- J301 pad 7_8: unconnected-(J301-Pad7_8) -> Net-(U303-8A)
- J301 pad 7_9: unconnected-(J301-Pad7_9) -> Net-(U305-4A)
- J301 pad 8_1: unconnected-(J301-Pad8_1) -> GND
- J301 pad 8_10: unconnected-(J301-Pad8_10) -> GND
- J301 pad 8_11: unconnected-(J301-Pad8_11) -> GND
- J301 pad 8_12: unconnected-(J301-Pad8_12) -> GND
- J301 pad 8_13: unconnected-(J301-Pad8_13) -> GND
- J301 pad 8_14: unconnected-(J301-Pad8_14) -> GND
- J301 pad 8_15: unconnected-(J301-Pad8_15) -> GND
- J301 pad 8_16: unconnected-(J301-Pad8_16) -> GND
- J301 pad 8_2: unconnected-(J301-Pad8_2) -> GND
- J301 pad 8_3: unconnected-(J301-Pad8_3) -> GND
- J301 pad 8_4: unconnected-(J301-Pad8_4) -> GND
- J301 pad 8_5: unconnected-(J301-Pad8_5) -> GND
- J301 pad 8_6: unconnected-(J301-Pad8_6) -> GND
- J301 pad 8_7: unconnected-(J301-Pad8_7) -> GND
- J301 pad 8_8: unconnected-(J301-Pad8_8) -> GND
- J301 pad 8_9: unconnected-(J301-Pad8_9) -> GND
- J301 pad 9_1: unconnected-(J301-Pad9_1) -> /Input Port/LED_G0S
- J301 pad 9_10: unconnected-(J301-Pad9_10) -> /Input Port/LED_G9S
- J301 pad 9_11: unconnected-(J301-Pad9_11) -> /Input Port/LED_G10S
- J301 pad 9_12: unconnected-(J301-Pad9_12) -> /Input Port/LED_G11S
- J301 pad 9_13: unconnected-(J301-Pad9_13) -> /Input Port/LED_G12S
- J301 pad 9_14: unconnected-(J301-Pad9_14) -> /Input Port/LED_G13S
- J301 pad 9_15: unconnected-(J301-Pad9_15) -> /Input Port/LED_G14S
- J301 pad 9_16: unconnected-(J301-Pad9_16) -> /Input Port/LED_G15S
- J301 pad 9_2: unconnected-(J301-Pad9_2) -> /Input Port/LED_G1S
- J301 pad 9_3: unconnected-(J301-Pad9_3) -> /Input Port/LED_G2S
- J301 pad 9_4: unconnected-(J301-Pad9_4) -> /Input Port/LED_G3S
- J301 pad 9_5: unconnected-(J301-Pad9_5) -> /Input Port/LED_G4S
- J301 pad 9_6: unconnected-(J301-Pad9_6) -> /Input Port/LED_G5S
- J301 pad 9_7: unconnected-(J301-Pad9_7) -> /Input Port/LED_G6S
- J301 pad 9_8: unconnected-(J301-Pad9_8) -> /Input Port/LED_G7S
- J301 pad 9_9: unconnected-(J301-Pad9_9) -> /Input Port/LED_G8S
- RN301 pad 1: unconnected-(RN301-R1.1-Pad1) -> /Input Port/LED_G7S
- RN301 pad 2: unconnected-(RN301-R2.1-Pad2) -> /Input Port/LED_G6S
- RN301 pad 3: unconnected-(RN301-R3.1-Pad3) -> /Input Port/LED_G5S
- RN301 pad 4: unconnected-(RN301-R4.1-Pad4) -> /Input Port/LED_G4S
- RN301 pad 5: unconnected-(RN301-R5.1-Pad5) -> /Input Port/LED_G3S
- RN301 pad 6: unconnected-(RN301-R6.1-Pad6) -> /Input Port/LED_G2S
- RN301 pad 7: unconnected-(RN301-R7.1-Pad7) -> /Input Port/LED_G1S
- RN301 pad 8: unconnected-(RN301-R8.1-Pad8) -> /Input Port/LED_G0S
- RN302 pad 1: unconnected-(RN302-R1.1-Pad1) -> /Input Port/LED_G15S
- RN302 pad 2: unconnected-(RN302-R2.1-Pad2) -> /Input Port/LED_G14S
- RN302 pad 3: unconnected-(RN302-R3.1-Pad3) -> /Input Port/LED_G13S
- RN302 pad 4: unconnected-(RN302-R4.1-Pad4) -> /Input Port/LED_G12S
- RN302 pad 5: unconnected-(RN302-R5.1-Pad5) -> /Input Port/LED_G11S
- RN302 pad 6: unconnected-(RN302-R6.1-Pad6) -> /Input Port/LED_G10S
- RN302 pad 7: unconnected-(RN302-R7.1-Pad7) -> /Input Port/LED_G9S
- RN302 pad 8: unconnected-(RN302-R8.1-Pad8) -> /Input Port/LED_G8S
- RN303 pad 1: unconnected-(RN303-R1.1-Pad1) -> /Input Port/LED_Y7S
- RN303 pad 2: unconnected-(RN303-R2.1-Pad2) -> /Input Port/LED_Y6S
- RN303 pad 3: unconnected-(RN303-R3.1-Pad3) -> /Input Port/LED_Y5S
- RN303 pad 4: unconnected-(RN303-R4.1-Pad4) -> /Input Port/LED_Y4S
- RN303 pad 5: unconnected-(RN303-R5.1-Pad5) -> /Input Port/LED_Y3S
- RN303 pad 6: unconnected-(RN303-R6.1-Pad6) -> /Input Port/LED_Y2S
- RN303 pad 7: unconnected-(RN303-R7.1-Pad7) -> /Input Port/LED_Y1S
- RN303 pad 8: unconnected-(RN303-R8.1-Pad8) -> /Input Port/LED_Y0S
- RN304 pad 1: unconnected-(RN304-R1.1-Pad1) -> /Input Port/LED_Y15S
- RN304 pad 2: unconnected-(RN304-R2.1-Pad2) -> /Input Port/LED_Y14S
- RN304 pad 3: unconnected-(RN304-R3.1-Pad3) -> /Input Port/LED_Y13S
- RN304 pad 4: unconnected-(RN304-R4.1-Pad4) -> /Input Port/LED_Y12S
- RN304 pad 5: unconnected-(RN304-R5.1-Pad5) -> /Input Port/LED_Y11S
- RN304 pad 6: unconnected-(RN304-R6.1-Pad6) -> /Input Port/LED_Y10S
- RN304 pad 7: unconnected-(RN304-R7.1-Pad7) -> /Input Port/LED_Y9S
- RN304 pad 8: unconnected-(RN304-R8.1-Pad8) -> /Input Port/LED_Y8S
- U101 pad AG1: unconnected-(U101I-PB4A/+/D7/IO7-PadAG1) -> /PORT77_1
- U101 pad AH1: unconnected-(U101I-PB4B/-/D6/IO6-PadAH1) -> /PORT77_2
- U101 pad AJ1: unconnected-(U101I-PB6A/+/D5/MISO2/IO5-PadAJ1) -> /PORT77_3
- U101 pad AJ2: unconnected-(U101I-PB11A/+/D1/MISO/IO1-PadAJ2) -> /PORT78_3
- U101 pad AK1: unconnected-(U101I-PB6B/-/D4/MOSI2/IO4-PadAK1) -> /PORT77_4
- U101 pad AK2: unconnected-(U101I-PB11B/-/D0/MOSI/IO0-PadAK2) -> /PORT78_4
- U101 pad AL1: unconnected-(U101I-PB9A/+/D3/IO3-PadAL1) -> /PORT78_1
- U101 pad AM2: unconnected-(U101I-PB9B/-/D2/IO2-PadAM2) -> /PORT78_2
Routing:
- net /PORT6: vias 1 -> 0
