File: hardware/ether.kicad_pcb (KiCad board)
At the start: 6 copper layers, 2.5 x 116.6 mm, 3 parts, among them J101 SS-74500-022, J102 SS-74500-022, U101 ECP5UM_85_CABGA756

Commit message: Save
Parts:
- removed J101, J102: SS-74500-022, connectors:BEL_SS-74500-022
- added C201: 4.7u, passive:C_0603, F.Cu at (163.1, 216.8)
- added C202: 4.7u, passive:C_0603, F.Cu at (163.1, 218.9)
- added C203: 4.7u, passive:C_0603, F.Cu at (163.1, 221.1)
- added C204: 4.7u, passive:C_0603, F.Cu at (163.1, 223.2)
- added C205: 10p, passive:C_0402, F.Cu at (162.7, 227.4)
- added C206: 10p, passive:C_0402, F.Cu at (162.7, 229.2)
- added C207: 10p, passive:C_0402, F.Cu at (162.7, 231.1)
- added C208: 10p, passive:C_0402, F.Cu at (162.7, 232.9)
- added C209: 22u, passive:C_0603, F.Cu at (163.1, 225.4)
- added C210: 22u, passive:C_0603, F.Cu at (166.4, 216.8)
- added C211: 22u, passive:C_0603, F.Cu at (166.4, 218.9)
- added C212: 22u, passive:C_0603, F.Cu at (166.4, 221.1)
- added C213: 22u, passive:C_0603, F.Cu at (166.4, 223.2)
- added C214: 22u, passive:C_0603, F.Cu at (166.4, 225.4)
- added J301: SS-74500-022, connectors:BEL_SS-74500-022, F.Cu at (212.5, 150.0)
- added J401: SS-74500-022, connectors:BEL_SS-74500-022, F.Cu at (87.0, 150.0)
- added R201: 100k, passive:R_0402, F.Cu at (165.4, 227.4)
- added R202: 120k, passive:R_0402, F.Cu at (165.4, 229.2)
- added R203: 150k, passive:R_0402, F.Cu at (165.4, 231.1)
- added R204: 100k, passive:R_0402, F.Cu at (165.4, 232.9)
- added R205: 261k, passive:R_0402, F.Cu at (168.0, 227.4)
- added R206: 82k, passive:R_0402, F.Cu at (168.0, 229.2)
- added R207: 365k, passive:R_0402, F.Cu at (168.0, 231.1)
- added R208: 82k, passive:R_0402, F.Cu at (168.0, 232.9)
- added RN301: 1k, Resistor_SMD:R_Array_Convex_8x0602, F.Cu at (112.5, 163.0)
- added RN302: 1k, Resistor_SMD:R_Array_Convex_8x0602, F.Cu at (116.6, 163.0)
- added RN303: 1k, Resistor_SMD:R_Array_Convex_8x0602, F.Cu at (120.8, 163.0)
- added RN304: 1k, Resistor_SMD:R_Array_Convex_8x0602, F.Cu at (124.9, 163.0)
- added U102: TXB0108DQSR, Package_SON:USON-20_2x4mm_P0.4mm, F.Cu at (118.9, 170.6)
- added U103: TCA9535RTWR, Package_DFN_QFN:WQFN-24-1EP_4x4mm_P0.5mm_EP2.45x2.45mm, F.Cu at (113.6, 171.0)
- added U104: TCA9535RTWR, Package_DFN_QFN:WQFN-24-1EP_4x4mm_P0.5mm_EP2.45x2.45mm, F.Cu at (113.6, 177.2)
- added U201: TLV62569DRL, Package_TO_SOT_SMD:SOT-563, F.Cu at (159.5, 217.3)
- added U202: TLV62569DRL, Package_TO_SOT_SMD:SOT-563, F.Cu at (159.5, 220.6)
- added U203: TLV62569DRL, Package_TO_SOT_SMD:SOT-563, F.Cu at (159.5, 223.8)
- added U204: TLV62569DRL, Package_TO_SOT_SMD:SOT-563, F.Cu at (159.5, 227.1)
- U101: value ECP5UM_85_CABGA756 -> ECP5U_85_CABGA756
Connections:
- net Net-(U101A-VCCAUX[8]-PadAC11) renamed +2V5
- net Net-(U101A-VCC[36]-PadAA12) renamed +1V1
- U101 pad A10: unconnected-(U101B-PT31B/--PadA10) -> /PORT1
- U101 pad A11: unconnected-(U101B-PT38B/--PadA11) -> /PORT1
- U101 pad A13: unconnected-(U101B-PT42B/--PadA13) -> /PORT1
- U101 pad A14: unconnected-(U101B-PT49B/--PadA14) -> /PORT1
- U101 pad A15: unconnected-(U101B-PT54B/--PadA15) -> /PORT1
- U101 pad A16: unconnected-(U101B-PT60B/-/GR_PCLK0_0-PadA16) -> /PORT1
- U101 pad A17: unconnected-(U101B-PT63A/+/PCLKT0_1-PadA17) -> /PORT1
- U101 pad A18: unconnected-(U101C-PT71A/+/PCLKT1_0-PadA18) -> /PORT2
- U101 pad A19: unconnected-(U101C-PT76A/+-PadA19) -> /PORT2
- U101 pad A2: unconnected-(U101B-PT6A/+-PadA2) -> /PORT1
- U101 pad A20: unconnected-(U101C-PT83A/+-PadA20) -> /PORT2
- U101 pad A22: unconnected-(U101C-PT87A/+-PadA22) -> /PORT2
- U101 pad A23: unconnected-(U101C-PT94A/+-PadA23) -> /PORT2
- U101 pad A24: unconnected-(U101C-PT101A/+-PadA24) -> /PORT2
- U101 pad A25: unconnected-(U101C-PT105A/+-PadA25) -> /PORT2
- U101 pad A26: unconnected-(U101C-PT112A/+-PadA26) -> /PORT2
- U101 pad A28: unconnected-(U101C-PT116A/+-PadA28) -> /PORT2
- U101 pad A29: unconnected-(U101C-PT116B/--PadA29) -> /PORT2
- U101 pad A3: unconnected-(U101B-PT6B/--PadA3) -> /PORT1
- U101 pad A30: unconnected-(U101C-PT119A/+-PadA30) -> /PORT2
- U101 pad A31: unconnected-(U101C-PT119B/--PadA31) -> /PORT2
- U101 pad A4: unconnected-(U101B-PT9A/+-PadA4) -> /PORT1
- U101 pad A5: unconnected-(U101B-PT9B/--PadA5) -> /PORT1
- U101 pad A7: unconnected-(U101B-PT13B/--PadA7) -> /PORT1
- U101 pad A8: unconnected-(U101B-PT20B/--PadA8) -> /PORT1
- U101 pad A9: unconnected-(U101B-PT24B/--PadA9) -> /PORT1
- U101 pad AB1: unconnected-(U101G-PL92A/+/HS/LDQ89-PadAB1) -> /PORT6
- U101 pad AB2: unconnected-(U101G-PL89B/-/HS/LDQSN89-PadAB2) -> /PORT6
- U101 pad AB26: unconnected-(U101E-PR74C/+/RDQ77-PadAB26) -> /PORT4
- U101 pad AB27: unconnected-(U101E-PR77B/-/HS/RDQSN77-PadAB27) -> /PORT4
- U101 pad AB28: unconnected-(U101E-PR77A/+/HS/RDQS77-PadAB28) -> /PORT4
- U101 pad AB29: unconnected-(U101E-PR83B/-/HS/RDQ89-PadAB29) -> /PORT4
- U101 pad AB3: unconnected-(U101G-PL83A/+/HS/LDQ89-PadAB3) -> /PORT6
- U101 pad AB30: unconnected-(U101E-PR83A/+/HS/RDQ89-PadAB30) -> /PORT4
- U101 pad AB31: unconnected-(U101E-PR89B/-/HS/RDQSN89-PadAB31) -> /PORT4
- U101 pad AB32: unconnected-(U101E-PR92A/+/HS/RDQ89-PadAB32) -> /PORT4
- U101 pad AB4: unconnected-(U101G-PL83B/-/HS/LDQ89-PadAB4) -> /PORT6
- U101 pad AB5: unconnected-(U101G-PL77A/+/HS/LDQS77-PadAB5) -> /PORT6
- U101 pad AB6: unconnected-(U101G-PL77B/-/HS/LDQSN77-PadAB6) -> /PORT6
- U101 pad AB7: unconnected-(U101G-PL74C/+/LDQ77-PadAB7) -> /PORT6
- U101 pad AC1: unconnected-(U101G-PL92B/-/HS/LDQ89-PadAC1) -> /PORT6
- U101 pad AC13: unconnected-(U101A-VCCHTX0_D0CH0-PadAC13) -> GND
- U101 pad AC14: unconnected-(U101A-VCCHRX0_D0CH0-PadAC14) -> GND
- U101 pad AC15: unconnected-(U101A-VCCHRX1_D0CH1-PadAC15) -> GND
- U101 pad AC16: unconnected-(U101A-VCCHTX1_D0CH1-PadAC16) -> GND
- U101 pad AC17: unconnected-(U101A-VCCHTX0_D1CH0-PadAC17) -> GND
- U101 pad AC18: unconnected-(U101A-VCCHRX0_D1CH0-PadAC18) -> GND
- U101 pad AC19: unconnected-(U101A-VCCHRX1_D1CH1-PadAC19) -> GND
- U101 pad AC2: unconnected-(U101G-PL89C/+/LDQ89-PadAC2) -> /PORT6
- U101 pad AC20: unconnected-(U101A-VCCHTX1_D1CH1-PadAC20) -> GND
- U101 pad AC26: unconnected-(U101E-PR77C/+/RDQ77-PadAC26) -> /PORT4
- U101 pad AC27: unconnected-(U101E-PR74D/-/RDQ77-PadAC27) -> /PORT4
- U101 pad AC28: unconnected-(U101E-PR83C/+/RDQ89-PadAC28) -> /PORT4
- U101 pad AC3: unconnected-(U101G-PL89A/+/HS/LDQS89-PadAC3) -> /PORT6
- U101 pad AC30: unconnected-(U101E-PR89A/+/HS/RDQS89-PadAC30) -> /PORT4
- U101 pad AC31: unconnected-(U101E-PR89C/+/RDQ89-PadAC31) -> /PORT4
- U101 pad AC32: unconnected-(U101E-PR92B/-/HS/RDQ89-PadAC32) -> /PORT4
- U101 pad AC5: unconnected-(U101G-PL83C/+/LDQ89-PadAC5) -> /PORT6
- U101 pad AC6: unconnected-(U101G-PL74D/-/LDQ77-PadAC6) -> /PORT6
- U101 pad AC7: unconnected-(U101G-PL77C/+/LDQ77-PadAC7) -> /PORT6
- U101 pad AD1: unconnected-(U101G-PL92C/+/LLC_GPLL0T_IN/LDQ89-PadAD1) -> /PORT6
- U101 pad AD26: unconnected-(U101E-PR77D/-/RDQ77-PadAD26) -> /PORT4
- U101 pad AD27: unconnected-(U101E-PR80A/+/HS/RDQ77-PadAD27) -> /PORT4
- U101 pad AD29: unconnected-(U101E-PR83D/-/RDQ89-PadAD29) -> /PORT4
- U101 pad AD3: unconnected-(U101G-PL86C/+/LDQ89-PadAD3) -> /PORT6
- U101 pad AD30: unconnected-(U101E-PR86C/+/RDQ89-PadAD30) -> /PORT4
- U101 pad AD32: unconnected-(U101E-PR92C/+/LRC_GPLL0T_IN/RDQ89-PadAD32) -> /PORT4
- U101 pad AD4: unconnected-(U101G-PL83D/-/LDQ89-PadAD4) -> /PORT6
- U101 pad AD6: unconnected-(U101G-PL80A/+/HS/LDQ77-PadAD6) -> /PORT6
- U101 pad AD7: unconnected-(U101G-PL77D/-/LDQ77-PadAD7) -> /PORT6
- U101 pad AE1: unconnected-(U101G-PL92D/-/LLC_GPLL0C_IN/LDQ89-PadAE1) -> /PORT6
- U101 pad AE2: unconnected-(U101G-PL89D/-/LDQ89-PadAE2) -> /PORT6
- U101 pad AE27: unconnected-(U101E-PR80B/-/HS/RDQ77-PadAE27) -> /PORT4
- U101 pad AE28: unconnected-(U101E-PR80C/+/RDQ77-PadAE28) -> /PORT4
- U101 pad AE29: unconnected-(U101E-PR80D/-/RDQ77-PadAE29) -> /PORT4
- U101 pad AE3: unconnected-(U101G-PL86D/-/LDQ89-PadAE3) -> /PORT6
- U101 pad AE30: unconnected-(U101E-PR86D/-/RDQ89-PadAE30) -> /PORT4
- U101 pad AE31: unconnected-(U101E-PR89D/-/RDQ89-PadAE31) -> /PORT4
- U101 pad AE32: unconnected-(U101E-PR92D/-/LRC_GPLL0C_IN/RDQ89-PadAE32) -> /PORT4
- U101 pad AE4: unconnected-(U101G-PL80D/-/LDQ77-PadAE4) -> /PORT6
- U101 pad AE5: unconnected-(U101G-PL80C/+/LDQ77-PadAE5) -> /PORT6
- U101 pad AE6: unconnected-(U101G-PL80B/-/HS/LDQ77-PadAE6) -> /PORT6
- U101 pad AF22: Net-(U101A-VCCA1[9]-PadAF22) -> GND
- U101 pad AG12: Net-(U101A-VCCA0[8]-PadAG12) -> GND
- U101 pad AG19: Net-(U101A-VCCA1[9]-PadAF22) -> GND
- U101 pad AG22: Net-(U101A-VCCA1[9]-PadAF22) -> GND
- U101 pad AG28: unconnected-(U101F-PB110A/+-PadAG28) -> /PORT5
- U101 pad AG29: unconnected-(U101F-PB110B/--PadAG29) -> /PORT5
- U101 pad AG30: unconnected-(U101F-PB114B/--PadAG30) -> /PORT5
- U101 pad AG32: unconnected-(U101F-PB119B/--PadAG32) -> /PORT5
- U101 pad AG9: Net-(U101A-VCCA0[8]-PadAG12) -> GND
- U101 pad AH12: Net-(U101A-VCCA0[8]-PadAG12) -> GND
- U101 pad AH19: Net-(U101A-VCCA1[9]-PadAF22) -> GND
- U101 pad AH22: Net-(U101A-VCCA1[9]-PadAF22) -> GND
- U101 pad AH28: unconnected-(U101F-PB112B/--PadAH28) -> /PORT5
- U101 pad AH30: unconnected-(U101F-PB114A/+-PadAH30) -> /PORT5
- U101 pad AH32: unconnected-(U101F-PB119A/+-PadAH32) -> /PORT5
- U101 pad AH9: Net-(U101A-VCCA0[8]-PadAG12) -> GND
- U101 pad AJ10: Net-(U101A-VCCA0[8]-PadAG12) -> GND
- U101 pad AJ12: Net-(U101A-VCCA0[8]-PadAG12) -> GND
- U101 pad AJ13: Net-(U101A-VCCA0[8]-PadAG12) -> GND
- U101 pad AJ15: Net-(U101A-VCCAUXA0[2]-PadAJ15) -> GND
- U101 pad AJ16: Net-(U101A-VCCAUXA0[2]-PadAJ15) -> GND
- U101 pad AJ18: Net-(U101A-VCCA1[9]-PadAF22) -> GND
- U101 pad AJ19: Net-(U101A-VCCA1[9]-PadAF22) -> GND
- U101 pad AJ21: Net-(U101A-VCCA1[9]-PadAF22) -> GND
- U101 pad AJ22: Net-(U101A-VCCA1[9]-PadAF22) -> GND
- U101 pad AJ24: Net-(U101A-VCCAUXA1[2]-PadAJ24) -> GND
- U101 pad AJ25: Net-(U101A-VCCAUXA1[2]-PadAJ24) -> GND
- U101 pad AJ28: unconnected-(U101F-PB112A/+-PadAJ28) -> /PORT5
- U101 pad AJ29: unconnected-(U101F-PB121A/+-PadAJ29) -> /PORT5
- U101 pad AJ30: unconnected-(U101F-PB121B/--PadAJ30) -> /PORT5
- U101 pad AJ31: unconnected-(U101F-PB105B/--PadAJ31) -> /PORT5
- U101 pad AJ32: unconnected-(U101F-PB101B/--PadAJ32) -> /PORT5
- U101 pad AJ9: Net-(U101A-VCCA0[8]-PadAG12) -> GND
- U101 pad AK28: unconnected-(U101F-PB98B/--PadAK28) -> /PORT5
- U101 pad AK29: unconnected-(U101F-PB116A/+-PadAK29) -> /PORT5
- U101 pad AK30: unconnected-(U101F-PB116B/--PadAK30) -> /PORT5
- U101 pad AK31: unconnected-(U101F-PB105A/+-PadAK31) -> /PORT5
- U101 pad AK32: unconnected-(U101F-PB101A/+-PadAK32) -> /PORT5
- U101 pad AL28: unconnected-(U101F-PB98A/+-PadAL28) -> /PORT5
- U101 pad AL30: unconnected-(U101F-PB103B/--PadAL30) -> /PORT5
- U101 pad AL32: unconnected-(U101F-PB107B/--PadAL32) -> /PORT5
- U101 pad AM11: unconnected-(U101K-HDRXP0_D0CH1/+-PadAM11) -> GND
- U101 pad AM12: unconnected-(U101K-HDRXN0_D0CH1/--PadAM12) -> GND
- U101 pad AM14: unconnected-(U101K-REFCLKP_D0/+-PadAM14) -> GND
- U101 pad AM15: unconnected-(U101K-REFCLKN_D0/--PadAM15) -> GND
- U101 pad AM17: unconnected-(U101L-HDRXP0_D1CH0/+-PadAM17) -> GND
- U101 pad AM18: unconnected-(U101L-HDRXN0_D1CH0/--PadAM18) -> GND
- U101 pad AM20: unconnected-(U101L-HDRXP0_D1CH1/+-PadAM20) -> GND
- U101 pad AM21: unconnected-(U101L-HDRXN0_D1CH1/--PadAM21) -> GND
- U101 pad AM23: unconnected-(U101L-REFCLKP_D1/+-PadAM23) -> GND
- U101 pad AM24: unconnected-(U101L-REFCLKN_D1/--PadAM24) -> GND
- U101 pad AM28: unconnected-(U101F-PB96A/+-PadAM28) -> /PORT5
- U101 pad AM29: unconnected-(U101F-PB96B/--PadAM29) -> /PORT5
- U101 pad AM30: unconnected-(U101F-PB103A/+-PadAM30) -> /PORT5
- U101 pad AM31: unconnected-(U101F-PB107A/+-PadAM31) -> /PORT5
- U101 pad AM8: unconnected-(U101K-HDRXP0_D0CH0/+-PadAM8) -> GND
- U101 pad AM9: unconnected-(U101K-HDRXN0_D0CH0/--PadAM9) -> GND
- U101 pad B1: unconnected-(U101H-PL17A/+/HS/LDQS17-PadB1) -> /PORT7
- U101 pad B10: unconnected-(U101B-PT31A/+-PadB10) -> /PORT1
- U101 pad B11: unconnected-(U101B-PT38A/+-PadB11) -> /PORT1
- U101 pad B14: unconnected-(U101B-PT49A/+-PadB14) -> /PORT1
- U101 pad B16: unconnected-(U101B-PT60A/+/GR_PCLK0_1-PadB16) -> /PORT1
- U101 pad B17: unconnected-(U101B-PT63B/-/PCLKC0_1-PadB17) -> /PORT1
- U101 pad B19: unconnected-(U101C-PT76B/--PadB19) -> /PORT2
- U101 pad B22: unconnected-(U101C-PT87B/--PadB22) -> /PORT2
- U101 pad B23: unconnected-(U101C-PT94B/--PadB23) -> /PORT2
- U101 pad B25: unconnected-(U101C-PT105B/--PadB25) -> /PORT2
- U101 pad B26: unconnected-(U101C-PT112B/--PadB26) -> /PORT2
- U101 pad B29: unconnected-(U101C-PT121A/+/URC_GPLL1T_IN-PadB29) -> /PORT2
- U101 pad B3: unconnected-(U101B-PT4A/+/ULC_GPLL1T_IN-PadB3) -> /PORT1
- U101 pad B30: unconnected-(U101C-PT121B/-/URC_GPLL1C_IN-PadB30) -> /PORT2
- U101 pad B32: unconnected-(U101D-PR17A/+/HS/RDQS17-PadB32) -> /PORT3
- U101 pad B4: unconnected-(U101B-PT4B/-/ULC_GPLL1C_IN-PadB4) -> /PORT1
- U101 pad B7: unconnected-(U101B-PT13A/+-PadB7) -> /PORT1
- U101 pad B8: unconnected-(U101B-PT20A/+-PadB8) -> /PORT1
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Routing:
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Other:
- board size 2.5 x 116.6 mm -> 244 x 90 mm

Commit message: Save
Parts:
- removed C213, C214: 22u, passive:C_0603
- removed J401: SS-74500-022, connectors:BEL_SS-74500-022
- added C101: 0.1u, passive:C_0201, F.Cu at (201.3, 78.6)
- added C102: 0.1u, passive:C_0201, F.Cu at (168.7, 71.1)
- added C103: 0.1u, passive:C_0201, F.Cu at (171.4, 79.4)
- added C104: 0.1u, passive:C_0201, F.Cu at (175.0, 79.4)
- added C105: 0.1u, passive:C_0201, F.Cu at (179.3, 76.8)
- added C106: 10p, passive:C_0402, F.Cu at (178.6, 67.6)
- added C107: 10p, passive:C_0402, F.Cu at (177.2, 66.0)
- added C108: 0.1u, passive:C_0201, F.Cu at (173.1, 68.7)
- added C109: 0.1u, passive:C_0201, F.Cu at (172.6, 68.7)
- added C110: 0.1u, passive:C_0201, F.Cu at (168.7, 75.1)
- added C111: 0.1u, passive:C_0201, F.Cu at (174.2, 79.4)
- added C112: 4.7u, passive:C_0603, F.Cu at (179.3, 78.4)
- added C113: 0.1u, passive:C_0201, F.Cu at (174.1, 68.7)
- added C114: 0.1u, passive:C_0201, F.Cu at (175.0, 68.7)
- added C115: 0.1u, passive:C_0201, F.Cu at (177.4, 69.3)
- added C116: 0.1u, passive:C_0201, F.Cu at (168.7, 74.6)
- added C117: 0.1u, passive:C_0201, F.Cu at (168.7, 71.8)
- added C118: 0.1u, passive:C_0201, F.Cu at (173.6, 68.7)
- added C119: 0.1u, passive:C_0201, F.Cu at (172.1, 68.7)
- added C120: 0.1u, passive:C_0201, F.Cu at (168.7, 70.4)
- added C121: 0.1u, passive:C_0201, F.Cu at (179.3, 71.7)
- added C215: 4.7u, passive:C_0603, F.Cu at (151.3, 233.8)
- added C216: 22p, passive:C_0402, F.Cu at (154.7, 215.9)
- added C217: 22u, passive:C_0603, F.Cu at (151.3, 236.0)
- added FB101: FerriteBead_Small, passive:R_0603, F.Cu at (205.2, 78.5)
- added J101: USB3_B_Micro, usb:AMPHENOL-GSB343K33HR, F.Cu at (204.5, 64.3)
- added L201: 2.2u, Inductor_SMD:L_Abracon_ASPI-3012S, F.Cu at (147.2, 217.3)
- added L202: 2.2u, Inductor_SMD:L_Abracon_ASPI-3012S, F.Cu at (147.2, 222.0)
- added L203: 2.2u, Inductor_SMD:L_Abracon_ASPI-3012S, F.Cu at (147.2, 226.7)
- added L204: 2.2u, Inductor_SMD:L_Abracon_ASPI-3012S, F.Cu at (147.2, 231.3)
- added L205: 2.2u, Inductor_SMD:L_Abracon_ASPI-3012S, F.Cu at (147.2, 235.9)
- added R101: 1.6k, passive:R_0201, F.Cu at (173.9, 67.5)
- added R102: 10k, passive:R_0201, F.Cu at (179.3, 71.2)
- added R103: 10k, passive:R_0201, F.Cu at (179.3, 72.2)
- added R104: 10k, passive:R_0201, F.Cu at (179.3, 74.3)
- added R105: 33, passive:R_0201, F.Cu at (179.3, 76.3)
- added R106: 33, passive:R_0201, F.Cu at (179.3, 75.8)
- added R107: 33, passive:R_0201, F.Cu at (179.3, 75.3)
- added R108: 33, passive:R_0201, F.Cu at (179.3, 74.8)
- added R109: 33, passive:R_0201, F.Cu at (179.3, 73.8)
- added R110: 33, passive:R_0201, F.Cu at (179.3, 73.3)
- added R111: 33, passive:R_0201, F.Cu at (179.3, 72.8)
- added R112: 33, passive:R_0201, F.Cu at (170.9, 79.4)
- added R113: 33, passive:R_0201, F.Cu at (168.7, 72.6)
- added R114: 33, passive:R_0201, F.Cu at (168.7, 73.1)
- added R115: 33, passive:R_0201, F.Cu at (168.7, 73.6)
- added R116: 33, passive:R_0201, F.Cu at (168.7, 74.1)
- added R117: 33, passive:R_0201, F.Cu at (168.7, 75.6)
- added R118: 33, passive:R_0201, F.Cu at (168.7, 76.1)
- added R119: 33, passive:R_0201, F.Cu at (168.7, 76.6)
- added R120: 33, passive:R_0201, F.Cu at (168.7, 77.1)
- added R121: 33, passive:R_0201, F.Cu at (171.9, 79.4)
- added R122: 33, passive:R_0201, F.Cu at (172.4, 79.4)
- added R123: 33, passive:R_0201, F.Cu at (172.9, 79.4)
- added R124: 33, passive:R_0201, F.Cu at (173.4, 79.4)
- added R125: 33, passive:R_0201, F.Cu at (175.5, 79.4)
- added R126: 33, passive:R_0201, F.Cu at (176.0, 79.4)
- added R127: 33, passive:R_0201, F.Cu at (176.5, 79.4)
- added R128: 33, passive:R_0201, F.Cu at (177.0, 79.4)
- added R209: ~, passive:R_0201, F.Cu at (154.7, 217.8)
- added R210: ~, passive:R_0201, F.Cu at (154.7, 219.7)
- added U105: PUSB3FR4Z, dfn:DFN-10-1.0x2.5mm_P0.5mm, F.Cu at (197.9, 69.8)
- added U106: FT600Q, qfn:QFN-56-1EP_7x7mm_P0.4mm_EP5.7x5.7mm_FT600, F.Cu at (174.0, 74.0)
- added U206: TPS62290, Package_SON:WSON-6-1EP_2x2mm_P0.65mm_EP1x1.6mm, F.Cu at (151.5, 231.0)
- added Y101: 30 MHz, crystals:Crystal_4Pin_2.0x1.6mm, F.Cu at (177.2, 67.6)
- C205, C206, C207, C208: value 10p -> 22p
- R201, R204: value 100k -> ~; footprint passive:R_0402 -> passive:R_0201
- R202: value 120k -> ~; footprint passive:R_0402 -> passive:R_0201
- R203: value 150k -> ~; footprint passive:R_0402 -> passive:R_0201
- R205: value 261k -> ~; footprint passive:R_0402 -> passive:R_0201
- R206, R208: value 82k -> ~; footprint passive:R_0402 -> passive:R_0201
- R207: value 365k -> ~; footprint passive:R_0402 -> passive:R_0201
- U201, U202, U203, U204: value TLV62569DRL -> TPS62290; footprint Package_TO_SOT_SMD:SOT-563 -> Package_SON:WSON-6-1EP_2x2mm_P0.65mm_EP1x1.6mm
- moved U201 8.01 mm to (151.5, 216.8)
- moved U204 8.00 mm to (151.5, 227.4)
- moved U202 8.00 mm to (151.5, 220.3)
- moved U203 8.00 mm to (151.5, 223.9)
Connections:
- U101 pad A18: /PORT2 -> /PORT3
- U101 pad A19: /PORT2 -> /PORT3
- U101 pad A20: /PORT2 -> /PORT3
- U101 pad A22: /PORT2 -> /PORT3
- U101 pad A23: /PORT2 -> /PORT3
- U101 pad A24: /PORT2 -> /PORT3
- U101 pad A25: /PORT2 -> /PORT3
- U101 pad A26: /PORT2 -> /PORT3
- U101 pad A28: /PORT2 -> /PORT3
- U101 pad A29: /PORT2 -> /PORT3
- U101 pad A30: /PORT2 -> /PORT3
- U101 pad A31: /PORT2 -> /PORT3
- U101 pad B19: /PORT2 -> /PORT3
- U101 pad B22: /PORT2 -> /PORT3
- U101 pad B23: /PORT2 -> /PORT3
- U101 pad B25: /PORT2 -> /PORT3
- U101 pad B26: /PORT2 -> /PORT3
- U101 pad B29: /PORT2 -> /PORT3
- U101 pad B30: /PORT2 -> /PORT3
- U101 pad B32: /PORT3 -> unconnected-(U101D-PR17A/+/HS/RDQS17-PadB32)
- U101 pad C18: /PORT2 -> /PORT3
- U101 pad C19: /PORT2 -> /PORT3
- U101 pad C20: /PORT2 -> /PORT3
- U101 pad C22: /PORT2 -> /PORT3
- U101 pad C23: /PORT2 -> /PORT3
- U101 pad C24: /PORT2 -> /PORT3
- U101 pad C25: /PORT2 -> /PORT3
- U101 pad C26: /PORT2 -> /PORT3
- U101 pad C28: /PORT3 -> /FT_CLKOUT
- U101 pad C29: /PORT3 -> unconnected-(U101D-PR11C/+/RDQ17-PadC29)
- U101 pad C30: /PORT3 -> unconnected-(U101D-PR11D/-/RDQ17-PadC30)
- U101 pad C31: /PORT3 -> unconnected-(U101D-PR17B/-/HS/RDQSN17-PadC31)
- U101 pad C32: /PORT3 -> /~{FT_RESET}
- U101 pad D18: /PORT2 -> /PORT3
- U101 pad D19: /PORT2 -> /PORT3
- U101 pad D20: /PORT2 -> /PORT3
- U101 pad D22: /PORT2 -> /PORT3
- U101 pad D23: /PORT2 -> /PORT3
- U101 pad D24: /PORT2 -> /PORT3
- U101 pad D25: /PORT2 -> /PORT3
- U101 pad D26: /PORT2 -> /PORT3
- U101 pad D28: /PORT3 -> +3V3
- U101 pad D29: /PORT3 -> unconnected-(U101D-PR14A/+/HS/RDQ17-PadD29)
- U101 pad D30: /PORT3 -> unconnected-(U101D-PR17C/+/RDQ17-PadD30)
- U101 pad D31: /PORT3 -> /FT_GPIO0
- U101 pad D32: /PORT3 -> /FT_WAKEUP
- U101 pad E17: /PORT2 -> /PORT3
- U101 pad E19: /PORT2 -> /PORT3
- U101 pad E22: /PORT2 -> /PORT3
- U101 pad E23: /PORT2 -> /PORT3
- U101 pad E25: /PORT2 -> /PORT3
- U101 pad E29: /PORT3 -> unconnected-(U101D-PR14B/-/HS/RDQ17-PadE29)
- U101 pad E30: /PORT3 -> /~{FT_SIWU}
- U101 pad E32: /PORT3 -> /FT_BE0
- U101 pad F17: /PORT2 -> /PORT3
- U101 pad F18: /PORT2 -> /PORT3
- U101 pad F19: /PORT2 -> /PORT3
- U101 pad F20: /PORT2 -> /PORT3
- U101 pad F22: /PORT2 -> /PORT3
- U101 pad F23: /PORT2 -> /PORT3
- U101 pad F24: /PORT2 -> /PORT3
- U101 pad F25: /PORT2 -> /PORT3
- U101 pad F28: /PORT3 -> unconnected-(U101D-PR14D/-/RDQ17-PadF28)
- U101 pad F29: /PORT3 -> unconnected-(U101D-PR14C/+/RDQ17-PadF29)
- U101 pad F30: /PORT3 -> /FT_GPIO1
- U101 pad F31: /PORT3 -> +3V3
- U101 pad F32: /PORT3 -> /FT_BE1
- U101 pad H27: /PORT3 -> /FT_D4
- U101 pad H28: /PORT3 -> /FT_D7
- U101 pad H30: /PORT3 -> /~{FT_RXF}
- U101 pad H31: /PORT3 -> unconnected-(U101D-PR26A/+/HS/RDQ29-PadH31)
- U101 pad H32: /PORT3 -> /~{FT_TXE}
- U101 pad J26: /PORT3 -> /FT_D6
- U101 pad J27: /PORT3 -> unconnected-(U101D-PR35D/-/RDQ41-PadJ27)
- U101 pad J29: /PORT3 -> +3V3
- U101 pad J30: /PORT3 -> /~{FT_WR}
- U101 pad J32: /PORT3 -> unconnected-(U101D-PR29B/-/HS/RDQSN29-PadJ32)
- U101 pad K26: /PORT3 -> /FT_D9
- U101 pad K27: /PORT3 -> /FT_D8
- U101 pad K28: /PORT3 -> /FT_D10
- U101 pad K29: /PORT3 -> /FT_D5
- U101 pad K30: /PORT3 -> /~{FT_RD}
- U101 pad K31: /PORT3 -> /~{FT_OE}
- U101 pad K32: /PORT3 -> /FT_D0
- U101 pad L26: /PORT3 -> /FT_D13
- U101 pad L27: /PORT3 -> /FT_D14
- U101 pad L29: /PORT3 -> /FT_D11
- U101 pad L30: /PORT3 -> /FT_D3
- U101 pad L31: /PORT3 -> /FT_D2
- U101 pad L32: /PORT3 -> /FT_D1
- U101 pad N26: /PORT3 -> +3V3
- U101 pad N27: /PORT3 -> /FT_D15
- U101 pad N29: /PORT3 -> /FT_D12
- U101 pad N30: /PORT3 -> +3V3
- U101 pad P26: /PORT3 -> unconnected-(U101D-PR44D/-/PCLKC2_0/RDQ41-PadP26)
- U101 pad P27: /PORT3 -> unconnected-(U101D-PR44C/+/PCLKT2_0/RDQ41-PadP27)
- U201 pad 1: /Power/FB_1V1 -> Net-(U201-SW)
- U201 pad 3: +5V -> /Power/FB_1V5
- U201 pad 4: Net-(U201-SW) -> +5V
- U201 pad 6: unconnected-(U201-NC-Pad6) -> GND
- U202 pad 1: /Power/FB_1V5 -> Net-(U202-SW)
- U202 pad 3: +5V -> /Power/FB_2V5
- U202 pad 4: Net-(U202-SW) -> +5V
- U202 pad 6: unconnected-(U202-NC-Pad6) -> GND
- U203 pad 1: /Power/FB_2V5 -> Net-(U203-SW)
- U203 pad 3: +5V -> /Power/FB_3V3
- U203 pad 4: Net-(U203-SW) -> +5V
- U203 pad 6: unconnected-(U203-NC-Pad6) -> GND
- U204 pad 1: /Power/FB_3V3 -> Net-(U204-SW)
- U204 pad 3: +5V -> /Power/FB_VDR
- U204 pad 4: Net-(U204-SW) -> +5V
- U204 pad 6: unconnected-(U204-NC-Pad6) -> GND
Routing:
- net /FT_BE1: track 0.00 -> 20.8 mm, vias 0 -> 1
- net /FT_BE0: track 0.00 -> 19.8 mm, vias 0 -> 1
- net /~{FT_WR}: track 0.00 -> 19.4 mm, vias 0 -> 1
- net /~{FT_OE}: track 0.00 -> 18.4 mm, vias 0 -> 1
- net /~{FT_TXE}: track 0.00 -> 17.4 mm, vias 0 -> 1
- net /FT_CLKOUT: track 0.00 -> 16.8 mm
- net /~{FT_RXF}: track 0.00 -> 15.8 mm, vias 0 -> 1
- net /~{FT_RD}: track 0.00 -> 15.8 mm, vias 0 -> 1
- net +3V3: track 0.00 -> 13.0 mm, vias 0 -> 10
- net GND: track 0.00 -> 12.4 mm, vias 0 -> 35
- net VD10: track 0.00 -> 9.86 mm, vias 0 -> 6
- net /~{FT_SIWU}: track 0.00 -> 7.79 mm
- net /FT_GPIO1: track 0.00 -> 7.34 mm
- net /FT_D11: track 0.00 -> 7.29 mm
- net /FT_D3: track 0.00 -> 7.28 mm
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
Commit message: Moved to PCIe connectors, added USB 3.0 Type B connector
Parts:
- removed J101: USB3_B_Micro, usb:AMPHENOL-GSB343K33HR
- removed RN301, RN302, RN303, RN304: 1k, Resistor_SMD:R_Array_Convex_8x0602
- added J102: GSB422137EU, connectors:AMPHENOL_GSB422137EU, B.Cu at (149.0, 67.0)
- added J301: 10061913-102PLF, connectors:AMPHENOL_10061913-102PLF, F.Cu at (167.7, 108.3)
- added J401: 10061913-102PLF, connectors:AMPHENOL_10061913-102PLF, F.Cu at (77.7, 108.3)
- added J501: 10061913-102PLF, connectors:AMPHENOL_10061913-102PLF, F.Cu at (202.7, 108.3)
- added J601: 10061913-102PLF, connectors:AMPHENOL_10061913-102PLF, F.Cu at (112.7, 108.3)
- added REF**: BUS_PCIexpress_x8, Connector_PCBEdge:BUS_PCIexpress_x8, F.Cu at (64.0, 121.5)
- moved J301 191.3 mm to (29.0, 96.0), turned to -90 degrees
- moved C101 64.0 mm to (142.6, 53.1)
- moved FB101 64.0 mm to (146.5, 53.0)
- moved U102 57.5 mm to (140.4, 70.2)
- moved R112 40.9 mm to (131.5, 90.4)
- moved C112 40.6 mm to (132.3, 90.4)
- moved C121 40.5 mm to (140.3, 89.5)
- moved C102 40.5 mm to (135.1, 79.7)
- moved C103 40.5 mm to (136.0, 79.7)
- moved C104 40.5 mm to (134.6, 79.7)
- moved C105 40.5 mm to (138.4, 80.3)
- moved C106 40.5 mm to (129.7, 81.4)
- moved C107 40.5 mm to (133.1, 79.7)
- moved C108 40.5 mm to (129.7, 85.6)
- moved C109 40.5 mm to (129.7, 82.1)
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- renumbered C113 to C102, C114 to C103, C118 to C104, C115 to C105, C120 to C106, C119 to C107, C116 to C108, C102 to C109, C121 to C110, C117 to C111, C103 to C112, C104 to C113, C105 to C114, C106 to C115, C107 to C116, C108 to C117, C109 to C118, C110 to C119, C111 to C120, C112 to C121, C215 to C205, C205 to C206, C206 to C207, C207 to C208, C208 to C209, C216 to C210, C209 to C211, C210 to C212, C211 to C213, C212 to C214, C217 to C215, U105 to U102, U106 to U103, U103 to U104, U104 to U105, U102 to U106, U206 to U201, U201 to U202, U202 to U203, U203 to U204, U204 to U205
Routing:
- net /RX_P: track 0.00 -> 31.4 mm
- net /RX_N: track 0.00 -> 29.2 mm
- net VD10: track 9.86 -> 32.2 mm, vias 6 -> 7
- net /TX_P: track 0.00 -> 19.9 mm
- net /TX_N: track 0.00 -> 16.9 mm
- net /FT_BE0: track 19.8 -> 3.90 mm, vias 1 -> 0
- net /FT_BE1: track 20.8 -> 4.92 mm, vias 1 -> 0
- net /~{FT_WR}: track 19.4 -> 3.57 mm, vias 1 -> 0
- net /~{FT_TXE}: track 17.4 -> 1.60 mm, vias 1 -> 0
- net /~{FT_RD}: track 15.8 -> 0.00 mm, vias 1 -> 0
- net /~{FT_OE}: track 18.4 -> 2.67 mm, vias 1 -> 0
- net /~{FT_RXF}: track 15.8 -> 0.49 mm
- net /FT_D0: track 5.82 -> 18.5 mm
- net /FT_D1: track 5.99 -> 17.8 mm
- net /FT_D2: track 6.64 -> 17.8 mm
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- added copper zone on B.Cu, net GND
- added copper zone on F.Cu, net GND
- added copper zone on In1.Cu, net GND
- added copper zone on In4.Cu, net GND
Other:
- board size 244 x 90 mm -> 184.5 x 127 mm

Commit message: Save
Parts:
- removed C205: 4.7u, passive:C_0603
- removed C210: 22p, passive:C_0402
- removed C215: 22u, passive:C_0603
- removed L205: 2.2u, Inductor_SMD:L_Abracon_ASPI-3012S
- removed R209, R210: ~, passive:R_0201
- removed U106: TXB0108DQSR, Package_SON:USON-20_2x4mm_P0.4mm
- removed U205: TPS62290, Package_SON:WSON-6-1EP_2x2mm_P0.65mm_EP1x1.6mm
- added C122: 0.1u, passive:C_0201, F.Cu at (160.6, 141.0)
- added C301: 0.1u, passive:C_0201, F.Cu at (176.1, 133.0)
- added C302: 0.1u, passive:C_0201, F.Cu at (176.1, 134.5)
- added C303: 0.1u, passive:C_0201, F.Cu at (176.1, 136.0)
- added C304: 0.1u, passive:C_0201, F.Cu at (176.1, 137.5)
- added C305: 0.1u, passive:C_0201, F.Cu at (178.1, 133.0)
- added C306: 0.1u, passive:C_0201, F.Cu at (178.1, 134.5)
- added C307: 0.1u, passive:C_0201, F.Cu at (178.1, 136.0)
- added C308: 0.1u, passive:C_0201, F.Cu at (178.1, 137.5)
- added C309: 0.1u, passive:C_0201, F.Cu at (180.2, 133.0)
- added C310: 0.1u, passive:C_0201, F.Cu at (180.2, 134.5)
- added C311: 0.1u, passive:C_0201, F.Cu at (180.2, 136.0)
- added C312: 0.1u, passive:C_0201, F.Cu at (180.2, 137.5)
- added C313: 0.1u, passive:C_0201, F.Cu at (182.2, 133.0)
- added C314: 0.1u, passive:C_0201, F.Cu at (182.2, 134.5)
- added C315: 0.1u, passive:C_0201, F.Cu at (182.2, 136.0)
- added C316: 0.1u, passive:C_0201, F.Cu at (182.2, 137.5)
- added C401: 0.1u, passive:C_0201, F.Cu at (89.1, 133.5)
- added C402: 0.1u, passive:C_0201, F.Cu at (89.1, 135.0)
- added C403: 0.1u, passive:C_0201, F.Cu at (89.1, 136.5)
- added C404: 0.1u, passive:C_0201, F.Cu at (89.1, 138.0)
- added C405: 0.1u, passive:C_0201, F.Cu at (91.1, 133.5)
- added C406: 0.1u, passive:C_0201, F.Cu at (91.1, 135.0)
- added C407: 0.1u, passive:C_0201, F.Cu at (91.1, 136.5)
- added C408: 0.1u, passive:C_0201, F.Cu at (91.1, 138.0)
- added C409: 0.1u, passive:C_0201, F.Cu at (93.2, 133.5)
- added C410: 0.1u, passive:C_0201, F.Cu at (93.2, 135.0)
- added C411: 0.1u, passive:C_0201, F.Cu at (93.2, 136.5)
- added C412: 0.1u, passive:C_0201, F.Cu at (93.2, 138.0)
- added C413: 0.1u, passive:C_0201, F.Cu at (95.2, 133.5)
- added C414: 0.1u, passive:C_0201, F.Cu at (95.2, 135.0)
- added C415: 0.1u, passive:C_0201, F.Cu at (95.2, 136.5)
- added C416: 0.1u, passive:C_0201, F.Cu at (95.2, 138.0)
- added C501: 0.1u, passive:C_0201, F.Cu at (218.7, 135.5)
- added C502: 0.1u, passive:C_0201, F.Cu at (218.7, 137.0)
- added C503: 0.1u, passive:C_0201, F.Cu at (218.7, 138.5)
- added C504: 0.1u, passive:C_0201, F.Cu at (218.7, 140.0)
- added C505: 0.1u, passive:C_0201, F.Cu at (220.8, 135.5)
- added C506: 0.1u, passive:C_0201, F.Cu at (220.8, 137.0)
- added C507: 0.1u, passive:C_0201, F.Cu at (220.8, 138.5)
- added C508: 0.1u, passive:C_0201, F.Cu at (220.8, 140.0)
- added C509: 0.1u, passive:C_0201, F.Cu at (222.8, 135.5)
- added C510: 0.1u, passive:C_0201, F.Cu at (222.8, 137.0)
- added C511: 0.1u, passive:C_0201, F.Cu at (222.8, 138.5)
- added C512: 0.1u, passive:C_0201, F.Cu at (222.8, 140.0)
- added C513: 0.1u, passive:C_0201, F.Cu at (224.9, 135.5)
- added C514: 0.1u, passive:C_0201, F.Cu at (224.9, 137.0)
- added C515: 0.1u, passive:C_0201, F.Cu at (224.9, 138.5)
- added C516: 0.1u, passive:C_0201, F.Cu at (224.9, 140.0)
- added C601: 0.1u, passive:C_0201, B.Cu at (114.9, 114.8)
- added C602: 0.1u, passive:C_0201, F.Cu at (122.6, 136.5)
- added C603: 0.1u, passive:C_0201, F.Cu at (122.6, 138.0)
- added C604: 0.1u, passive:C_0201, F.Cu at (122.6, 139.5)
- added C605: 0.1u, passive:C_0201, F.Cu at (124.7, 135.0)
- added C606: 0.1u, passive:C_0201, F.Cu at (124.7, 136.5)
- added C607: 0.1u, passive:C_0201, F.Cu at (124.7, 138.0)
- added C608: 0.1u, passive:C_0201, F.Cu at (124.7, 139.5)
- added C609: 0.1u, passive:C_0201, B.Cu at (116.1, 114.2)
- added C610: 0.1u, passive:C_0201, F.Cu at (126.7, 136.5)
- added C611: 0.1u, passive:C_0201, F.Cu at (126.7, 138.0)
- added C612: 0.1u, passive:C_0201, F.Cu at (126.7, 139.5)
- added C613: 0.1u, passive:C_0201, F.Cu at (128.8, 135.0)
- added C614: 0.1u, passive:C_0201, F.Cu at (128.8, 136.5)
- added C615: 0.1u, passive:C_0201, F.Cu at (128.8, 138.0)
- added C616: 0.1u, passive:C_0201, F.Cu at (128.8, 139.5)
- added D101: LED_Small, LED_SMD:LED_0402_1005Metric, F.Cu at (161.3, 145.7)
- added H101: MountingHole_Pad, MountingHole:MountingHole_3.2mm_M3_Pad_Via, F.Cu at (79.0, 125.5)
- added H102: MountingHole_Pad, MountingHole:MountingHole_3.2mm_M3_Pad_Via, F.Cu at (79.0, 64.5)
- added H103: MountingHole_Pad, MountingHole:MountingHole_3.2mm_M3_Pad_Via, F.Cu at (145.5, 64.5)
- added H104: MountingHole_Pad, MountingHole:MountingHole_3.2mm_M3_Pad_Via, F.Cu at (222.0, 64.5)
- added H105: MountingHole_Pad, MountingHole:MountingHole_3.2mm_M3_Pad_Via, F.Cu at (150.5, 125.5)
- added H106: MountingHole_Pad, MountingHole:MountingHole_3.2mm_M3_Pad_Via, F.Cu at (222.0, 125.5)
- added H107: MountingHole_Pad, MountingHole:MountingHole_3.2mm_M3_Pad_Via, F.Cu at (168.5, 64.5)
- added J101: TC2050, Connector:Tag-Connect_TC2050-IDC-NL_2x05_P1.27mm_Vertical, B.Cu at (169.5, 125.5)
- added R129: 1k, passive:R_0201, F.Cu at (160.6, 142.5)
- added R130: 1k, passive:R_0201, F.Cu at (160.6, 144.0)
- added R131: 1k, passive:R_0201, F.Cu at (162.7, 141.0)
- added R132: 1k, passive:R_0201, F.Cu at (162.7, 142.5)
- added R133: 10k, passive:R_0201, F.Cu at (162.7, 144.0)
- added R134: 1k, passive:R_0201, F.Cu at (164.7, 141.0)
- added R135: 0, passive:R_0201, F.Cu at (164.7, 142.5)
- added R136: 10k, passive:R_0201, F.Cu at (164.7, 144.0)
- added U108: USBLC6-2P6, Package_TO_SOT_SMD:SOT-666, F.Cu at (163.4, 71.9)
- added U301: TXB0108DQSR, Package_SON:USON-20_2x4mm_P0.4mm, F.Cu at (170.5, 114.5)
- added U303: TXB0108DQSR, Package_SON:USON-20_2x4mm_P0.4mm, F.Cu at (170.5, 100.5)
- added U305: TXB0108DQSR, Package_SON:USON-20_2x4mm_P0.4mm, F.Cu at (170.5, 88.5)
- added U307: TXB0108DQSR, Package_SON:USON-20_2x4mm_P0.4mm, F.Cu at (170.5, 76.5)
- added U309: TXB0108DQSR, Package_SON:USON-20_2x4mm_P0.4mm, F.Cu at (185.0, 114.5)
- added U310: TXB0108DQSR, Package_SON:USON-20_2x4mm_P0.4mm, F.Cu at (185.0, 100.5)
- added U311: TXB0108DQSR, Package_SON:USON-20_2x4mm_P0.4mm, F.Cu at (185.0, 88.5)
- added U312: TXB0108DQSR, Package_SON:USON-20_2x4mm_P0.4mm, F.Cu at (185.0, 76.5)
- added U401: TXB0108DQSR, Package_SON:USON-20_2x4mm_P0.4mm, F.Cu at (80.5, 114.5)
- added U403: TXB0108DQSR, Package_SON:USON-20_2x4mm_P0.4mm, F.Cu at (80.5, 100.5)
- added U405: TXB0108DQSR, Package_SON:USON-20_2x4mm_P0.4mm, F.Cu at (80.5, 88.5)
- added U407: TXB0108DQSR, Package_SON:USON-20_2x4mm_P0.4mm, F.Cu at (80.5, 76.5)
- added U409: TXB0108DQSR, Package_SON:USON-20_2x4mm_P0.4mm, F.Cu at (95.0, 114.5)
- added U410: TXB0108DQSR, Package_SON:USON-20_2x4mm_P0.4mm, F.Cu at (95.0, 100.5)
- added U411: TXB0108DQSR, Package_SON:USON-20_2x4mm_P0.4mm, F.Cu at (95.0, 88.5)
- added U412: TXB0108DQSR, Package_SON:USON-20_2x4mm_P0.4mm, F.Cu at (95.0, 76.5)
- added U501: TXB0108DQSR, Package_SON:USON-20_2x4mm_P0.4mm, F.Cu at (205.5, 114.5)
- added U503: TXB0108DQSR, Package_SON:USON-20_2x4mm_P0.4mm, F.Cu at (205.5, 100.5)
- added U505: TXB0108DQSR, Package_SON:USON-20_2x4mm_P0.4mm, F.Cu at (205.5, 88.5)
- added U507: TXB0108DQSR, Package_SON:USON-20_2x4mm_P0.4mm, F.Cu at (205.5, 76.5)
- added U509: TXB0108DQSR, Package_SON:USON-20_2x4mm_P0.4mm, F.Cu at (220.0, 114.5)
- added U510: TXB0108DQSR, Package_SON:USON-20_2x4mm_P0.4mm, F.Cu at (220.0, 100.5)
- added U511: TXB0108DQSR, Package_SON:USON-20_2x4mm_P0.4mm, F.Cu at (220.0, 88.5)
- added U512: TXB0108DQSR, Package_SON:USON-20_2x4mm_P0.4mm, F.Cu at (220.0, 76.5)
- added U601: TXB0108DQSR, Package_SON:USON-20_2x4mm_P0.4mm, F.Cu at (115.5, 114.5)
- added U603: TXB0108DQSR, Package_SON:USON-20_2x4mm_P0.4mm, F.Cu at (115.5, 100.5)
- added U605: TXB0108DQSR, Package_SON:USON-20_2x4mm_P0.4mm, F.Cu at (115.5, 88.5)
- added U607: TXB0108DQSR, Package_SON:USON-20_2x4mm_P0.4mm, F.Cu at (115.5, 76.5)
- added U609: TXB0108DQSR, Package_SON:USON-20_2x4mm_P0.4mm, F.Cu at (130.0, 114.5)
- added U610: TXB0108DQSR, Package_SON:USON-20_2x4mm_P0.4mm, F.Cu at (130.0, 100.5)
- added U611: TXB0108DQSR, Package_SON:USON-20_2x4mm_P0.4mm, F.Cu at (130.0, 88.5)
- added U612: TXB0108DQSR, Package_SON:USON-20_2x4mm_P0.4mm, F.Cu at (130.0, 76.5)
- C206, C207, C208, C209: footprint passive:C_0402 -> passive:C_0201
- U104: moved to B.Cu
- U105: value TCA9535RTWR -> W25Q128JVP; footprint Package_DFN_QFN:WQFN-24-1EP_4x4mm_P0.5mm_EP2.45x2.45mm -> Package_SON:WSON-8-1EP_6x5mm_P1.27mm_EP3.4x4.3mm
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Connections:
- C207 pad 2: +1V5 -> Vdrive
- C212 pad 1: +1V5 -> Vdrive
- J102 pad 2: /D_N -> /D_C_N
- J102 pad 3: /D_P -> /D_C_P
- J301 pad A1: /Input Port 1/IO_0 -> /Input Port 1/IO_C_0
- J301 pad A10: /Input Port 1/IO_6 -> /Input Port 1/IO_C_6
- J301 pad A12: /Input Port 1/IO_7 -> /Input Port 1/IO_C_7
- J301 pad A13: /Input Port 1/IO_8 -> /Input Port 1/IO_C_8
- J301 pad A15: /Input Port 1/IO_9 -> /Input Port 1/IO_C_9
- J301 pad A16: /Input Port 1/IO_10 -> /Input Port 1/IO_C_10
- J301 pad A18: /Input Port 1/IO_11 -> /Input Port 1/IO_C_11
- J301 pad A19: /Input Port 1/IO_12 -> /Input Port 1/IO_C_12
- J301 pad A21: /Input Port 1/IO_13 -> /Input Port 1/IO_C_13
- J301 pad A22: /Input Port 1/IO_14 -> /Input Port 1/IO_C_14
- J301 pad A24: /Input Port 1/IO_15 -> /Input Port 1/IO_C_15
- J301 pad A25: /Input Port 1/IO_16 -> /Input Port 1/IO_C_16
- J301 pad A27: /Input Port 1/IO_17 -> /Input Port 1/IO_C_17
- J301 pad A28: /Input Port 1/IO_18 -> /Input Port 1/IO_C_18
- J301 pad A3: /Input Port 1/IO_1 -> /Input Port 1/IO_C_1
- J301 pad A30: /Input Port 1/IO_19 -> /Input Port 1/IO_C_19
- J301 pad A31: /Input Port 1/IO_20 -> /Input Port 1/IO_C_20
- J301 pad A33: /Input Port 1/IO_21 -> /Input Port 1/IO_C_21
- J301 pad A34: /Input Port 1/IO_22 -> /Input Port 1/IO_C_22
- J301 pad A36: /Input Port 1/IO_23 -> /Input Port 1/IO_C_23
- J301 pad A37: /Input Port 1/IO_24 -> /Input Port 1/IO_C_24
- J301 pad A39: /Input Port 1/IO_25 -> /Input Port 1/IO_C_25
- J301 pad A4: /Input Port 1/IO_2 -> /Input Port 1/IO_C_2
- J301 pad A40: /Input Port 1/IO_26 -> /Input Port 1/IO_C_26
- J301 pad A42: /Input Port 1/IO_27 -> /Input Port 1/IO_C_27
- J301 pad A43: /Input Port 1/IO_28 -> /Input Port 1/IO_C_28
- J301 pad A45: /Input Port 1/IO_29 -> /Input Port 1/IO_C_29
- J301 pad A46: /Input Port 1/IO_30 -> /Input Port 1/IO_C_30
- J301 pad A47: GND -> /Input Port 1/IO_C_31
- J301 pad A48: /Input Port 1/TRANSLATOR_VCC_OUT -> GND
- J301 pad A49: +3V3 -> /Input Port 1/SDA
- J301 pad A6: /Input Port 1/IO_3 -> /Input Port 1/IO_C_3
- J301 pad A7: /Input Port 1/IO_4 -> /Input Port 1/IO_C_4
- J301 pad A9: /Input Port 1/IO_5 -> /Input Port 1/IO_C_5
- J301 pad B1: /Input Port 1/IO_32 -> /Input Port 1/IO_C_32
- J301 pad B10: /Input Port 1/IO_38 -> /Input Port 1/IO_C_38
- J301 pad B12: /Input Port 1/IO_39 -> /Input Port 1/IO_C_39
- J301 pad B13: /Input Port 1/IO_40 -> /Input Port 1/IO_C_40
- J301 pad B15: /Input Port 1/IO_41 -> /Input Port 1/IO_C_41
- J301 pad B16: /Input Port 1/IO_42 -> /Input Port 1/IO_C_42
- J301 pad B18: /Input Port 1/IO_43 -> /Input Port 1/IO_C_43
- J301 pad B19: /Input Port 1/IO_44 -> /Input Port 1/IO_C_44
- J301 pad B21: /Input Port 1/IO_45 -> /Input Port 1/IO_C_45
- J301 pad B22: /Input Port 1/IO_46 -> /Input Port 1/IO_C_46
- J301 pad B24: /Input Port 1/IO_47 -> /Input Port 1/IO_C_47
- J301 pad B25: /Input Port 1/IO_48 -> /Input Port 1/IO_C_48
- J301 pad B27: /Input Port 1/IO_49 -> /Input Port 1/IO_C_49
- J301 pad B28: /Input Port 1/IO_50 -> /Input Port 1/IO_C_50
- J301 pad B3: /Input Port 1/IO_33 -> /Input Port 1/IO_C_33
- J301 pad B30: /Input Port 1/IO_51 -> /Input Port 1/IO_C_51
- J301 pad B31: /Input Port 1/IO_52 -> /Input Port 1/IO_C_52
- J301 pad B33: /Input Port 1/IO_53 -> /Input Port 1/IO_C_53
- J301 pad B34: /Input Port 1/IO_54 -> /Input Port 1/IO_C_54
- J301 pad B36: /Input Port 1/IO_55 -> /Input Port 1/IO_C_55
- J301 pad B37: /Input Port 1/IO_56 -> /Input Port 1/IO_C_56
- J301 pad B39: /Input Port 1/IO_57 -> /Input Port 1/IO_C_57
- J301 pad B4: /Input Port 1/IO_34 -> /Input Port 1/IO_C_34
- J301 pad B40: /Input Port 1/IO_58 -> /Input Port 1/IO_C_58
- J301 pad B42: /Input Port 1/IO_59 -> /Input Port 1/IO_C_59
- J301 pad B43: /Input Port 1/IO_60 -> /Input Port 1/IO_C_60
- J301 pad B45: /Input Port 1/IO_61 -> /Input Port 1/IO_C_61
- J301 pad B46: /Input Port 1/IO_62 -> /Input Port 1/IO_C_62
- J301 pad B47: GND -> /Input Port 1/IO_C_63
- J301 pad B48: /Input Port 1/SDA -> +3V3
- J301 pad B6: /Input Port 1/IO_35 -> /Input Port 1/IO_C_35
- J301 pad B7: /Input Port 1/IO_36 -> /Input Port 1/IO_C_36
- J301 pad B9: /Input Port 1/IO_37 -> /Input Port 1/IO_C_37
- J401 pad A1: /Input Port 2/IO_0 -> /Input Port 2/IO_C_0
- J401 pad A10: /Input Port 2/IO_6 -> /Input Port 2/IO_C_6
- J401 pad A12: /Input Port 2/IO_7 -> /Input Port 2/IO_C_7
- J401 pad A13: /Input Port 2/IO_8 -> /Input Port 2/IO_C_8
- J401 pad A15: /Input Port 2/IO_9 -> /Input Port 2/IO_C_9
- J401 pad A16: /Input Port 2/IO_10 -> /Input Port 2/IO_C_10
- J401 pad A18: /Input Port 2/IO_11 -> /Input Port 2/IO_C_11
- J401 pad A19: /Input Port 2/IO_12 -> /Input Port 2/IO_C_12
- J401 pad A21: /Input Port 2/IO_13 -> /Input Port 2/IO_C_13
- J401 pad A22: /Input Port 2/IO_14 -> /Input Port 2/IO_C_14
- J401 pad A24: /Input Port 2/IO_15 -> /Input Port 2/IO_C_15
- J401 pad A25: /Input Port 2/IO_16 -> /Input Port 2/IO_C_16
- J401 pad A27: /Input Port 2/IO_17 -> /Input Port 2/IO_C_17
- J401 pad A28: /Input Port 2/IO_18 -> /Input Port 2/IO_C_18
- J401 pad A3: /Input Port 2/IO_1 -> /Input Port 2/IO_C_1
- J401 pad A30: /Input Port 2/IO_19 -> /Input Port 2/IO_C_19
- J401 pad A31: /Input Port 2/IO_20 -> /Input Port 2/IO_C_20
- J401 pad A33: /Input Port 2/IO_21 -> /Input Port 2/IO_C_21
- J401 pad A34: /Input Port 2/IO_22 -> /Input Port 2/IO_C_22
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Routing:
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Other:
- board size 184.5 x 127 mm -> 200 x 127 mm
- board text added: "1"
- board text added: "2"
- board text added: "3"
- board text added: "4"
- board text added: "ETHER"
- board text added: "GH: {GITHASH}"
- board text added: "LISTEN TO THE"
- board text added: "v1.0"
