File: hardware/ether.kicad_pcb (KiCad board)
At the start: 6 copper layers, 200 x 127 mm, 206 parts, among them J101 TC2050, J102 GSB422137EU, J301 10061913-102PLF, J301 SS-74500-022, J401 10061913-102PLF, J501 10061913-102PLF, J601 10061913-102PLF, U101 ECP5U_85_CABGA756, U102 PUSB3FR4Z, U103 FT600Q, U104 TCA9535RTWR, U105 W25Q128JVP, U108 USBLC6-2P6, U201 TPS62290, U202 TPS62290, U203 TPS62290, U204 TPS62290, U301 TXB0108DQSR, U303 TXB0108DQSR, U305 TXB0108DQSR, U307 TXB0108DQSR, U309 TXB0108DQSR, U310 TXB0108DQSR, U311 TXB0108DQSR, U312 TXB0108DQSR, U401 TXB0108DQSR, U403 TXB0108DQSR, U405 TXB0108DQSR, U407 TXB0108DQSR, U409 TXB0108DQSR, U410 TXB0108DQSR, U411 TXB0108DQSR, U412 TXB0108DQSR, U501 TXB0108DQSR, U503 TXB0108DQSR, U505 TXB0108DQSR, U507 TXB0108DQSR, U509 TXB0108DQSR, U510 TXB0108DQSR, U511 TXB0108DQSR, U512 TXB0108DQSR, U601 TXB0108DQSR, U603 TXB0108DQSR, U605 TXB0108DQSR, U607 TXB0108DQSR, U609 TXB0108DQSR, U610 TXB0108DQSR, U611 TXB0108DQSR, U612 TXB0108DQSR, Y101 30 MHz

Commit message: Save
Parts:
- added C205: 4.7u, passive:C_0603, F.Cu at (135.2, 56.7)
- added C210: 22p, passive:C_0201, F.Cu at (137.9, 53.2)
- added C215: 22u, passive:C_0603, F.Cu at (137.4, 54.8)
- added L205: 2.2u, Inductor_SMD:L_Abracon_ASPI-3012S, F.Cu at (140.4, 56.1)
- added R209: ~, passive:R_0201, F.Cu at (137.9, 53.8)
- added R210: ~, passive:R_0201, F.Cu at (136.8, 53.8)
- added REF**: MountingHole_3.2mm_M3_Pad_Via, MountingHole:MountingHole_3.2mm_M3_Pad_Via, F.Cu at (55.5, 159.5)
- added REF**: MountingHole_3.2mm_M3_Pad_Via, MountingHole:MountingHole_3.2mm_M3_Pad_Via, F.Cu at (30.0, 159.5)
- added REF**: MountingHole_3.2mm_M3_Pad_Via, MountingHole:MountingHole_3.2mm_M3_Pad_Via, F.Cu at (55.5, 32.5)
- added REF**: MountingHole_3.2mm_M3_Pad_Via, MountingHole:MountingHole_3.2mm_M3_Pad_Via, F.Cu at (30.0, 32.5)
- added U205: TPS62290, Package_SON:WSON-6-1EP_2x2mm_P0.65mm_EP1x1.6mm, F.Cu at (137.2, 56.7)
- moved C309 92.9 mm to (87.3, 133.5)
- moved C310 92.9 mm to (87.3, 135.0)
- moved C311 92.9 mm to (87.3, 136.5)
- moved C312 92.9 mm to (87.3, 138.0)
- moved C301 92.9 mm to (83.2, 133.5)
- moved C302 92.9 mm to (83.2, 135.0)
- moved C303 92.9 mm to (83.2, 136.5)
- moved C304 92.9 mm to (83.2, 138.0)
- moved C305 92.9 mm to (85.3, 133.5)
- moved C306 92.9 mm to (85.3, 135.0)
- moved C307 92.9 mm to (85.3, 136.5)
- moved C308 92.9 mm to (85.3, 138.0)
- moved C313 92.9 mm to (89.4, 133.5)
- moved C314 92.9 mm to (89.4, 135.0)
- moved C315 92.9 mm to (89.4, 136.5)
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Connections:
- C301 pad 1: +3V3 -> +1V5
- C302 pad 1: +3V3 -> +1V5
- C303 pad 1: +3V3 -> +1V5
- C304 pad 1: +3V3 -> +1V5
- C305 pad 1: +3V3 -> +1V5
- C306 pad 1: +3V3 -> +1V5
- C307 pad 1: +3V3 -> +1V5
- C308 pad 1: +3V3 -> +1V5
- C401 pad 1: +3V3 -> +1V5
- C402 pad 1: +3V3 -> +1V5
- C403 pad 1: +3V3 -> +1V5
- C404 pad 1: +3V3 -> +1V5
- C405 pad 1: +3V3 -> +1V5
- C406 pad 1: +3V3 -> +1V5
- C407 pad 1: +3V3 -> +1V5
- C408 pad 1: +3V3 -> +1V5
- C501 pad 1: +3V3 -> +1V5
- C502 pad 1: +3V3 -> +1V5
- C503 pad 1: +3V3 -> +1V5
- C504 pad 1: +3V3 -> +1V5
- C505 pad 1: +3V3 -> +1V5
- C506 pad 1: +3V3 -> +1V5
- C507 pad 1: +3V3 -> +1V5
- C508 pad 1: +3V3 -> +1V5
- C601 pad 1: +3V3 -> +1V5
- C602 pad 1: +3V3 -> +1V5
- C603 pad 1: +3V3 -> +1V5
- C604 pad 1: +3V3 -> +1V5
- C605 pad 1: +3V3 -> +1V5
- C606 pad 1: +3V3 -> +1V5
- C607 pad 1: +3V3 -> +1V5
- C608 pad 1: +3V3 -> +1V5
- U301 pad 5: +3V3 -> +1V5
- U303 pad 5: +3V3 -> +1V5
- U305 pad 5: +3V3 -> +1V5
- U307 pad 5: +3V3 -> +1V5
- U309 pad 5: +3V3 -> +1V5
- U310 pad 5: +3V3 -> +1V5
- U311 pad 5: +3V3 -> +1V5
- U312 pad 5: +3V3 -> +1V5
- U401 pad 5: +3V3 -> +1V5
- U403 pad 5: +3V3 -> +1V5
- U405 pad 5: +3V3 -> +1V5
- U407 pad 5: +3V3 -> +1V5
- U409 pad 5: +3V3 -> +1V5
- U410 pad 5: +3V3 -> +1V5
- U411 pad 5: +3V3 -> +1V5
- U412 pad 5: +3V3 -> +1V5
- U501 pad 5: +3V3 -> +1V5
- U503 pad 5: +3V3 -> +1V5
- U505 pad 5: +3V3 -> +1V5
- U507 pad 5: +3V3 -> +1V5
- U509 pad 5: +3V3 -> +1V5
- U510 pad 5: +3V3 -> +1V5
- U511 pad 5: +3V3 -> +1V5
- U512 pad 5: +3V3 -> +1V5
- U601 pad 5: +3V3 -> +1V5
- U603 pad 5: +3V3 -> +1V5
- U605 pad 5: +3V3 -> +1V5
- U607 pad 5: +3V3 -> +1V5
- U609 pad 5: +3V3 -> +1V5
- U610 pad 5: +3V3 -> +1V5
- U611 pad 5: +3V3 -> +1V5
- U612 pad 5: +3V3 -> +1V5
Routing:
- net +1V5: track 0.00 -> 32.9 mm, vias 0 -> 32
- net +3V3: track 47.2 -> 17.4 mm, vias 45 -> 10
- net /FT_D0: track 14.0 -> 4.44 mm
- net /FT_D1: track 13.7 -> 4.20 mm
- net /FT_D2: track 13.9 -> 5.16 mm
- net /FT_D4: track 7.56 -> 0.00 mm
- net /FT_D3: track 12.9 -> 6.00 mm
- net /FT_D5: track 6.51 -> 0.00 mm
- net /FT_D6: track 5.59 -> 0.00 mm
- net /FT_CLKOUT: track 10.4 -> 15.4 mm
- net /Power/FB_3V3: track 2.85 -> 7.61 mm
- net /FT_D7: track 4.62 -> 0.00 mm
- net /~{FT_TXE}: track 11.0 -> 14.3 mm
- net unconnected-(U101D-PR29B/-/HS/RDQSN29-PadJ32): track 1.70 -> 4.84 mm
- net /~{FT_OE}: track 15.9 -> 18.8 mm
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Other:
- board size 200 x 127 mm -> 200 x 134 mm

Commit message: Moved to new level translator with less input current requirement
Parts:
- removed C205: 4.7u, passive:C_0603
- removed C210: 22p, passive:C_0201
- removed C215: 22u, passive:C_0603
- removed L205: 2.2u, Inductor_SMD:L_Abracon_ASPI-3012S
- removed R209, R210: ~, passive:R_0201
- removed U205: TPS62290, Package_SON:WSON-6-1EP_2x2mm_P0.65mm_EP1x1.6mm
- U301, U303, U305, U307, U309, U310, U311, U312, U401, U403, U405, U407, U409, U410, U411, U412, U501, U503, U505, U507, U509, U510, U511, U512, U601, U603, U605, U607, U609, U610, U611, U612: footprint Package_SON:USON-20_2x4mm_P0.4mm -> Package_SO:TSSOP-20_4.4x6.5mm_P0.65mm
- moved U104 12.0 mm to (42.4, 157.5)
- moved U309 2.00 mm to (97.0, 114.5)
- moved U310 2.00 mm to (97.0, 100.5)
- moved U311 2.00 mm to (97.0, 88.5)
- moved U312 2.00 mm to (97.0, 76.5)
- moved U409 2.00 mm to (132.0, 114.5)
- moved U410 2.00 mm to (132.0, 100.5)
- moved U411 2.00 mm to (132.0, 88.5)
- moved U412 2.00 mm to (132.0, 76.5)
- moved U509 2.00 mm to (187.0, 114.5)
- moved U510 2.00 mm to (187.0, 100.5)
- moved U511 2.00 mm to (187.0, 88.5)
- moved U512 2.00 mm to (187.0, 76.5)
- moved U609 2.00 mm to (222.0, 114.5)
- moved U610 2.00 mm to (222.0, 100.5)
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Connections:
- U301 pad 10: /Input Port 1/IO_0 -> /Input Port 1/OE
- U301 pad 11: /Input Port 1/IO_C_0 -> GND
- U301 pad 12: /Input Port 1/IO_C_1 -> /Input Port 1/IO_C_0
- U301 pad 13: /Input Port 1/IO_C_2 -> /Input Port 1/IO_C_1
- U301 pad 14: /Input Port 1/IO_C_3 -> /Input Port 1/IO_C_2
- U301 pad 15: GND -> /Input Port 1/IO_C_3
- U301 pad 16: Vdrive -> /Input Port 1/IO_C_4
- U301 pad 17: /Input Port 1/IO_C_4 -> /Input Port 1/IO_C_5
- U301 pad 18: /Input Port 1/IO_C_5 -> /Input Port 1/IO_C_6
- U301 pad 19: /Input Port 1/IO_C_6 -> Vdrive
- U301 pad 2: /Input Port 1/IO_6 -> +1V5
- U301 pad 3: /Input Port 1/IO_5 -> /Input Port 1/IO_6
- U301 pad 4: /Input Port 1/IO_4 -> /Input Port 1/IO_5
- U301 pad 5: +1V5 -> /Input Port 1/IO_4
- U301 pad 6: /Input Port 1/OE -> /Input Port 1/IO_3
- U301 pad 7: /Input Port 1/IO_3 -> /Input Port 1/IO_2
- U301 pad 8: /Input Port 1/IO_2 -> /Input Port 1/IO_1
- U301 pad 9: /Input Port 1/IO_1 -> /Input Port 1/IO_0
- U303 pad 10: /Input Port 1/IO_8 -> /Input Port 1/OE
- U303 pad 11: /Input Port 1/IO_C_8 -> GND
- U303 pad 12: /Input Port 1/IO_C_9 -> /Input Port 1/IO_C_8
- U303 pad 13: /Input Port 1/IO_C_10 -> /Input Port 1/IO_C_9
- U303 pad 14: /Input Port 1/IO_C_11 -> /Input Port 1/IO_C_10
- U303 pad 15: GND -> /Input Port 1/IO_C_11
- U303 pad 16: Vdrive -> /Input Port 1/IO_C_12
- U303 pad 17: /Input Port 1/IO_C_12 -> /Input Port 1/IO_C_13
- U303 pad 18: /Input Port 1/IO_C_13 -> /Input Port 1/IO_C_14
- U303 pad 19: /Input Port 1/IO_C_14 -> Vdrive
- U303 pad 2: /Input Port 1/IO_14 -> +1V5
- U303 pad 3: /Input Port 1/IO_13 -> /Input Port 1/IO_14
- U303 pad 4: /Input Port 1/IO_12 -> /Input Port 1/IO_13
- U303 pad 5: +1V5 -> /Input Port 1/IO_12
- U303 pad 6: /Input Port 1/OE -> /Input Port 1/IO_11
- U303 pad 7: /Input Port 1/IO_11 -> /Input Port 1/IO_10
- U303 pad 8: /Input Port 1/IO_10 -> /Input Port 1/IO_9
- U303 pad 9: /Input Port 1/IO_9 -> /Input Port 1/IO_8
- U305 pad 10: /Input Port 1/IO_16 -> /Input Port 1/OE
- U305 pad 11: /Input Port 1/IO_C_16 -> GND
- U305 pad 12: /Input Port 1/IO_C_17 -> /Input Port 1/IO_C_16
- U305 pad 13: /Input Port 1/IO_C_18 -> /Input Port 1/IO_C_17
- U305 pad 14: /Input Port 1/IO_C_19 -> /Input Port 1/IO_C_18
- U305 pad 15: GND -> /Input Port 1/IO_C_19
- U305 pad 16: Vdrive -> /Input Port 1/IO_C_20
- U305 pad 17: /Input Port 1/IO_C_20 -> /Input Port 1/IO_C_21
- U305 pad 18: /Input Port 1/IO_C_21 -> /Input Port 1/IO_C_22
- U305 pad 19: /Input Port 1/IO_C_22 -> Vdrive
- U305 pad 2: /Input Port 1/IO_22 -> +1V5
- U305 pad 3: /Input Port 1/IO_21 -> /Input Port 1/IO_22
- U305 pad 4: /Input Port 1/IO_20 -> /Input Port 1/IO_21
- U305 pad 5: +1V5 -> /Input Port 1/IO_20
- U305 pad 6: /Input Port 1/OE -> /Input Port 1/IO_19
- U305 pad 7: /Input Port 1/IO_19 -> /Input Port 1/IO_18
- U305 pad 8: /Input Port 1/IO_18 -> /Input Port 1/IO_17
- U305 pad 9: /Input Port 1/IO_17 -> /Input Port 1/IO_16
- U307 pad 10: /Input Port 1/IO_24 -> /Input Port 1/OE
- U307 pad 11: /Input Port 1/IO_C_24 -> GND
- U307 pad 12: /Input Port 1/IO_C_25 -> /Input Port 1/IO_C_24
- U307 pad 13: /Input Port 1/IO_C_26 -> /Input Port 1/IO_C_25
- U307 pad 14: /Input Port 1/IO_C_27 -> /Input Port 1/IO_C_26
- U307 pad 15: GND -> /Input Port 1/IO_C_27
- U307 pad 16: Vdrive -> /Input Port 1/IO_C_28
- U307 pad 17: /Input Port 1/IO_C_28 -> /Input Port 1/IO_C_29
- U307 pad 18: /Input Port 1/IO_C_29 -> /Input Port 1/IO_C_30
- U307 pad 19: /Input Port 1/IO_C_30 -> Vdrive
- U307 pad 2: /Input Port 1/IO_30 -> +1V5
- U307 pad 3: /Input Port 1/IO_29 -> /Input Port 1/IO_30
- U307 pad 4: /Input Port 1/IO_28 -> /Input Port 1/IO_29
- U307 pad 5: +1V5 -> /Input Port 1/IO_28
- U307 pad 6: /Input Port 1/OE -> /Input Port 1/IO_27
- U307 pad 7: /Input Port 1/IO_27 -> /Input Port 1/IO_26
- U307 pad 8: /Input Port 1/IO_26 -> /Input Port 1/IO_25
- U307 pad 9: /Input Port 1/IO_25 -> /Input Port 1/IO_24
- U309 pad 10: /Input Port 1/IO_39 -> /Input Port 1/OE
- U309 pad 11: /Input Port 1/IO_C_39 -> GND
- U309 pad 12: /Input Port 1/IO_C_38 -> /Input Port 1/IO_C_39
- U309 pad 13: /Input Port 1/IO_C_37 -> /Input Port 1/IO_C_38
- U309 pad 14: /Input Port 1/IO_C_36 -> /Input Port 1/IO_C_37
- U309 pad 15: GND -> /Input Port 1/IO_C_36
- U309 pad 16: Vdrive -> /Input Port 1/IO_C_35
- U309 pad 17: /Input Port 1/IO_C_35 -> /Input Port 1/IO_C_34
- U309 pad 18: /Input Port 1/IO_C_34 -> /Input Port 1/IO_C_33
- U309 pad 19: /Input Port 1/IO_C_33 -> Vdrive
- U309 pad 2: /Input Port 1/IO_33 -> +1V5
- U309 pad 3: /Input Port 1/IO_34 -> /Input Port 1/IO_33
- U309 pad 4: /Input Port 1/IO_35 -> /Input Port 1/IO_34
- U309 pad 5: +1V5 -> /Input Port 1/IO_35
- U309 pad 6: /Input Port 1/OE -> /Input Port 1/IO_36
- U309 pad 7: /Input Port 1/IO_36 -> /Input Port 1/IO_37
- U309 pad 8: /Input Port 1/IO_37 -> /Input Port 1/IO_38
- U309 pad 9: /Input Port 1/IO_38 -> /Input Port 1/IO_39
- U310 pad 10: /Input Port 1/IO_47 -> /Input Port 1/OE
- U310 pad 11: /Input Port 1/IO_C_47 -> GND
- U310 pad 12: /Input Port 1/IO_C_46 -> /Input Port 1/IO_C_47
- U310 pad 13: /Input Port 1/IO_C_45 -> /Input Port 1/IO_C_46
- U310 pad 14: /Input Port 1/IO_C_44 -> /Input Port 1/IO_C_45
- U310 pad 15: GND -> /Input Port 1/IO_C_44
- U310 pad 16: Vdrive -> /Input Port 1/IO_C_43
- U310 pad 17: /Input Port 1/IO_C_43 -> /Input Port 1/IO_C_42
- U310 pad 18: /Input Port 1/IO_C_42 -> /Input Port 1/IO_C_41
- U310 pad 19: /Input Port 1/IO_C_41 -> Vdrive
- U310 pad 2: /Input Port 1/IO_41 -> +1V5
- U310 pad 3: /Input Port 1/IO_42 -> /Input Port 1/IO_41
- U310 pad 4: /Input Port 1/IO_43 -> /Input Port 1/IO_42
- U310 pad 5: +1V5 -> /Input Port 1/IO_43
- U310 pad 6: /Input Port 1/OE -> /Input Port 1/IO_44
- U310 pad 7: /Input Port 1/IO_44 -> /Input Port 1/IO_45
- U310 pad 8: /Input Port 1/IO_45 -> /Input Port 1/IO_46
- U310 pad 9: /Input Port 1/IO_46 -> /Input Port 1/IO_47
- U311 pad 10: /Input Port 1/IO_55 -> /Input Port 1/OE
- U311 pad 11: /Input Port 1/IO_C_55 -> GND
- U311 pad 12: /Input Port 1/IO_C_54 -> /Input Port 1/IO_C_55
- U311 pad 13: /Input Port 1/IO_C_53 -> /Input Port 1/IO_C_54
- U311 pad 14: /Input Port 1/IO_C_52 -> /Input Port 1/IO_C_53
- U311 pad 15: GND -> /Input Port 1/IO_C_52
- U311 pad 16: Vdrive -> /Input Port 1/IO_C_51
- U311 pad 17: /Input Port 1/IO_C_51 -> /Input Port 1/IO_C_50
- U311 pad 18: /Input Port 1/IO_C_50 -> /Input Port 1/IO_C_49
- U311 pad 19: /Input Port 1/IO_C_49 -> Vdrive
- U311 pad 2: /Input Port 1/IO_49 -> +1V5
- U311 pad 3: /Input Port 1/IO_50 -> /Input Port 1/IO_49
- U311 pad 4: /Input Port 1/IO_51 -> /Input Port 1/IO_50
- U311 pad 5: +1V5 -> /Input Port 1/IO_51
- U311 pad 6: /Input Port 1/OE -> /Input Port 1/IO_52
- U311 pad 7: /Input Port 1/IO_52 -> /Input Port 1/IO_53
- U311 pad 8: /Input Port 1/IO_53 -> /Input Port 1/IO_54
- U311 pad 9: /Input Port 1/IO_54 -> /Input Port 1/IO_55
- U312 pad 10: /Input Port 1/IO_63 -> /Input Port 1/OE
- U312 pad 11: /Input Port 1/IO_C_63 -> GND
- U312 pad 12: /Input Port 1/IO_C_62 -> /Input Port 1/IO_C_63
- U312 pad 13: /Input Port 1/IO_C_61 -> /Input Port 1/IO_C_62
- U312 pad 14: /Input Port 1/IO_C_60 -> /Input Port 1/IO_C_61
- U312 pad 15: GND -> /Input Port 1/IO_C_60
- U312 pad 16: Vdrive -> /Input Port 1/IO_C_59
- U312 pad 17: /Input Port 1/IO_C_59 -> /Input Port 1/IO_C_58
- U312 pad 18: /Input Port 1/IO_C_58 -> /Input Port 1/IO_C_57
- U312 pad 19: /Input Port 1/IO_C_57 -> Vdrive
- U312 pad 2: /Input Port 1/IO_57 -> +1V5
- U312 pad 3: /Input Port 1/IO_58 -> /Input Port 1/IO_57
- U312 pad 4: /Input Port 1/IO_59 -> /Input Port 1/IO_58
- U312 pad 5: +1V5 -> /Input Port 1/IO_59
- U312 pad 6: /Input Port 1/OE -> /Input Port 1/IO_60
- U312 pad 7: /Input Port 1/IO_60 -> /Input Port 1/IO_61
- U312 pad 8: /Input Port 1/IO_61 -> /Input Port 1/IO_62
- U312 pad 9: /Input Port 1/IO_62 -> /Input Port 1/IO_63
- U401 pad 10: /Input Port 2/IO_0 -> /Input Port 2/OE
- U401 pad 11: /Input Port 2/IO_C_0 -> GND
- U401 pad 12: /Input Port 2/IO_C_1 -> /Input Port 2/IO_C_0
- U401 pad 13: /Input Port 2/IO_C_2 -> /Input Port 2/IO_C_1
- U401 pad 14: /Input Port 2/IO_C_3 -> /Input Port 2/IO_C_2
- U401 pad 15: GND -> /Input Port 2/IO_C_3
- U401 pad 16: Vdrive -> /Input Port 2/IO_C_4
- U401 pad 17: /Input Port 2/IO_C_4 -> /Input Port 2/IO_C_5
- U401 pad 18: /Input Port 2/IO_C_5 -> /Input Port 2/IO_C_6
- U401 pad 19: /Input Port 2/IO_C_6 -> Vdrive
- U401 pad 2: /Input Port 2/IO_6 -> +1V5
- U401 pad 3: /Input Port 2/IO_5 -> /Input Port 2/IO_6
- U401 pad 4: /Input Port 2/IO_4 -> /Input Port 2/IO_5
- U401 pad 5: +1V5 -> /Input Port 2/IO_4
- U401 pad 6: /Input Port 2/OE -> /Input Port 2/IO_3
- U401 pad 7: /Input Port 2/IO_3 -> /Input Port 2/IO_2
- U401 pad 8: /Input Port 2/IO_2 -> /Input Port 2/IO_1
- U401 pad 9: /Input Port 2/IO_1 -> /Input Port 2/IO_0
- U403 pad 10: /Input Port 2/IO_8 -> /Input Port 2/OE
- U403 pad 11: /Input Port 2/IO_C_8 -> GND
- U403 pad 12: /Input Port 2/IO_C_9 -> /Input Port 2/IO_C_8
- U403 pad 13: /Input Port 2/IO_C_10 -> /Input Port 2/IO_C_9
- U403 pad 14: /Input Port 2/IO_C_11 -> /Input Port 2/IO_C_10
- U403 pad 15: GND -> /Input Port 2/IO_C_11
- U403 pad 16: Vdrive -> /Input Port 2/IO_C_12
- U403 pad 17: /Input Port 2/IO_C_12 -> /Input Port 2/IO_C_13
- U403 pad 18: /Input Port 2/IO_C_13 -> /Input Port 2/IO_C_14
- U403 pad 19: /Input Port 2/IO_C_14 -> Vdrive
- U403 pad 2: /Input Port 2/IO_14 -> +1V5
- U403 pad 3: /Input Port 2/IO_13 -> /Input Port 2/IO_14
- U403 pad 4: /Input Port 2/IO_12 -> /Input Port 2/IO_13
- U403 pad 5: +1V5 -> /Input Port 2/IO_12
- U403 pad 6: /Input Port 2/OE -> /Input Port 2/IO_11
- U403 pad 7: /Input Port 2/IO_11 -> /Input Port 2/IO_10
- U403 pad 8: /Input Port 2/IO_10 -> /Input Port 2/IO_9
- U403 pad 9: /Input Port 2/IO_9 -> /Input Port 2/IO_8
- U405 pad 10: /Input Port 2/IO_16 -> /Input Port 2/OE
- U405 pad 11: /Input Port 2/IO_C_16 -> GND
- U405 pad 12: /Input Port 2/IO_C_17 -> /Input Port 2/IO_C_16
- U405 pad 13: /Input Port 2/IO_C_18 -> /Input Port 2/IO_C_17
- U405 pad 14: /Input Port 2/IO_C_19 -> /Input Port 2/IO_C_18
- U405 pad 15: GND -> /Input Port 2/IO_C_19
- U405 pad 16: Vdrive -> /Input Port 2/IO_C_20
- U405 pad 17: /Input Port 2/IO_C_20 -> /Input Port 2/IO_C_21
- U405 pad 18: /Input Port 2/IO_C_21 -> /Input Port 2/IO_C_22
- U405 pad 19: /Input Port 2/IO_C_22 -> Vdrive
- U405 pad 2: /Input Port 2/IO_22 -> +1V5
- U405 pad 3: /Input Port 2/IO_21 -> /Input Port 2/IO_22
- U405 pad 4: /Input Port 2/IO_20 -> /Input Port 2/IO_21
- U405 pad 5: +1V5 -> /Input Port 2/IO_20
- U405 pad 6: /Input Port 2/OE -> /Input Port 2/IO_19
- U405 pad 7: /Input Port 2/IO_19 -> /Input Port 2/IO_18
- U405 pad 8: /Input Port 2/IO_18 -> /Input Port 2/IO_17
- U405 pad 9: /Input Port 2/IO_17 -> /Input Port 2/IO_16
- U407 pad 10: /Input Port 2/IO_24 -> /Input Port 2/OE
- U407 pad 11: /Input Port 2/IO_C_24 -> GND
- U407 pad 12: /Input Port 2/IO_C_25 -> /Input Port 2/IO_C_24
- U407 pad 13: /Input Port 2/IO_C_26 -> /Input Port 2/IO_C_25
- U407 pad 14: /Input Port 2/IO_C_27 -> /Input Port 2/IO_C_26
- U407 pad 15: GND -> /Input Port 2/IO_C_27
- U407 pad 16: Vdrive -> /Input Port 2/IO_C_28
- U407 pad 17: /Input Port 2/IO_C_28 -> /Input Port 2/IO_C_29
- U407 pad 18: /Input Port 2/IO_C_29 -> /Input Port 2/IO_C_30
- U407 pad 19: /Input Port 2/IO_C_30 -> Vdrive
- U407 pad 2: /Input Port 2/IO_30 -> +1V5
- U407 pad 3: /Input Port 2/IO_29 -> /Input Port 2/IO_30
- U407 pad 4: /Input Port 2/IO_28 -> /Input Port 2/IO_29
- U407 pad 5: +1V5 -> /Input Port 2/IO_28
- U407 pad 6: /Input Port 2/OE -> /Input Port 2/IO_27
- U407 pad 7: /Input Port 2/IO_27 -> /Input Port 2/IO_26
- U407 pad 8: /Input Port 2/IO_26 -> /Input Port 2/IO_25
- U407 pad 9: /Input Port 2/IO_25 -> /Input Port 2/IO_24
- U409 pad 10: /Input Port 2/IO_39 -> /Input Port 2/OE
- U409 pad 11: /Input Port 2/IO_C_39 -> GND
- U409 pad 12: /Input Port 2/IO_C_38 -> /Input Port 2/IO_C_39
- U409 pad 13: /Input Port 2/IO_C_37 -> /Input Port 2/IO_C_38
- U409 pad 14: /Input Port 2/IO_C_36 -> /Input Port 2/IO_C_37
- U409 pad 15: GND -> /Input Port 2/IO_C_36
- U409 pad 16: Vdrive -> /Input Port 2/IO_C_35
- U409 pad 17: /Input Port 2/IO_C_35 -> /Input Port 2/IO_C_34
- U409 pad 18: /Input Port 2/IO_C_34 -> /Input Port 2/IO_C_33
- U409 pad 19: /Input Port 2/IO_C_33 -> Vdrive
- U409 pad 2: /Input Port 2/IO_33 -> +1V5
- U409 pad 3: /Input Port 2/IO_34 -> /Input Port 2/IO_33
- U409 pad 4: /Input Port 2/IO_35 -> /Input Port 2/IO_34
- U409 pad 5: +1V5 -> /Input Port 2/IO_35
- U409 pad 6: /Input Port 2/OE -> /Input Port 2/IO_36
- U409 pad 7: /Input Port 2/IO_36 -> /Input Port 2/IO_37
- U409 pad 8: /Input Port 2/IO_37 -> /Input Port 2/IO_38
- U409 pad 9: /Input Port 2/IO_38 -> /Input Port 2/IO_39
- U410 pad 10: /Input Port 2/IO_47 -> /Input Port 2/OE
- U410 pad 11: /Input Port 2/IO_C_47 -> GND
- U410 pad 12: /Input Port 2/IO_C_46 -> /Input Port 2/IO_C_47
- U410 pad 13: /Input Port 2/IO_C_45 -> /Input Port 2/IO_C_46
- U410 pad 14: /Input Port 2/IO_C_44 -> /Input Port 2/IO_C_45
- U410 pad 15: GND -> /Input Port 2/IO_C_44
- U410 pad 16: Vdrive -> /Input Port 2/IO_C_43
- U410 pad 17: /Input Port 2/IO_C_43 -> /Input Port 2/IO_C_42
- U410 pad 18: /Input Port 2/IO_C_42 -> /Input Port 2/IO_C_41
- U410 pad 19: /Input Port 2/IO_C_41 -> Vdrive
- U410 pad 2: /Input Port 2/IO_41 -> +1V5
- U410 pad 3: /Input Port 2/IO_42 -> /Input Port 2/IO_41
- U410 pad 4: /Input Port 2/IO_43 -> /Input Port 2/IO_42
- U410 pad 5: +1V5 -> /Input Port 2/IO_43
- U410 pad 6: /Input Port 2/OE -> /Input Port 2/IO_44
- U410 pad 7: /Input Port 2/IO_44 -> /Input Port 2/IO_45
- U410 pad 8: /Input Port 2/IO_45 -> /Input Port 2/IO_46
- U410 pad 9: /Input Port 2/IO_46 -> /Input Port 2/IO_47
- U411 pad 10: /Input Port 2/IO_55 -> /Input Port 2/OE
- U411 pad 11: /Input Port 2/IO_C_55 -> GND
- U411 pad 12: /Input Port 2/IO_C_54 -> /Input Port 2/IO_C_55
- U411 pad 13: /Input Port 2/IO_C_53 -> /Input Port 2/IO_C_54
- U411 pad 14: /Input Port 2/IO_C_52 -> /Input Port 2/IO_C_53
- U411 pad 15: GND -> /Input Port 2/IO_C_52
- U411 pad 16: Vdrive -> /Input Port 2/IO_C_51
- U411 pad 17: /Input Port 2/IO_C_51 -> /Input Port 2/IO_C_50
- U411 pad 18: /Input Port 2/IO_C_50 -> /Input Port 2/IO_C_49
- U411 pad 19: /Input Port 2/IO_C_49 -> Vdrive
- U411 pad 2: /Input Port 2/IO_49 -> +1V5
- U411 pad 3: /Input Port 2/IO_50 -> /Input Port 2/IO_49
- U411 pad 4: /Input Port 2/IO_51 -> /Input Port 2/IO_50
- U411 pad 5: +1V5 -> /Input Port 2/IO_51
- U411 pad 6: /Input Port 2/OE -> /Input Port 2/IO_52
- U411 pad 7: /Input Port 2/IO_52 -> /Input Port 2/IO_53
- U411 pad 8: /Input Port 2/IO_53 -> /Input Port 2/IO_54
- U411 pad 9: /Input Port 2/IO_54 -> /Input Port 2/IO_55
- U412 pad 10: /Input Port 2/IO_63 -> /Input Port 2/OE
- U412 pad 11: /Input Port 2/IO_C_63 -> GND
- U412 pad 12: /Input Port 2/IO_C_62 -> /Input Port 2/IO_C_63
- U412 pad 13: /Input Port 2/IO_C_61 -> /Input Port 2/IO_C_62
- U412 pad 14: /Input Port 2/IO_C_60 -> /Input Port 2/IO_C_61
- U412 pad 15: GND -> /Input Port 2/IO_C_60
- U412 pad 16: Vdrive -> /Input Port 2/IO_C_59
- U412 pad 17: /Input Port 2/IO_C_59 -> /Input Port 2/IO_C_58
- U412 pad 18: /Input Port 2/IO_C_58 -> /Input Port 2/IO_C_57
- U412 pad 19: /Input Port 2/IO_C_57 -> Vdrive
- U412 pad 2: /Input Port 2/IO_57 -> +1V5
- U412 pad 3: /Input Port 2/IO_58 -> /Input Port 2/IO_57
- U412 pad 4: /Input Port 2/IO_59 -> /Input Port 2/IO_58
- U412 pad 5: +1V5 -> /Input Port 2/IO_59
- U412 pad 6: /Input Port 2/OE -> /Input Port 2/IO_60
- U412 pad 7: /Input Port 2/IO_60 -> /Input Port 2/IO_61
- U412 pad 8: /Input Port 2/IO_61 -> /Input Port 2/IO_62
- U412 pad 9: /Input Port 2/IO_62 -> /Input Port 2/IO_63
- U501 pad 10: /Input Port 3/IO_0 -> /Input Port 3/OE
- U501 pad 11: /Input Port 3/IO_C_0 -> GND
- U501 pad 12: /Input Port 3/IO_C_1 -> /Input Port 3/IO_C_0
- U501 pad 13: /Input Port 3/IO_C_2 -> /Input Port 3/IO_C_1
- U501 pad 14: /Input Port 3/IO_C_3 -> /Input Port 3/IO_C_2
- U501 pad 15: GND -> /Input Port 3/IO_C_3
- U501 pad 16: Vdrive -> /Input Port 3/IO_C_4
- U501 pad 17: /Input Port 3/IO_C_4 -> /Input Port 3/IO_C_5
- U501 pad 18: /Input Port 3/IO_C_5 -> /Input Port 3/IO_C_6
- U501 pad 19: /Input Port 3/IO_C_6 -> Vdrive
- U501 pad 2: /Input Port 3/IO_6 -> +1V5
- U501 pad 3: /Input Port 3/IO_5 -> /Input Port 3/IO_6
- U501 pad 4: /Input Port 3/IO_4 -> /Input Port 3/IO_5
- U501 pad 5: +1V5 -> /Input Port 3/IO_4
- U501 pad 6: /Input Port 3/OE -> /Input Port 3/IO_3
- U501 pad 7: /Input Port 3/IO_3 -> /Input Port 3/IO_2
- U501 pad 8: /Input Port 3/IO_2 -> /Input Port 3/IO_1
- U501 pad 9: /Input Port 3/IO_1 -> /Input Port 3/IO_0
- U503 pad 10: /Input Port 3/IO_8 -> /Input Port 3/OE
- U503 pad 11: /Input Port 3/IO_C_8 -> GND
- U503 pad 12: /Input Port 3/IO_C_9 -> /Input Port 3/IO_C_8
- U503 pad 13: /Input Port 3/IO_C_10 -> /Input Port 3/IO_C_9
- U503 pad 14: /Input Port 3/IO_C_11 -> /Input Port 3/IO_C_10
- U503 pad 15: GND -> /Input Port 3/IO_C_11
- U503 pad 16: Vdrive -> /Input Port 3/IO_C_12
- U503 pad 17: /Input Port 3/IO_C_12 -> /Input Port 3/IO_C_13
- U503 pad 18: /Input Port 3/IO_C_13 -> /Input Port 3/IO_C_14
- U503 pad 19: /Input Port 3/IO_C_14 -> Vdrive
- U503 pad 2: /Input Port 3/IO_14 -> +1V5
- U503 pad 3: /Input Port 3/IO_13 -> /Input Port 3/IO_14
- U503 pad 4: /Input Port 3/IO_12 -> /Input Port 3/IO_13
- U503 pad 5: +1V5 -> /Input Port 3/IO_12
- U503 pad 6: /Input Port 3/OE -> /Input Port 3/IO_11
- U503 pad 7: /Input Port 3/IO_11 -> /Input Port 3/IO_10
- U503 pad 8: /Input Port 3/IO_10 -> /Input Port 3/IO_9
- U503 pad 9: /Input Port 3/IO_9 -> /Input Port 3/IO_8
- U505 pad 10: /Input Port 3/IO_16 -> /Input Port 3/OE
- U505 pad 11: /Input Port 3/IO_C_16 -> GND
- U505 pad 12: /Input Port 3/IO_C_17 -> /Input Port 3/IO_C_16
- U505 pad 13: /Input Port 3/IO_C_18 -> /Input Port 3/IO_C_17
- U505 pad 14: /Input Port 3/IO_C_19 -> /Input Port 3/IO_C_18
- U505 pad 15: GND -> /Input Port 3/IO_C_19
- U505 pad 16: Vdrive -> /Input Port 3/IO_C_20
- U505 pad 17: /Input Port 3/IO_C_20 -> /Input Port 3/IO_C_21
- U505 pad 18: /Input Port 3/IO_C_21 -> /Input Port 3/IO_C_22
- U505 pad 19: /Input Port 3/IO_C_22 -> Vdrive
- U505 pad 2: /Input Port 3/IO_22 -> +1V5
- U505 pad 3: /Input Port 3/IO_21 -> /Input Port 3/IO_22
- U505 pad 4: /Input Port 3/IO_20 -> /Input Port 3/IO_21
- U505 pad 5: +1V5 -> /Input Port 3/IO_20
- U505 pad 6: /Input Port 3/OE -> /Input Port 3/IO_19
- U505 pad 7: /Input Port 3/IO_19 -> /Input Port 3/IO_18
- U505 pad 8: /Input Port 3/IO_18 -> /Input Port 3/IO_17
- U505 pad 9: /Input Port 3/IO_17 -> /Input Port 3/IO_16
- U507 pad 10: /Input Port 3/IO_24 -> /Input Port 3/OE
- U507 pad 11: /Input Port 3/IO_C_24 -> GND
- U507 pad 12: /Input Port 3/IO_C_25 -> /Input Port 3/IO_C_24
- U507 pad 13: /Input Port 3/IO_C_26 -> /Input Port 3/IO_C_25
- U507 pad 14: /Input Port 3/IO_C_27 -> /Input Port 3/IO_C_26
- U507 pad 15: GND -> /Input Port 3/IO_C_27
- U507 pad 16: Vdrive -> /Input Port 3/IO_C_28
- U507 pad 17: /Input Port 3/IO_C_28 -> /Input Port 3/IO_C_29
- U507 pad 18: /Input Port 3/IO_C_29 -> /Input Port 3/IO_C_30
- U507 pad 19: /Input Port 3/IO_C_30 -> Vdrive
- U507 pad 2: /Input Port 3/IO_30 -> +1V5
- U507 pad 3: /Input Port 3/IO_29 -> /Input Port 3/IO_30
- U507 pad 4: /Input Port 3/IO_28 -> /Input Port 3/IO_29
- U507 pad 5: +1V5 -> /Input Port 3/IO_28
- U507 pad 6: /Input Port 3/OE -> /Input Port 3/IO_27
- U507 pad 7: /Input Port 3/IO_27 -> /Input Port 3/IO_26
- U507 pad 8: /Input Port 3/IO_26 -> /Input Port 3/IO_25
- U507 pad 9: /Input Port 3/IO_25 -> /Input Port 3/IO_24
- U509 pad 10: /Input Port 3/IO_39 -> /Input Port 3/OE
- U509 pad 11: /Input Port 3/IO_C_39 -> GND
- U509 pad 12: /Input Port 3/IO_C_38 -> /Input Port 3/IO_C_39
- U509 pad 13: /Input Port 3/IO_C_37 -> /Input Port 3/IO_C_38
- U509 pad 14: /Input Port 3/IO_C_36 -> /Input Port 3/IO_C_37
- U509 pad 15: GND -> /Input Port 3/IO_C_36
- U509 pad 16: Vdrive -> /Input Port 3/IO_C_35
- U509 pad 17: /Input Port 3/IO_C_35 -> /Input Port 3/IO_C_34
- U509 pad 18: /Input Port 3/IO_C_34 -> /Input Port 3/IO_C_33
- U509 pad 19: /Input Port 3/IO_C_33 -> Vdrive
- U509 pad 2: /Input Port 3/IO_33 -> +1V5
- U509 pad 3: /Input Port 3/IO_34 -> /Input Port 3/IO_33
- U509 pad 4: /Input Port 3/IO_35 -> /Input Port 3/IO_34
- U509 pad 5: +1V5 -> /Input Port 3/IO_35
- U509 pad 6: /Input Port 3/OE -> /Input Port 3/IO_36
- U509 pad 7: /Input Port 3/IO_36 -> /Input Port 3/IO_37
- U509 pad 8: /Input Port 3/IO_37 -> /Input Port 3/IO_38
- U509 pad 9: /Input Port 3/IO_38 -> /Input Port 3/IO_39
- U510 pad 10: /Input Port 3/IO_47 -> /Input Port 3/OE
- U510 pad 11: /Input Port 3/IO_C_47 -> GND
- U510 pad 12: /Input Port 3/IO_C_46 -> /Input Port 3/IO_C_47
- U510 pad 13: /Input Port 3/IO_C_45 -> /Input Port 3/IO_C_46
- U510 pad 14: /Input Port 3/IO_C_44 -> /Input Port 3/IO_C_45
- U510 pad 15: GND -> /Input Port 3/IO_C_44
- U510 pad 16: Vdrive -> /Input Port 3/IO_C_43
- U510 pad 17: /Input Port 3/IO_C_43 -> /Input Port 3/IO_C_42
- U510 pad 18: /Input Port 3/IO_C_42 -> /Input Port 3/IO_C_41
- U510 pad 19: /Input Port 3/IO_C_41 -> Vdrive
- U510 pad 2: /Input Port 3/IO_41 -> +1V5
- U510 pad 3: /Input Port 3/IO_42 -> /Input Port 3/IO_41
- U510 pad 4: /Input Port 3/IO_43 -> /Input Port 3/IO_42
- U510 pad 5: +1V5 -> /Input Port 3/IO_43
- U510 pad 6: /Input Port 3/OE -> /Input Port 3/IO_44
- U510 pad 7: /Input Port 3/IO_44 -> /Input Port 3/IO_45
- U510 pad 8: /Input Port 3/IO_45 -> /Input Port 3/IO_46
- U510 pad 9: /Input Port 3/IO_46 -> /Input Port 3/IO_47
- U511 pad 10: /Input Port 3/IO_55 -> /Input Port 3/OE
- U511 pad 11: /Input Port 3/IO_C_55 -> GND
- U511 pad 12: /Input Port 3/IO_C_54 -> /Input Port 3/IO_C_55
- U511 pad 13: /Input Port 3/IO_C_53 -> /Input Port 3/IO_C_54
- U511 pad 14: /Input Port 3/IO_C_52 -> /Input Port 3/IO_C_53
- U511 pad 15: GND -> /Input Port 3/IO_C_52
- U511 pad 16: Vdrive -> /Input Port 3/IO_C_51
- U511 pad 17: /Input Port 3/IO_C_51 -> /Input Port 3/IO_C_50
- U511 pad 18: /Input Port 3/IO_C_50 -> /Input Port 3/IO_C_49
- U511 pad 19: /Input Port 3/IO_C_49 -> Vdrive
- U511 pad 2: /Input Port 3/IO_49 -> +1V5
- U511 pad 3: /Input Port 3/IO_50 -> /Input Port 3/IO_49
- U511 pad 4: /Input Port 3/IO_51 -> /Input Port 3/IO_50
- U511 pad 5: +1V5 -> /Input Port 3/IO_51
- U511 pad 6: /Input Port 3/OE -> /Input Port 3/IO_52
- U511 pad 7: /Input Port 3/IO_52 -> /Input Port 3/IO_53
- U511 pad 8: /Input Port 3/IO_53 -> /Input Port 3/IO_54
- U511 pad 9: /Input Port 3/IO_54 -> /Input Port 3/IO_55
- U512 pad 10: /Input Port 3/IO_63 -> /Input Port 3/OE
- U512 pad 11: /Input Port 3/IO_C_63 -> GND
- U512 pad 12: /Input Port 3/IO_C_62 -> /Input Port 3/IO_C_63
- U512 pad 13: /Input Port 3/IO_C_61 -> /Input Port 3/IO_C_62
- U512 pad 14: /Input Port 3/IO_C_60 -> /Input Port 3/IO_C_61
- U512 pad 15: GND -> /Input Port 3/IO_C_60
- U512 pad 16: Vdrive -> /Input Port 3/IO_C_59
- U512 pad 17: /Input Port 3/IO_C_59 -> /Input Port 3/IO_C_58
- U512 pad 18: /Input Port 3/IO_C_58 -> /Input Port 3/IO_C_57
- U512 pad 19: /Input Port 3/IO_C_57 -> Vdrive
- U512 pad 2: /Input Port 3/IO_57 -> +1V5
- U512 pad 3: /Input Port 3/IO_58 -> /Input Port 3/IO_57
- U512 pad 4: /Input Port 3/IO_59 -> /Input Port 3/IO_58
- U512 pad 5: +1V5 -> /Input Port 3/IO_59
- U512 pad 6: /Input Port 3/OE -> /Input Port 3/IO_60
- U512 pad 7: /Input Port 3/IO_60 -> /Input Port 3/IO_61
- U512 pad 8: /Input Port 3/IO_61 -> /Input Port 3/IO_62
- U512 pad 9: /Input Port 3/IO_62 -> /Input Port 3/IO_63
- U601 pad 10: /Input Port 4/IO_0 -> /Input Port 4/OE
- U601 pad 11: /Input Port 4/IO_C_0 -> GND
- U601 pad 12: /Input Port 4/IO_C_1 -> /Input Port 4/IO_C_0
- U601 pad 13: /Input Port 4/IO_C_2 -> /Input Port 4/IO_C_1
- U601 pad 14: /Input Port 4/IO_C_3 -> /Input Port 4/IO_C_2
- U601 pad 15: GND -> /Input Port 4/IO_C_3
- U601 pad 16: Vdrive -> /Input Port 4/IO_C_4
- U601 pad 17: /Input Port 4/IO_C_4 -> /Input Port 4/IO_C_5
- U601 pad 18: /Input Port 4/IO_C_5 -> /Input Port 4/IO_C_6
- U601 pad 19: /Input Port 4/IO_C_6 -> Vdrive
- U601 pad 2: /Input Port 4/IO_6 -> +1V5
- U601 pad 3: /Input Port 4/IO_5 -> /Input Port 4/IO_6
- U601 pad 4: /Input Port 4/IO_4 -> /Input Port 4/IO_5
- U601 pad 5: +1V5 -> /Input Port 4/IO_4
- U601 pad 6: /Input Port 4/OE -> /Input Port 4/IO_3
- U601 pad 7: /Input Port 4/IO_3 -> /Input Port 4/IO_2
- U601 pad 8: /Input Port 4/IO_2 -> /Input Port 4/IO_1
- U601 pad 9: /Input Port 4/IO_1 -> /Input Port 4/IO_0
- U603 pad 10: /Input Port 4/IO_8 -> /Input Port 4/OE
- U603 pad 11: /Input Port 4/IO_C_8 -> GND
- U603 pad 12: /Input Port 4/IO_C_9 -> /Input Port 4/IO_C_8
- U603 pad 13: /Input Port 4/IO_C_10 -> /Input Port 4/IO_C_9
- U603 pad 14: /Input Port 4/IO_C_11 -> /Input Port 4/IO_C_10
- U603 pad 15: GND -> /Input Port 4/IO_C_11
- U603 pad 16: Vdrive -> /Input Port 4/IO_C_12
- U603 pad 17: /Input Port 4/IO_C_12 -> /Input Port 4/IO_C_13
- U603 pad 18: /Input Port 4/IO_C_13 -> /Input Port 4/IO_C_14
- U603 pad 19: /Input Port 4/IO_C_14 -> Vdrive
- U603 pad 2: /Input Port 4/IO_14 -> +1V5
- U603 pad 3: /Input Port 4/IO_13 -> /Input Port 4/IO_14
- U603 pad 4: /Input Port 4/IO_12 -> /Input Port 4/IO_13
- U603 pad 5: +1V5 -> /Input Port 4/IO_12
- U603 pad 6: /Input Port 4/OE -> /Input Port 4/IO_11
- U603 pad 7: /Input Port 4/IO_11 -> /Input Port 4/IO_10
- U603 pad 8: /Input Port 4/IO_10 -> /Input Port 4/IO_9
- U603 pad 9: /Input Port 4/IO_9 -> /Input Port 4/IO_8
- U605 pad 10: /Input Port 4/IO_16 -> /Input Port 4/OE
- U605 pad 11: /Input Port 4/IO_C_16 -> GND
- U605 pad 12: /Input Port 4/IO_C_17 -> /Input Port 4/IO_C_16
- U605 pad 13: /Input Port 4/IO_C_18 -> /Input Port 4/IO_C_17
- U605 pad 14: /Input Port 4/IO_C_19 -> /Input Port 4/IO_C_18
- U605 pad 15: GND -> /Input Port 4/IO_C_19
- U605 pad 16: Vdrive -> /Input Port 4/IO_C_20
- U605 pad 17: /Input Port 4/IO_C_20 -> /Input Port 4/IO_C_21
- U605 pad 18: /Input Port 4/IO_C_21 -> /Input Port 4/IO_C_22
- U605 pad 19: /Input Port 4/IO_C_22 -> Vdrive
- U605 pad 2: /Input Port 4/IO_22 -> +1V5
- U605 pad 3: /Input Port 4/IO_21 -> /Input Port 4/IO_22
- U605 pad 4: /Input Port 4/IO_20 -> /Input Port 4/IO_21
- U605 pad 5: +1V5 -> /Input Port 4/IO_20
- U605 pad 6: /Input Port 4/OE -> /Input Port 4/IO_19
- U605 pad 7: /Input Port 4/IO_19 -> /Input Port 4/IO_18
- U605 pad 8: /Input Port 4/IO_18 -> /Input Port 4/IO_17
- U605 pad 9: /Input Port 4/IO_17 -> /Input Port 4/IO_16
- U607 pad 10: /Input Port 4/IO_24 -> /Input Port 4/OE
- U607 pad 11: /Input Port 4/IO_C_24 -> GND
- U607 pad 12: /Input Port 4/IO_C_25 -> /Input Port 4/IO_C_24
- U607 pad 13: /Input Port 4/IO_C_26 -> /Input Port 4/IO_C_25
- U607 pad 14: /Input Port 4/IO_C_27 -> /Input Port 4/IO_C_26
- U607 pad 15: GND -> /Input Port 4/IO_C_27
- U607 pad 16: Vdrive -> /Input Port 4/IO_C_28
- U607 pad 17: /Input Port 4/IO_C_28 -> /Input Port 4/IO_C_29
- U607 pad 18: /Input Port 4/IO_C_29 -> /Input Port 4/IO_C_30
- U607 pad 19: /Input Port 4/IO_C_30 -> Vdrive
- U607 pad 2: /Input Port 4/IO_30 -> +1V5
- U607 pad 3: /Input Port 4/IO_29 -> /Input Port 4/IO_30
- U607 pad 4: /Input Port 4/IO_28 -> /Input Port 4/IO_29
- U607 pad 5: +1V5 -> /Input Port 4/IO_28
- U607 pad 6: /Input Port 4/OE -> /Input Port 4/IO_27
- U607 pad 7: /Input Port 4/IO_27 -> /Input Port 4/IO_26
- U607 pad 8: /Input Port 4/IO_26 -> /Input Port 4/IO_25
- U607 pad 9: /Input Port 4/IO_25 -> /Input Port 4/IO_24
- U609 pad 10: /Input Port 4/IO_39 -> /Input Port 4/OE
- U609 pad 11: /Input Port 4/IO_C_39 -> GND
- U609 pad 12: /Input Port 4/IO_C_38 -> /Input Port 4/IO_C_39
- U609 pad 13: /Input Port 4/IO_C_37 -> /Input Port 4/IO_C_38
- U609 pad 14: /Input Port 4/IO_C_36 -> /Input Port 4/IO_C_37
- U609 pad 15: GND -> /Input Port 4/IO_C_36
- U609 pad 16: Vdrive -> /Input Port 4/IO_C_35
- U609 pad 17: /Input Port 4/IO_C_35 -> /Input Port 4/IO_C_34
- U609 pad 18: /Input Port 4/IO_C_34 -> /Input Port 4/IO_C_33
- U609 pad 19: /Input Port 4/IO_C_33 -> Vdrive
- U609 pad 2: /Input Port 4/IO_33 -> +1V5
- U609 pad 3: /Input Port 4/IO_34 -> /Input Port 4/IO_33
- U609 pad 4: /Input Port 4/IO_35 -> /Input Port 4/IO_34
- U609 pad 5: +1V5 -> /Input Port 4/IO_35
- U609 pad 6: /Input Port 4/OE -> /Input Port 4/IO_36
- U609 pad 7: /Input Port 4/IO_36 -> /Input Port 4/IO_37
- U609 pad 8: /Input Port 4/IO_37 -> /Input Port 4/IO_38
- U609 pad 9: /Input Port 4/IO_38 -> /Input Port 4/IO_39
- U610 pad 10: /Input Port 4/IO_47 -> /Input Port 4/OE
- U610 pad 11: /Input Port 4/IO_C_47 -> GND
- U610 pad 12: /Input Port 4/IO_C_46 -> /Input Port 4/IO_C_47
- U610 pad 13: /Input Port 4/IO_C_45 -> /Input Port 4/IO_C_46
- U610 pad 14: /Input Port 4/IO_C_44 -> /Input Port 4/IO_C_45
- U610 pad 15: GND -> /Input Port 4/IO_C_44
- U610 pad 16: Vdrive -> /Input Port 4/IO_C_43
- U610 pad 17: /Input Port 4/IO_C_43 -> /Input Port 4/IO_C_42
- U610 pad 18: /Input Port 4/IO_C_42 -> /Input Port 4/IO_C_41
- U610 pad 19: /Input Port 4/IO_C_41 -> Vdrive
- U610 pad 2: /Input Port 4/IO_41 -> +1V5
- U610 pad 3: /Input Port 4/IO_42 -> /Input Port 4/IO_41
- U610 pad 4: /Input Port 4/IO_43 -> /Input Port 4/IO_42
- U610 pad 5: +1V5 -> /Input Port 4/IO_43
- U610 pad 6: /Input Port 4/OE -> /Input Port 4/IO_44
- U610 pad 7: /Input Port 4/IO_44 -> /Input Port 4/IO_45
- U610 pad 8: /Input Port 4/IO_45 -> /Input Port 4/IO_46
- U610 pad 9: /Input Port 4/IO_46 -> /Input Port 4/IO_47
- U611 pad 10: /Input Port 4/IO_55 -> /Input Port 4/OE
- U611 pad 11: /Input Port 4/IO_C_55 -> GND
- U611 pad 12: /Input Port 4/IO_C_54 -> /Input Port 4/IO_C_55
- U611 pad 13: /Input Port 4/IO_C_53 -> /Input Port 4/IO_C_54
- U611 pad 14: /Input Port 4/IO_C_52 -> /Input Port 4/IO_C_53
- U611 pad 15: GND -> /Input Port 4/IO_C_52
- U611 pad 16: Vdrive -> /Input Port 4/IO_C_51
- U611 pad 17: /Input Port 4/IO_C_51 -> /Input Port 4/IO_C_50
- U611 pad 18: /Input Port 4/IO_C_50 -> /Input Port 4/IO_C_49
- U611 pad 19: /Input Port 4/IO_C_49 -> Vdrive
- U611 pad 2: /Input Port 4/IO_49 -> +1V5
- U611 pad 3: /Input Port 4/IO_50 -> /Input Port 4/IO_49
- U611 pad 4: /Input Port 4/IO_51 -> /Input Port 4/IO_50
- U611 pad 5: +1V5 -> /Input Port 4/IO_51
- U611 pad 6: /Input Port 4/OE -> /Input Port 4/IO_52
- U611 pad 7: /Input Port 4/IO_52 -> /Input Port 4/IO_53
- U611 pad 8: /Input Port 4/IO_53 -> /Input Port 4/IO_54
- U611 pad 9: /Input Port 4/IO_54 -> /Input Port 4/IO_55
- U612 pad 10: /Input Port 4/IO_63 -> /Input Port 4/OE
- U612 pad 11: /Input Port 4/IO_C_63 -> GND
- U612 pad 12: /Input Port 4/IO_C_62 -> /Input Port 4/IO_C_63
- U612 pad 13: /Input Port 4/IO_C_61 -> /Input Port 4/IO_C_62
- U612 pad 14: /Input Port 4/IO_C_60 -> /Input Port 4/IO_C_61
- U612 pad 15: GND -> /Input Port 4/IO_C_60
- U612 pad 16: Vdrive -> /Input Port 4/IO_C_59
- U612 pad 17: /Input Port 4/IO_C_59 -> /Input Port 4/IO_C_58
- U612 pad 18: /Input Port 4/IO_C_58 -> /Input Port 4/IO_C_57
- U612 pad 19: /Input Port 4/IO_C_57 -> Vdrive
- U612 pad 2: /Input Port 4/IO_57 -> +1V5
- U612 pad 3: /Input Port 4/IO_58 -> /Input Port 4/IO_57
- U612 pad 4: /Input Port 4/IO_59 -> /Input Port 4/IO_58
- U612 pad 5: +1V5 -> /Input Port 4/IO_59
- U612 pad 6: /Input Port 4/OE -> /Input Port 4/IO_60
- U612 pad 7: /Input Port 4/IO_60 -> /Input Port 4/IO_61
- U612 pad 8: /Input Port 4/IO_61 -> /Input Port 4/IO_62
- U612 pad 9: /Input Port 4/IO_62 -> /Input Port 4/IO_63
Routing:
- net Vdrive: track 38.8 -> 4.67 mm, vias 32 -> 0
- net GND: track 39.1 -> 5.05 mm, vias 73 -> 41
- net +1V5: track 32.9 -> 0.61 mm, vias 32 -> 0
- net /Power/FB_3V3: track 7.61 -> 3.80 mm
- net Net-(U205-SW): track 2.35 -> 0.00 mm
Other:
- board text added: "VORTESSENCE"
- board text removed: "ETHER"
