File: hardware/ether.kicad_sch (KiCad schematic)
At the start: 4 parts, among them U101 ECP5U_85_CABGA756, U102 TXB0108DQSR, U103 TCA9535RTWR, U104 TCA9535RTWR

Commit message: Save
Connections:
- net PORT77_1: now reaches U101.AG1 (PB4A/+/D7/IO7)
- net PORT77_2: now reaches U101.AH1 (PB4B/-/D6/IO6)
- net PORT77_3: now reaches U101.AJ1 (PB6A/+/D5/MISO2/IO5)
- net PORT78_3: now reaches U101.AJ2 (PB11A/+/D1/MISO/IO1)
- net PORT77_4: now reaches U101.AK1 (PB6B/-/D4/MOSI2/IO4)
- net PORT78_4: now reaches U101.AK2 (PB11B/-/D0/MOSI/IO0)
- net PORT78_1: now reaches U101.AL1 (PB9A/+/D3/IO3)
- net PORT78_2: now reaches U101.AM2 (PB9B/-/D2/IO2)
Changed lines of the file:
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@@
+    (effects (font (size 1.27 1.27)) (justify right bottom))
+  )
+  (label "PORT77_1" (at 444.5 58.42 180) (fields_autoplaced)
     (effects (font (size 1.27 1.27)) (justify right bottom))
   )
@@
     (effects (font (size 1.27 1.27)) (justify right bottom))
   )
+  (label "PORT78_4" (at 444.5 76.2 180) (fields_autoplaced)
+    (effects (font (size 1.27 1.27)) (justify right bottom))
+  )
   (label "PORT6" (at 313.69 58.42 180) (fields_autoplaced)
     (effects (font (size 1.27 1.27)) (justify right bottom))
@@
     (effects (font (size 1.27 1.27)) (justify right bottom))
   )
+  (label "PORT77_2" (at 444.5 60.96 180) (fields_autoplaced)
+    (effects (font (size 1.27 1.27)) (justify right bottom))
+  )
   (label "PORT2" (at 107.95 104.14 180) (fields_autoplaced)
     (effects (font (size 1.27 1.27)) (justify right bottom))
@@
     (effects (font (size 1.27 1.27)) (justify right bottom))
   )
+  (label "PORT77_3" (at 444.5 63.5 180) (fields_autoplaced)
+    (effects (font (size 1.27 1.27)) (justify right bottom))
+  )
   (label "PORT2" (at 107.95 101.6 180) (fields_autoplaced)
     (effects (font (size 1.27 1.27)) (justify right bottom))
@@
     (effects (font (size 1.27 1.27)) (justify right bottom))
   )
+  (label "PORT78_3" (at 444.5 73.66 180) (fields_autoplaced)
+    (effects (font (size 1.27 1.27)) (justify right bottom))
+  )
   (label "PORT3" (at 157.48 119.38 180) (fields_autoplaced)
     (effects (font (size 1.27 1.27)) (justify right bottom))
@@
     (effects (font (size 1.27 1.27)) (justify right bottom))
   )
+  (label "PORT78_2" (at 444.5 71.12 180) (fields_autoplaced)
+    (effects (font (size 1.27 1.27)) (justify right bottom))
+  )
   (label "PORT3" (at 157.48 71.12 180) (fields_autoplaced)
     (effects (font (size 1.27 1.27)) (justify right bottom))
@@
     (effects (font (size 1.27 1.27)) (justify right bottom))
   )
+  (label "PORT78_1" (at 444.5 68.58 180) (fields_autoplaced)
+    (effects (font (size 1.27 1.27)) (justify right bottom))
+  )
   (label "PORT4" (at 215.9 147.32 180) (fields_autoplaced)
     (effects (font (size 1.27 1.27)) (justify right bottom))
@@
     (effects (font (size 1.27 1.27)) (justify right bottom))
   )
+  (label "PORT77_4" (at 444.5 66.04 180) (fields_autoplaced)
+    (effects (font (size 1.27 1.27)) (justify right bottom))
+  )
