File: hardware/ether.kicad_sch (KiCad schematic)
At the start: 3 parts, among them J101 SS-74500-022, J102 SS-74500-022, U101 ECP5UM_85_CABGA756

Commit message: Save
Parts:
- removed J101, J102: SS-74500-022, BEL_SS-74500-022, symbol connectors:SS-74500-022
- removed U101: ECP5UM_85_CABGA756, Package_BGA:Lattice_caBGA-756_27.0x27.0mm_Layout32x32_P0.8mm, symbol Lattice_ECP5_FPGA:ECP5UM_85_CABGA756
- added U101: ECP5U_85_CABGA756, Package_BGA:Lattice_caBGA-756_27.0x27.0mm_Layout32x32_P0.8mm, symbol Lattice_ECP5_FPGA:ECP5U_85_CABGA756
- added U102: TXB0108DQSR, Package_SON:USON-20_2x4mm_P0.4mm, symbol Logic_LevelTranslator:TXB0108DQSR
- added U103, U104: TCA9535RTWR, Package_DFN_QFN:WQFN-24-1EP_4x4mm_P0.5mm_EP2.45x2.45mm, symbol Interface_Expansion:TCA9535RTWR
Connections:
- new net: U101.AA10 (VCCIO6[4]), U101.U10 (VCCIO6[4]), U101.V10 (VCCIO6[4]), U101.W10 (VCCIO6[4])
- new net: U101.M23 (VCCIO2[4]), U101.P23 (VCCIO2[4]), U101.R23 (VCCIO2[4]), U101.T23 (VCCIO2[4])
- new net: U101.AB23 (VCCIO4[2]), U101.AC23 (VCCIO4[2])
- new net: U101.K17 (VCCIO1[4]), U101.K18 (VCCIO1[4]), U101.K19 (VCCIO1[4]), U101.K21 (VCCIO1[4])
- new net: U101.AA23 (VCCIO3[4]), U101.U23 (VCCIO3[4]), U101.V23 (VCCIO3[4]), U101.W23 (VCCIO3[4])
- new net: U101.K12 (VCCIO0[4]), U101.K14 (VCCIO0[4]), U101.K15 (VCCIO0[4]), U101.K16 (VCCIO0[4])
- new net: U101.AB10 (VCCIO8[2]), U101.AC10 (VCCIO8[2])
- new net: U101.M10 (VCCIO7[4]), U101.P10 (VCCIO7[4]), U101.R10 (VCCIO7[4]), U101.T10 (VCCIO7[4])
- new net PORT1: U101.A10 (PT31B/-), U101.A11 (PT38B/-), U101.A13 (PT42B/-), U101.A14 (PT49B/-), U101.A15 (PT54B/-), U101.A16 (PT60B/-/GR_PCLK0_0), U101.A17 (PT63A/+/PCLKT0_1), U101.A2 (PT6A/+), U101.A3 (PT6B/-), U101.A4 (PT9A/+), U101.A5 (PT9B/-), U101.A7 (PT13B/-), U101.A8 (PT20B/-), U101.A9 (PT24B/-), U101.B10 (PT31A/+), U101.B11 (PT38A/+), U101.B14 (PT49A/+), U101.B16 (PT60A/+/GR_PCLK0_1), U101.B17 (PT63B/-/PCLKC0_1), U101.B3 (PT4A/+/ULC_GPLL1T_IN), U101.B4 (PT4B/-/ULC_GPLL1C_IN), U101.B7 (PT13A/+), U101.B8 (PT20A/+), U101.C10 (PT29B/-), U101.C11 (PT36B/-), U101.C13 (PT42A/+), U101.C14 (PT47B/-), U101.C15 (PT54A/+), U101.C16 (PT58B/-), U101.C17 (PT65A/+/PCLKT0_0), U101.C7 (PT11B/-), U101.C8 (PT18B/-), U101.C9 (PT24A/+), U101.D10 (PT29A/+), U101.D11 (PT36A/+), U101.D13 (PT40B/-), U101.D14 (PT47A/+), U101.D15 (PT51B/-), U101.D16 (PT58A/+), U101.D17 (PT65B/-/PCLKC0_0), U101.D7 (PT11A/+), U101.D8 (PT18A/+), U101.D9 (PT22B/-), U101.E10 (PT27B/-), U101.E11 (PT33B/-), U101.E14 (PT45B/-), U101.E16 (PT56B/-), U101.E8 (PT15B/-), U101.F10 (PT27A/+), U101.F11 (PT33A/+), U101.F13 (PT40A/+), U101.F14 (PT45A/+), U101.F15 (PT51A/+), U101.F16 (PT56A/+), U101.F8 (PT15A/+), U101.F9 (PT22A/+)
- new net PORT2: U101.A18 (PT71A/+/PCLKT1_0), U101.A19 (PT76A/+), U101.A20 (PT83A/+), U101.A22 (PT87A/+), U101.A23 (PT94A/+), U101.A24 (PT101A/+), U101.A25 (PT105A/+), U101.A26 (PT112A/+), U101.A28 (PT116A/+), U101.A29 (PT116B/-), U101.A30 (PT119A/+), U101.A31 (PT119B/-), U101.B19 (PT76B/-), U101.B22 (PT87B/-), U101.B23 (PT94B/-), U101.B25 (PT105B/-), U101.B26 (PT112B/-), U101.B29 (PT121A/+/URC_GPLL1T_IN), U101.B30 (PT121B/-/URC_GPLL1C_IN), U101.C18 (PT71B/-/PCLKC1_0), U101.C19 (PT78A/+), U101.C20 (PT83B/-), U101.C22 (PT89A/+), U101.C23 (PT96A/+), U101.C24 (PT101B/-), U101.C25 (PT107A/+), U101.C26 (PT114A/+), U101.D18 (PT74A/+/GR_PCLK1_0), U101.D19 (PT78B/-), U101.D20 (PT85A/+), U101.D22 (PT89B/-), U101.D23 (PT96B/-), U101.D24 (PT103A/+), U101.D25 (PT107B/-), U101.D26 (PT114B/-), U101.E17 (PT69A/+/PCLKT1_1), U101.E19 (PT80A/+), U101.E22 (PT92A/+), U101.E23 (PT98A/+), U101.E25 (PT110A/+), U101.F17 (PT69B/-/PCLKC1_1), U101.F18 (PT74B/-/GR_PCLK1_1), U101.F19 (PT80B/-), U101.F20 (PT85B/-), U101.F22 (PT92B/-), U101.F23 (PT98B/-), U101.F24 (PT103B/-), U101.F25 (PT110B/-)
- new net PORT3: U101.B32 (PR17A/+/HS/RDQS17), U101.C28 (PR11A/+/URC_GPLL0T_IN/HS/RDQ17), U101.C29 (PR11C/+/RDQ17), U101.C30 (PR11D/-/RDQ17), U101.C31 (PR17B/-/HS/RDQSN17), U101.C32 (PR20C/+/RDQ17), U101.D28 (PR11B/-/URC_GPLL0C_IN/HS/RDQ17), U101.D29 (PR14A/+/HS/RDQ17), U101.D30 (PR17C/+/RDQ17), U101.D31 (PR17D/-/RDQ17), U101.D32 (PR20D/-/RDQ17), U101.E29 (PR14B/-/HS/RDQ17), U101.E30 (PR20B/-/HS/RDQ17), U101.E32 (PR23B/-/HS/RDQ29), U101.F28 (PR14D/-/RDQ17), U101.F29 (PR14C/+/RDQ17), U101.F30 (PR20A/+/HS/RDQ17), U101.F31 (PR23A/+/HS/RDQ29), U101.F32 (PR23C/+/RDQ29), U101.H27 (PR35A/+/HS/RDQ41), U101.H28 (PR35B/-/HS/RDQ41), U101.H30 (PR26B/-/HS/RDQ29), U101.H31 (PR26A/+/HS/RDQ29), U101.H32 (PR23D/-/RDQ29), U101.J26 (PR35C/+/VREF1_2/RDQ41), U101.J27 (PR35D/-/RDQ41), U101.J29 (PR32C/+/RDQ29), U101.J30 (PR26C/+/RDQ29), U101.J32 (PR29B/-/HS/RDQSN29), U101.K26 (PR38B/-/HS/RDQ41), U101.K27 (PR38A/+/HS/RDQ41), U101.K28 (PR38C/+/RDQ41), U101.K29 (PR32D/-/RDQ29), U101.K30 (PR26D/-/RDQ29), U101.K31 (PR29A/+/HS/RDQS29), U101.K32 (PR29C/+/RDQ29), U101.L26 (PR41C/+/GR_PCLK2_0/RDQ41), U101.L27 (PR41D/-/RDQ41), U101.L29 (PR38D/-/RDQ41), U101.L30 (PR32B/-/HS/RDQ29), U101.L31 (PR32A/+/HS/RDQ29), U101.L32 (PR29D/-/RDQ29), U101.N26 (PR44B/-/PCLKC2_1/HS/RDQ41), U101.N27 (PR44A/+/PCLKT2_1/HS/RDQ41), U101.N29 (PR41B/-/HS/RDQSN41), U101.N30 (PR41A/+/GR_PCLK2_1/HS/RDQS41), U101.P26 (PR44D/-/PCLKC2_0/RDQ41), U101.P27 (PR44C/+/PCLKT2_0/RDQ41)
- new net PORT4: U101.AB26 (PR74C/+/RDQ77), U101.AB27 (PR77B/-/HS/RDQSN77), U101.AB28 (PR77A/+/HS/RDQS77), U101.AB29 (PR83B/-/HS/RDQ89), U101.AB30 (PR83A/+/HS/RDQ89), U101.AB31 (PR89B/-/HS/RDQSN89), U101.AB32 (PR92A/+/HS/RDQ89), U101.AC26 (PR77C/+/RDQ77), U101.AC27 (PR74D/-/RDQ77), U101.AC28 (PR83C/+/RDQ89), U101.AC30 (PR89A/+/HS/RDQS89), U101.AC31 (PR89C/+/RDQ89), U101.AC32 (PR92B/-/HS/RDQ89), U101.AD26 (PR77D/-/RDQ77), U101.AD27 (PR80A/+/HS/RDQ77), U101.AD29 (PR83D/-/RDQ89), U101.AD30 (PR86C/+/RDQ89), U101.AD32 (PR92C/+/LRC_GPLL0T_IN/RDQ89), U101.AE27 (PR80B/-/HS/RDQ77), U101.AE28 (PR80C/+/RDQ77), U101.AE29 (PR80D/-/RDQ77), U101.AE30 (PR86D/-/RDQ89), U101.AE31 (PR89D/-/RDQ89), U101.AE32 (PR92D/-/LRC_GPLL0C_IN/RDQ89), U101.N32 (PR62A/+/HS/RDQ65), U101.P28 (PR47A/+/PCLKT3_1/HS/RDQ53), U101.P29 (PR47B/-/PCLKC3_1/HS/RDQ53), U101.P30 (PR59B/-/HS/RDQ65), U101.P31 (PR59A/+/HS/RDQ65), U101.P32 (PR62B/-/HS/RDQ65), U101.R26 (PR47C/+/PCLKT3_0/RDQ53), U101.R27 (PR50A/+/GR_PCLK3_0/HS/RDQ53), U101.R29 (PR53A/+/HS/RDQS53), U101.R30 (PR59C/+/RDQ65), U101.R32 (PR65A/+/HS/RDQS65), U101.T26 (PR47D/-/PCLKC3_0/RDQ53), U101.T27 (PR50B/-/HS/RDQ53), U101.T28 (PR53B/-/HS/RDQSN53), U101.T29 (PR53C/+/RDQ53), U101.T30 (PR59D/-/RDQ65), U101.T31 (PR65B/-/HS/RDQSN65), U101.T32 (PR68A/+/HS/RDQ65), U101.U26 (PR50D/-/RDQ53), U101.U27 (PR50C/+/GR_PCLK3_1/RDQ53), U101.U28 (PR53D/-/RDQ53), U101.U29 (PR56A/+/HS/RDQ53), U101.U30 (PR62D/-/RDQ65), U101.U31 (PR62C/+/RDQ65), U101.U32 (PR68B/-/HS/RDQ65), U101.V26 (PR56D/-/RDQ53), U101.V27 (PR56C/+/RDQ53), U101.V29 (PR56B/-/VREF1_3/HS/RDQ53), U101.V32 (PR68C/+/RDQ65), U101.W28 (PR71D/-/RDQ77), U101.W29 (PR74B/-/HS/RDQ77), U101.W30 (PR65C/+/RDQ65), U101.W31 (PR86A/+/HS/RDQ89), U101.W32 (PR68D/-/RDQ65), U101.Y26 (PR71A/+/HS/RDQ77), U101.Y27 (PR71B/-/HS/RDQ77), U101.Y28 (PR71C/+/RDQ77), U101.Y29 (PR74A/+/HS/RDQ77), U101.Y30 (PR65D/-/RDQ65), U101.Y32 (PR86B/-/HS/RDQ89)
- new net PORT5: U101.AG28 (PB110A/+), U101.AG29 (PB110B/-), U101.AG30 (PB114B/-), U101.AG32 (PB119B/-), U101.AH28 (PB112B/-), U101.AH30 (PB114A/+), U101.AH32 (PB119A/+), U101.AJ28 (PB112A/+), U101.AJ29 (PB121A/+), U101.AJ30 (PB121B/-), U101.AJ31 (PB105B/-), U101.AJ32 (PB101B/-), U101.AK28 (PB98B/-), U101.AK29 (PB116A/+), U101.AK30 (PB116B/-), U101.AK31 (PB105A/+), U101.AK32 (PB101A/+), U101.AL28 (PB98A/+), U101.AL30 (PB103B/-), U101.AL32 (PB107B/-), U101.AM28 (PB96A/+), U101.AM29 (PB96B/-), U101.AM30 (PB103A/+), U101.AM31 (PB107A/+)
- new net PORT6: U101.AB1 (PL92A/+/HS/LDQ89), U101.AB2 (PL89B/-/HS/LDQSN89), U101.AB3 (PL83A/+/HS/LDQ89), U101.AB4 (PL83B/-/HS/LDQ89), U101.AB5 (PL77A/+/HS/LDQS77), U101.AB6 (PL77B/-/HS/LDQSN77), U101.AB7 (PL74C/+/LDQ77), U101.AC1 (PL92B/-/HS/LDQ89), U101.AC2 (PL89C/+/LDQ89), U101.AC3 (PL89A/+/HS/LDQS89), U101.AC5 (PL83C/+/LDQ89), U101.AC6 (PL74D/-/LDQ77), U101.AC7 (PL77C/+/LDQ77), U101.AD1 (PL92C/+/LLC_GPLL0T_IN/LDQ89), U101.AD3 (PL86C/+/LDQ89), U101.AD4 (PL83D/-/LDQ89), U101.AD6 (PL80A/+/HS/LDQ77), U101.AD7 (PL77D/-/LDQ77), U101.AE1 (PL92D/-/LLC_GPLL0C_IN/LDQ89), U101.AE2 (PL89D/-/LDQ89), U101.AE3 (PL86D/-/LDQ89), U101.AE4 (PL80D/-/LDQ77), U101.AE5 (PL80C/+/LDQ77), U101.AE6 (PL80B/-/HS/LDQ77), U101.N1 (PL62A/+/HS/LDQ65), U101.P1 (PL62B/-/HS/LDQ65), U101.P2 (PL59A/+/HS/LDQ65), U101.P3 (PL59B/-/HS/LDQ65), U101.P4 (PL47B/-/PCLKC6_1/HS/LDQ53), U101.P5 (PL47A/+/PCLKT6_1/HS/LDQ53), U101.R1 (PL65A/+/HS/LDQS65), U101.R3 (PL59C/+/LDQ65), U101.R4 (PL53A/+/HS/LDQS53), U101.R6 (PL50A/+/GR_PCLK6_0/HS/LDQ53), U101.R7 (PL47C/+/PCLKT6_0/LDQ53), U101.T1 (PL68A/+/HS/LDQ65), U101.T2 (PL65B/-/HS/LDQSN65), U101.T3 (PL59D/-/LDQ65), U101.T4 (PL53C/+/LDQ53), U101.T5 (PL53B/-/HS/LDQSN53), U101.T6 (PL50B/-/HS/LDQ53), U101.T7 (PL47D/-/PCLKC6_0/LDQ53), U101.U1 (PL68B/-/HS/LDQ65), U101.U2 (PL62C/+/LDQ65), U101.U3 (PL62D/-/LDQ65), U101.U4 (PL56A/+/HS/LDQ53), U101.U5 (PL53D/-/LDQ53), U101.U6 (PL50C/+/GR_PCLK6_1/LDQ53), U101.U7 (PL50D/-/LDQ53), U101.V1 (PL68C/+/LDQ65), U101.V4 (PL56B/-/VREF1_6/HS/LDQ53), U101.V6 (PL56C/+/LDQ53), U101.V7 (PL56D/-/LDQ53), U101.W1 (PL68D/-/LDQ65), U101.W2 (PL86A/+/HS/LDQ89), U101.W3 (PL65C/+/LDQ65), U101.W4 (PL74B/-/HS/LDQ77), U101.W5 (PL71D/-/LDQ77), U101.Y1 (PL86B/-/HS/LDQ89), U101.Y3 (PL65D/-/LDQ65), U101.Y4 (PL74A/+/HS/LDQ77), U101.Y5 (PL71C/+/LDQ77), U101.Y6 (PL71B/-/HS/LDQ77), U101.Y7 (PL71A/+/HS/LDQ77)
- new net PORT7: U101.B1 (PL17A/+/HS/LDQS17), U101.C1 (PL20C/+/LDQ17), U101.C2 (PL17B/-/HS/LDQSN17), U101.C3 (PL11D/-/LDQ17), U101.C4 (PL11C/+/LDQ17), U101.C5 (PL11A/+/ULC_GPLL0T_IN/HS/LDQ17), U101.D1 (PL20D/-/LDQ17), U101.D2 (PL17D/-/LDQ17), U101.D3 (PL17C/+/LDQ17), U101.D4 (PL14A/+/HS/LDQ17), U101.D5 (PL11B/-/ULC_GPLL0C_IN/HS/LDQ17), U101.E1 (PL23B/-/HS/LDQ29), U101.E3 (PL20B/-/HS/LDQ17), U101.E4 (PL14B/-/HS/LDQ17), U101.F1 (PL23C/+/LDQ29), U101.F2 (PL23A/+/HS/LDQ29), U101.F3 (PL20A/+/HS/LDQ17), U101.F4 (PL14C/+/LDQ17), U101.F5 (PL14D/-/LDQ17), U101.H1 (PL23D/-/LDQ29), U101.H2 (PL26A/+/HS/LDQ29), U101.H3 (PL26B/-/HS/LDQ29), U101.H5 (PL35B/-/HS/LDQ41), U101.H6 (PL35A/+/HS/LDQ41), U101.J1 (PL29B/-/HS/LDQSN29), U101.J3 (PL26C/+/LDQ29), U101.J4 (PL32C/+/LDQ29), U101.J6 (PL35D/-/LDQ41), U101.J7 (PL35C/+/VREF1_7/LDQ41), U101.K1 (PL29C/+/LDQ29), U101.K2 (PL29A/+/HS/LDQS29), U101.K3 (PL26D/-/LDQ29), U101.K4 (PL32D/-/LDQ29), U101.K5 (PL38C/+/LDQ41), U101.K6 (PL38A/+/HS/LDQ41), U101.K7 (PL38B/-/HS/LDQ41), U101.L1 (PL29D/-/LDQ29), U101.L2 (PL32A/+/HS/LDQ29), U101.L3 (PL32B/-/HS/LDQ29), U101.L4 (PL38D/-/LDQ41), U101.L6 (PL41D/-/LDQ41), U101.L7 (PL41C/+/GR_PCLK7_0/LDQ41), U101.N3 (PL41A/+/GR_PCLK7_1/HS/LDQS41), U101.N4 (PL41B/-/HS/LDQSN41), U101.N6 (PL44A/+/PCLKT7_1/HS/LDQ41), U101.N7 (PL44B/-/PCLKC7_1/HS/LDQ41), U101.P6 (PL44C/+/PCLKT7_0/LDQ41), U101.P7 (PL44D/-/PCLKC7_0/LDQ41)
Other:
- added sheet Input Port (input_port.kicad_sch)
- added sheet Power (power.kicad_sch)

Commit message: Save
Parts:
- added C101, C102, C103, C104, C105, C108, C109, C110, C111, C113, C114, C115, C116, C117, C118, C119, C120, C121: 0.1u, passive:C_0201, symbol Device:C_Small
- added C106, C107: 10p, passive:C_0402, symbol Device:C_Small
- added C112: 4.7u, passive:C_0603, symbol Device:C_Small
- added FB101: FerriteBead_Small, passive:R_0603, symbol Device:FerriteBead_Small
- added J101: USB3_B_Micro, usb:AMPHENOL-GSB343K33HR, symbol connectors:USB3_B_Micro
- added R101: 1.6k, passive:R_0201, symbol Device:R_Small
- added R102, R103, R104: 10k, passive:R_0201, symbol Device:R_Small
- added R105, R106, R107, R108, R109, R110, R111, R112, R113, R114, R115, R116, R117, R118, R119, R120, R121, R122, R123, R124, R125, R126, R127, R128: 33, passive:R_0201, symbol Device:R_Small
- added U105: PUSB3FR4Z, dfn:DFN-10-1.0x2.5mm_P0.5mm, symbol Connector_Generic:Conn_02x05_Counter_Clockwise
- added U106: FT600Q, qfn:QFN-56-1EP_7x7mm_P0.4mm_EP5.7x5.7mm_FT600, symbol ftdi:FT600Q
- added Y101: 30 MHz, crystals:Crystal_4Pin_2.0x1.6mm, symbol Device:Crystal_GND24_Small
Connections:
- net PORT2 is gone; now on net PORT3: U101.A18 (PT71A/+/PCLKT1_0), U101.A19 (PT76A/+), U101.A20 (PT83A/+), U101.A22 (PT87A/+), U101.A23 (PT94A/+), U101.A24 (PT101A/+), U101.A25 (PT105A/+), U101.A26 (PT112A/+), U101.A28 (PT116A/+), U101.A29 (PT116B/-), U101.A30 (PT119A/+), U101.A31 (PT119B/-), U101.B19 (PT76B/-), U101.B22 (PT87B/-), U101.B23 (PT94B/-), U101.B25 (PT105B/-), U101.B26 (PT112B/-), U101.B29 (PT121A/+/URC_GPLL1T_IN), U101.B30 (PT121B/-/URC_GPLL1C_IN), U101.C18 (PT71B/-/PCLKC1_0), U101.C19 (PT78A/+), U101.C20 (PT83B/-), U101.C22 (PT89A/+), U101.C23 (PT96A/+), U101.C24 (PT101B/-), U101.C25 (PT107A/+), U101.C26 (PT114A/+), U101.D18 (PT74A/+/GR_PCLK1_0), U101.D19 (PT78B/-), U101.D20 (PT85A/+), U101.D22 (PT89B/-), U101.D23 (PT96B/-), U101.D24 (PT103A/+), U101.D25 (PT107B/-), U101.D26 (PT114B/-), U101.E17 (PT69A/+/PCLKT1_1), U101.E19 (PT80A/+), U101.E22 (PT92A/+), U101.E23 (PT98A/+), U101.E25 (PT110A/+), U101.F17 (PT69B/-/PCLKC1_1), U101.F18 (PT74B/-/GR_PCLK1_1), U101.F19 (PT80B/-), U101.F20 (PT85B/-), U101.F22 (PT92B/-), U101.F23 (PT98B/-), U101.F24 (PT103B/-), U101.F25 (PT110B/-)
- net PORT3: no longer U101.B32 (PR17A/+/HS/RDQS17), U101.C28 (PR11A/+/URC_GPLL0T_IN/HS/RDQ17), U101.C29 (PR11C/+/RDQ17), U101.C30 (PR11D/-/RDQ17), U101.C31 (PR17B/-/HS/RDQSN17), U101.C32 (PR20C/+/RDQ17), U101.D28 (PR11B/-/URC_GPLL0C_IN/HS/RDQ17), U101.D29 (PR14A/+/HS/RDQ17), U101.D30 (PR17C/+/RDQ17), U101.D31 (PR17D/-/RDQ17), U101.D32 (PR20D/-/RDQ17), U101.E29 (PR14B/-/HS/RDQ17), U101.E30 (PR20B/-/HS/RDQ17), U101.E32 (PR23B/-/HS/RDQ29), U101.F28 (PR14D/-/RDQ17), U101.F29 (PR14C/+/RDQ17), U101.F30 (PR20A/+/HS/RDQ17), U101.F31 (PR23A/+/HS/RDQ29), U101.F32 (PR23C/+/RDQ29), U101.H27 (PR35A/+/HS/RDQ41), U101.H28 (PR35B/-/HS/RDQ41), U101.H30 (PR26B/-/HS/RDQ29), U101.H31 (PR26A/+/HS/RDQ29), U101.H32 (PR23D/-/RDQ29), U101.J26 (PR35C/+/VREF1_2/RDQ41), U101.J27 (PR35D/-/RDQ41), U101.J29 (PR32C/+/RDQ29), U101.J30 (PR26C/+/RDQ29), U101.J32 (PR29B/-/HS/RDQSN29), U101.K26 (PR38B/-/HS/RDQ41), U101.K27 (PR38A/+/HS/RDQ41), U101.K28 (PR38C/+/RDQ41), U101.K29 (PR32D/-/RDQ29), U101.K30 (PR26D/-/RDQ29), U101.K31 (PR29A/+/HS/RDQS29), U101.K32 (PR29C/+/RDQ29), U101.L26 (PR41C/+/GR_PCLK2_0/RDQ41), U101.L27 (PR41D/-/RDQ41), U101.L29 (PR38D/-/RDQ41), U101.L30 (PR32B/-/HS/RDQ29), U101.L31 (PR32A/+/HS/RDQ29), U101.L32 (PR29D/-/RDQ29), U101.N26 (PR44B/-/PCLKC2_1/HS/RDQ41), U101.N27 (PR44A/+/PCLKT2_1/HS/RDQ41), U101.N29 (PR41B/-/HS/RDQSN41), U101.N30 (PR41A/+/GR_PCLK2_1/HS/RDQS41), U101.P26 (PR44D/-/PCLKC2_0/RDQ41), U101.P27 (PR44C/+/PCLKT2_0/RDQ41)
- new net: C106.1, U106.16 (XI), Y101.1
- new net: C107.1, U106.17 (XO), Y101.3
- new net +3V3: C102.1, C103.1, C104.1, C110.1, C113.1, C114.1, C115.1, R102.1, R103.1, R104.1, U101.D28 (PR11B/-/URC_GPLL0C_IN/HS/RDQ17), U101.F31 (PR23A/+/HS/RDQ29), U101.J29 (PR32C/+/RDQ29), U101.N26 (PR44B/-/PCLKC2_1/HS/RDQ41), U101.N30 (PR41A/+/GR_PCLK2_1/HS/RDQS41), U106.15 (VCC33[3]), U106.19 (VCC33), U106.22 (VDDA), U106.30 (VCC33), U106.38 (VCCIO[3]), U106.44 (VCCIO), U106.52 (VCCIO)
- new net +5V: C120.1, FB101.2, U106.29 (VBUS)
- new net D_N: J101.2 (D-), U106.20 (DM)
- new net D_P: J101.3 (D+), U106.18 (DP)
- new net FT_BE0: R105.2, U101.E32 (PR23B/-/HS/RDQ29)
- new net FT_BE1: R106.2, U101.F32 (PR23C/+/RDQ29)
- new net FT_CLKOUT: R112.2, U101.C28 (PR11A/+/URC_GPLL0T_IN/HS/RDQ17)
- new net FT_D0: R113.2, U101.K32 (PR29C/+/RDQ29)
- new net FT_D1: R114.2, U101.L32 (PR29D/-/RDQ29)
- new net FT_D10: R123.2, U101.K28 (PR38C/+/RDQ41)
- new net FT_D11: R124.2, U101.L29 (PR38D/-/RDQ41)
- new net FT_D12: R125.2, U101.N29 (PR41B/-/HS/RDQSN41)
- new net FT_D13: R126.2, U101.L26 (PR41C/+/GR_PCLK2_0/RDQ41)
- new net FT_D14: R127.2, U101.L27 (PR41D/-/RDQ41)
- new net FT_D15: R128.2, U101.N27 (PR44A/+/PCLKT2_1/HS/RDQ41)
- new net FT_D2: R115.2, U101.L31 (PR32A/+/HS/RDQ29)
- new net FT_D3: R116.2, U101.L30 (PR32B/-/HS/RDQ29)
- new net FT_D4: R117.2, U101.H27 (PR35A/+/HS/RDQ41)
- new net FT_D5: R118.2, U101.K29 (PR32D/-/RDQ29)
- new net FT_D6: R119.2, U101.J26 (PR35C/+/VREF1_2/RDQ41)
- new net FT_D7: R120.2, U101.H28 (PR35B/-/HS/RDQ41)
- new net FT_D8: R121.2, U101.K27 (PR38A/+/HS/RDQ41)
- new net FT_D9: R122.2, U101.K26 (PR38B/-/HS/RDQ41)
- new net FT_GPIO0: U101.D31 (PR17D/-/RDQ17), U106.12 (GPIO0)
- new net FT_GPIO1: U101.F30 (PR20A/+/HS/RDQ17), U106.13 (GPIO1)
- new net FT_P_BE0: R105.1, U106.2 (BE_0)
- new net FT_P_BE1: R106.1, U106.3 (BE_1)
- new net FT_P_CLKOUT: R112.1, U106.43 (CLK)
- new net FT_P_D0: R113.1, U106.33 (DATA_0)
- new net FT_P_D1: R114.1, U106.34 (DATA_1)
- new net FT_P_D10: R123.1, U106.47 (DATA_10)
- new net FT_P_D11: R124.1, U106.48 (DATA_11)
- new net FT_P_D12: R125.1, U106.53 (DATA_12)
- new net FT_P_D13: R126.1, U106.54 (DATA_13)
- new net FT_P_D14: R127.1, U106.55 (DATA_14)
- new net FT_P_D15: R128.1, U106.56 (DATA_15)
- new net FT_P_D2: R115.1, U106.35 (DATA_2)
- new net FT_P_D3: R116.1, U106.36 (DATA_3)
- new net FT_P_D4: R117.1, U106.39 (DATA_4)
- new net FT_P_D5: R118.1, U106.40 (DATA_5)
- new net FT_P_D6: R119.1, U106.41 (DATA_6)
- new net FT_P_D7: R120.1, U106.42 (DATA_7)
- new net FT_P_D8: R121.1, U106.45 (DATA_8)
- new net FT_P_D9: R122.1, U106.46 (DATA_9)
- new net FT_REF: R101.1, U106.21 (RREF)
- new net FT_WAKEUP: R102.2, U101.D32 (PR20D/-/RDQ17), U106.11 (WAKEUP_N)
- new net GND: C101.2, C102.2, C103.2, C104.2, C105.2, C106.2, C107.2, C110.2, C111.2, C112.2, C113.2, C114.2, C115.2, C116.2, C117.2, C118.2, C119.2, C120.2, C121.2, J101.11 (Shield), J101.5 (GND), J101.8 (GND_DRAIN), R101.2, U105.3 (Pin_3), U105.8 (Pin_8), U106.32 (GND[4]), U106.49 (GND), U106.51 (GND), U106.57 (GND), Y101.2, Y101.4
- new net RX_N: J101.9 (SSRX-), U105.4 (Pin_4), U105.7 (Pin_7), U106.27 (RIDN)
- new net RX_P: J101.10 (SSRX+), U105.5 (Pin_5), U105.6 (Pin_6), U106.28 (RIDP)
- new net TX_N: C108.1, J101.6 (SSTX-), U105.1 (Pin_1), U105.10 (Pin_10)
- new net TX_P: C109.1, J101.7 (SSTX+), U105.2 (Pin_2), U105.9 (Pin_9)
- new net TX_P_N: C108.2, U106.24 (TODN)
- new net TX_P_P: C109.2, U106.25 (TODP)
- new net VBUS_IN: C101.1, FB101.1, J101.1 (VBUS)
- new net VD10: C105.1, C111.1, C112.1, C116.1, C117.1, C118.1, C119.1, U106.1 (AVDD), U106.23 (VD10[4]), U106.26 (VD10), U106.31 (DV10), U106.37 (VD10), U106.50 (VD10)
- new net ~{FT_OE}: R111.2, U101.K31 (PR29A/+/HS/RDQS29)
- new net ~{FT_P_OE}: R111.1, U106.9 (OE_N)
- new net ~{FT_P_RD}: R110.1, U106.8 (RD_N)
- new net ~{FT_P_RXF}: R108.1, U106.5 (RXF_N)
- new net ~{FT_P_TXE}: R107.1, U106.4 (TXE_N)
- new net ~{FT_P_WR}: R109.1, U106.7 (WR_N)
- new net ~{FT_RD}: R110.2, U101.K30 (PR26D/-/RDQ29)
- new net ~{FT_RESET}: C121.1, R103.2, U101.C32 (PR20C/+/RDQ17), U106.10 (RESET_N)
- new net ~{FT_RXF}: R108.2, U101.H30 (PR26B/-/HS/RDQ29)
- new net ~{FT_SIWU}: R104.2, U101.E30 (PR20B/-/HS/RDQ17), U106.6 (SIWU_N)
- new net ~{FT_TXE}: R107.2, U101.H32 (PR23D/-/RDQ29)
- new net ~{FT_WR}: R109.2, U101.J30 (PR26C/+/RDQ29)
- no-connect marks 0 -> 1
Other:
- note added: "DESIGN NOTE: Pseudo power pins."
- note added: "DESIGN NOTE: The data clock needs to go to a clock capable pin on the FPGA."
- note added: "DESIGN NOTE: This should provide about 200 MB/s of bandwidth with a computer."
- note added: "ESD Protection"
- note added: "TOTAL: 352 IO"
- moved on the sheet: U101C, U101D

Commit message: Moved to PCIe connectors, added USB 3.0 Type B connector
Parts:
- removed J101: USB3_B_Micro, usb:AMPHENOL-GSB343K33HR, symbol connectors:USB3_B_Micro
- added J102: GSB422137EU, connectors:AMPHENOL_GSB422137EU, symbol connectors:GSB422137EU
- renumbered C113 to C102, C114 to C103, C118 to C104, C115 to C105, C120 to C106, C119 to C107, C116 to C108, C102 to C109, C121 to C110, C117 to C111, C103 to C112, C104 to C113, C105 to C114, C106 to C115, C107 to C116, C108 to C117, C109 to C118, C110 to C119, C111 to C120, C112 to C121, U105 to U102, U106 to U103, U103 to U104, U104 to U105, U102 to U106
Connections:
- net D_N: now also J102.2 (D-)
- net D_P: now also J102.3 (D+)
- net GND: now also J102.4 (GND), J102.7 (GND_DRAIN), J102.SH1 (SHIELD), J102.SH2 (SHIELD__1), J102.SH3 (SHIELD__2)
- net RX_N: now also J102.8 (STDB_SSRX-)
- net RX_P: now also J102.9 (STDB_SSRX+)
- net TX_N: now also J102.5 (STDB_SSTX-)
- net TX_P: now also J102.6 (STDB_SSTX+)
- net VBUS_IN: now also J102.1 (VBUS)
- no-connect marks 1 -> 0
Other:
- sheet Input Port renamed Input Port 1
- added sheet Input Port 2 (input_port.kicad_sch)
- added sheet Input Port 3 (input_port.kicad_sch)
- added sheet Input Port 4 (input_port.kicad_sch)
- moved on the sheet: C101, FB101

Commit message: Save
Parts:
- removed U105: TCA9535RTWR, Package_DFN_QFN:WQFN-24-1EP_4x4mm_P0.5mm_EP2.45x2.45mm, symbol Interface_Expansion:TCA9535RTWR
- removed U106: TXB0108DQSR, Package_SON:USON-20_2x4mm_P0.4mm, symbol Logic_LevelTranslator:TXB0108DQSR
- added C122: 0.1u, passive:C_0201, symbol Device:C_Small
- added D101: LED_Small, LED_SMD:LED_0402_1005Metric, symbol Device:LED_Small
- added H101, H102, H103, H104, H105, H106, H107: MountingHole_Pad, MountingHole:MountingHole_3.2mm_M3_Pad_Via, symbol Mechanical:MountingHole_Pad
- added J101: TC2050, Connector:Tag-Connect_TC2050-IDC-NL_2x05_P1.27mm_Vertical, symbol Connector_Generic:Conn_01x10
- added R129, R130, R131, R132, R134: 1k, passive:R_0201, symbol Device:R_Small
- added R133, R136: 10k, passive:R_0201, symbol Device:R_Small
- added R135: 0, passive:R_0201, symbol Device:R_Small
- added U105: W25Q128JVP, Package_SON:WSON-8-1EP_6x5mm_P1.27mm_EP3.4x4.3mm, symbol Memory_Flash:W25Q32JVZP
- added U108: USBLC6-2P6, Package_TO_SOT_SMD:SOT-666, symbol Power_Protection:USBLC6-2P6
Connections:
- net +3V3: now also C122.1, J101.1 (Pin_1), R129.1, R130.1, R131.1, R132.1, R133.1, R136.1, U105.8 (VCC)
- net +5V: now also R135.2
- net D_N: now also U108.1 (I/O1); no longer J102.2 (D-)
- net D_P: now also U108.3 (I/O2); no longer J102.3 (D+)
- net GND: now also U101.AK4 (CFG_2), U101.AM4 (CFG_0), C122.2, H101.1, H102.1, H103.1, H104.1, H105.1, H106.1, H107.1, J101.3 (Pin_3), R134.2, U105.4 (GND), U105.9 (EP), U108.2 (GND)
- net VBUS_IN: now also U108.5 (VBUS)
- net TDO: now reaches U101.AG5 (TDO)
- net TDO: now also J101.6 (Pin_6)
- net TDI: now reaches U101.AJ5 (TDI)
- net TDI: now also J101.8 (Pin_8)
- net TCK: now reaches U101.AK5 (TCK)
- net TCK: now also J101.4 (Pin_4), R134.1
- net TMS: now reaches U101.AM5 (TMS)
- net TMS: now also J101.2 (Pin_2)
- net INITN: now reaches U101.AG4 (INITN)
- net INITN: now also R133.2
- net PROGRAMN: now reaches U101.AH4 (PROGRAMN)
- net PROGRAMN: now also R132.2
- net SPI_MISO: now reaches U101.AJ2 (PB11A/+/D1/MISO/IO1)
- net SPI_MISO: now also U105.2 (DO(IO1))
- net SPI_CS: now reaches U101.AJ3 (PB15A/+/HOLDN/DI/BUSY/CSSPIN/CEN)
- net SPI_CS: now also R136.2, U105.1 (~{CS})
- net DONE: now reaches U101.AJ4 (DONE)
- net DONE: now also D101.1 (K)
- net SPI_MOSI: now reaches U101.AK2 (PB11B/-/D0/MOSI/IO0)
- net SPI_MOSI: now also U105.5 (DI(IO0))
- net SPI_D3: now reaches U101.AL1 (PB9A/+/D3/IO3)
- net SPI_D3: now also U105.7 (IO3)
- net CFG_1: now reaches U101.AL4 (CFG_1)
- net CFG_1: now also R130.2
- net SPI_D2: now reaches U101.AM2 (PB9B/-/D2/IO2)
- net SPI_D2: now also U105.3 (IO2)
- net SPI_CLK: now reaches U101.AM3 (CCLK/MCLK/SCK)
- net SPI_CLK: now also R129.2, U105.6 (CLK)
- new net: D101.2 (A), R131.2
- new net: J101.5 (Pin_5), R135.1
- new net D_C_N: J102.2 (D-), U108.6 (I/O1)
- new net D_C_P: J102.3 (D+), U108.4 (I/O2)
- no-connect marks 0 -> 11
Other:
- sheet Input Port 1 ports: added IO_[0..63], PORT_ENABLE, SCL, SDA; removed none
- sheet Input Port 2 ports: added IO_[0..63], PORT_ENABLE, SCL, SDA; removed none
- sheet Input Port 3 ports: added IO_[0..63], PORT_ENABLE, SCL, SDA; removed none
- sheet Input Port 4 ports: added IO_[0..63], PORT_ENABLE, SCL, SDA; removed none
- note added: "DESIGN NOTE: Master SPI config."
- note added: "DESIGN NOTE: The bitstream will only take max 32 MBits, leaving 75% of the flash for user data."
- note added: "TOTAL: 304 IO"
- note removed: "TOTAL: 352 IO"
- moved on the sheet: C101, FB101, J102, U101I, U101J, U102

Commit message: Moved to new level translator with less input current requirement
Parts:
- C101, C102, C103, C104, C105, C106, C107, C108, C109, C110, C111, C112, C113, C114, C117, C118, C119, C120, C122: footprint passive:C_0201 -> passive:C_0402
- R101, R102, R103, R104, R105, R106, R107, R108, R109, R110, R111, R112, R113, R114, R115, R116, R117, R118, R119, R120, R121, R122, R123, R124, R125, R126, R127, R128, R129, R130, R131, R132, R133, R134, R135, R136: footprint passive:R_0201 -> passive:R_0402
