File: hardware/input_port.kicad_sch (KiCad schematic)
At the start: 5 parts, among them J101 SS-74500-022

Commit message: Save
Parts:
- added U301, U302, U303, U304, U305, U306, U307, U308: NUF8401MNT4G, dfn:DFN-16-1EP_1.6x4mm_P0.5mm, symbol interface_esd:NUF8401MNT4G
Connections:
- net GND: now also J101.2_1, J101.2_10, J101.2_11, J101.2_12, J101.2_13, J101.2_14, J101.2_15, J101.2_16, J101.2_2, J101.2_3, J101.2_4, J101.2_5, J101.2_6, J101.2_7, J101.2_8, J101.2_9, J101.4_1, J101.4_10, J101.4_11, J101.4_12, J101.4_13, J101.4_14, J101.4_15, J101.4_16, J101.4_2, J101.4_3, J101.4_4, J101.4_5, J101.4_6, J101.4_7, J101.4_8, J101.4_9, J101.6_1, J101.6_10, J101.6_11, J101.6_12, J101.6_13, J101.6_14, J101.6_15, J101.6_16, J101.6_2, J101.6_3, J101.6_4, J101.6_5, J101.6_6, J101.6_7, J101.6_8, J101.6_9, J101.8_1, J101.8_10, J101.8_11, J101.8_12, J101.8_13, J101.8_14, J101.8_15, J101.8_16, J101.8_2, J101.8_3, J101.8_4, J101.8_5, J101.8_6, J101.8_7, J101.8_8, J101.8_9, U301.17 (GND), U302.17 (GND), U303.17 (GND), U304.17 (GND), U305.17 (GND), U306.17 (GND), U307.17 (GND), U308.17 (GND)
- net LED_Y15S: now reaches RN304.1 (R1.1)
- net LED_Y15S: now also J101.11_16
- net LED_Y14S: now reaches RN304.2 (R2.1)
- net LED_Y14S: now also J101.11_15
- net LED_Y13S: now reaches RN304.3 (R3.1)
- net LED_Y13S: now also J101.11_14
- net LED_Y12S: now reaches RN304.4 (R4.1)
- net LED_Y12S: now also J101.11_13
- net LED_Y11S: now reaches RN304.5 (R5.1)
- net LED_Y11S: now also J101.11_12
- net LED_Y10S: now reaches RN304.6 (R6.1)
- net LED_Y10S: now also J101.11_11
- net LED_Y9S: now reaches RN304.7 (R7.1)
- net LED_Y9S: now also J101.11_10
- net LED_Y8S: now reaches RN304.8 (R8.1)
- net LED_Y8S: now also J101.11_9
- net LED_Y2S: now reaches J101.11_3
- net LED_Y2S: now also RN303.6 (R6.1)
- net at J101.1_3: now also U302.1 (1A)
- net at J101.3_3: now also U302.2 (2A)
- net at J101.5_3: now also U302.3 (3A)
- net at J101.7_3: now also U302.4 (4A)
- net LED_G2S: now reaches J101.9_3
- net LED_G2S: now also RN301.6 (R6.1)
- net LED_Y4S: now reaches J101.11_5
- net LED_Y4S: now also RN303.4 (R4.1)
- net at J101.1_5: now also U304.1 (1A)
- net at J101.3_5: now also U304.2 (2A)
- net at J101.5_5: now also U304.3 (3A)
- net at J101.7_5: now also U304.4 (4A)
- net LED_G4S: now reaches J101.9_5
- net LED_G4S: now also RN301.4 (R4.1)
- net LED_Y7S: now reaches J101.11_8
- net LED_Y7S: now also RN303.1 (R1.1)
- net at J101.1_8: now also U303.5 (5A)
- net at J101.3_8: now also U303.6 (6A)
- net at J101.5_8: now also U303.7 (7A)
- net at J101.7_8: now also U303.8 (8A)
- net LED_G7S: now reaches J101.9_8
- net LED_G7S: now also RN301.1 (R1.1)
- net at J101.1_15: now also U308.1 (1A)
- net at J101.3_15: now also U308.2 (2A)
- net at J101.5_15: now also U308.3 (3A)
- net at J101.7_15: now also U308.4 (4A)
- net LED_G14S: now reaches J101.9_15
- net LED_G14S: now also RN302.2 (R2.1)
- net at J101.1_10: now also U305.5 (5A)
- net at J101.3_10: now also U305.6 (6A)
- net at J101.5_10: now also U305.7 (7A)
- net at J101.7_10: now also U305.8 (8A)
- net LED_G9S: now reaches J101.9_10
- net LED_G9S: now also RN302.7 (R7.1)
- net at J101.1_11: now also U306.1 (1A)
- net at J101.3_11: now also U306.2 (2A)
- net at J101.5_11: now also U306.3 (3A)
- net at J101.7_11: now also U306.4 (4A)
- net LED_G10S: now reaches J101.9_11
- net LED_G10S: now also RN302.6 (R6.1)
- net LED_G6S: now reaches RN301.2 (R2.1)
- net LED_G6S: now also J101.9_7
- net LED_G5S: now reaches RN301.3 (R3.1)
- net LED_G5S: now also J101.9_6
- net LED_G3S: now reaches RN301.5 (R5.1)
- net LED_G3S: now also J101.9_4
- net LED_G1S: now reaches RN301.7 (R7.1)
- net LED_G1S: now also J101.9_2
- net LED_G0S: now reaches RN301.8 (R8.1)
- net LED_G0S: now also J101.9_1
- net LED_Y5S: now reaches J101.11_6
- net LED_Y5S: now also RN303.3 (R3.1)
- net at J101.1_6: now also U304.5 (5A)
- net at J101.3_6: now also U304.6 (6A)
- net at J101.5_6: now also U304.7 (7A)
- net at J101.7_6: now also U304.8 (8A)
- net at J101.1_14: now also U307.5 (5A)
- net at J101.3_14: now also U307.6 (6A)
- net at J101.5_14: now also U307.7 (7A)
- net at J101.7_14: now also U307.8 (8A)
- net LED_G13S: now reaches J101.9_14
- net LED_G13S: now also RN302.3 (R3.1)
- net LED_Y1S: now reaches J101.11_2
- net LED_Y1S: now also RN303.7 (R7.1)
- net at J101.1_2: now also U301.5 (5A)
- net at J101.3_2: now also U301.6 (6A)
- net at J101.5_2: now also U301.7 (7A)
- net at J101.7_2: now also U301.8 (8A)
- net at J101.1_12: now also U306.5 (5A)
- net at J101.3_12: now also U306.6 (6A)
- net at J101.5_12: now also U306.7 (7A)
- net at J101.7_12: now also U306.8 (8A)
- net LED_G11S: now reaches J101.9_12
- net LED_G11S: now also RN302.5 (R5.1)
- net at J101.1_13: now also U307.1 (1A)
- net at J101.3_13: now also U307.2 (2A)
- net at J101.5_13: now also U307.3 (3A)
- net at J101.7_13: now also U307.4 (4A)
- net LED_G12S: now reaches J101.9_13
- net LED_G12S: now also RN302.4 (R4.1)
- net LED_Y6S: now reaches RN303.2 (R2.1)
- net LED_Y6S: now also J101.11_7
- net LED_Y3S: now reaches RN303.5 (R5.1)
- net LED_Y3S: now also J101.11_4
- net LED_Y0S: now reaches RN303.8 (R8.1)
- net LED_Y0S: now also J101.11_1
- net LED_G15S: now reaches RN302.1 (R1.1)
- net LED_G15S: now also J101.9_16
- net LED_G8S: now reaches RN302.8 (R8.1)
- net LED_G8S: now also J101.9_9
- net at J101.1_7: now also U303.1 (1A)
- net at J101.3_7: now also U303.2 (2A)
- net at J101.5_7: now also U303.3 (3A)
- net at J101.7_7: now also U303.4 (4A)
- net at J101.1_1: now also U301.1 (1A)
- net at J101.3_1: now also U301.2 (2A)
- net at J101.5_1: now also U301.3 (3A)
- net at J101.7_1: now also U301.4 (4A)
- net at J101.1_9: now also U305.1 (1A)
- net at J101.3_9: now also U305.2 (2A)
- net at J101.5_9: now also U305.3 (3A)
- net at J101.7_9: now also U305.4 (4A)
- net at J101.1_16: now also U308.5 (5A)
- net at J101.3_16: now also U308.6 (6A)
- net at J101.5_16: now also U308.7 (7A)
- net at J101.7_16: now also U308.8 (8A)
- net at J101.1_4: now also U302.5 (5A)
- net at J101.3_4: now also U302.6 (6A)
- net at J101.5_4: now also U302.7 (7A)
- net at J101.7_4: now also U302.8 (8A)
- net LED_G_1 renamed LED_Y0
- net LED_G_10 renamed LED_Y9
- net LED_G_11 renamed LED_Y10
- net LED_G_12 renamed LED_Y11
- net LED_G_13 renamed LED_Y12
- net LED_G_14 renamed LED_Y13
- net LED_G_15 renamed LED_Y14
- net LED_G_16 renamed LED_Y15
- net LED_G_2 renamed LED_Y1
- net LED_G_3 renamed LED_Y2
- net LED_G_4 renamed LED_Y3
- net LED_G_5 renamed LED_Y4
- net LED_G_6 renamed LED_Y5
- net LED_G_7 renamed LED_Y6
- net LED_G_8 renamed LED_Y7
- net LED_G_9 renamed LED_Y8
- net LED_Y_1 renamed LED_G0
- net LED_Y_10 renamed LED_G9
- net LED_Y_11 renamed LED_G10
- net LED_Y_12 renamed LED_G11
- net LED_Y_13 renamed LED_G12
- net LED_Y_14 renamed LED_G13
- net LED_Y_15 renamed LED_G14
- net LED_Y_16 renamed LED_G15
- net LED_Y_2 renamed LED_G1
- net LED_Y_3 renamed LED_G2
- net LED_Y_4 renamed LED_G3
- net LED_Y_5 renamed LED_G4
- net LED_Y_6 renamed LED_G5
- net LED_Y_7 renamed LED_G6
- net LED_Y_8 renamed LED_G7
- net LED_Y_9 renamed LED_G8
- new net IN10_0: U305.12 (5B)
- new net IN10_1: U305.11 (6B)
- new net IN10_2: U305.10 (7B)
- new net IN10_3: U305.9 (8B)
- new net IN11_0: U306.16 (1B)
- new net IN11_1: U306.15 (2B)
- new net IN11_2: U306.14 (3B)
- new net IN11_3: U306.13 (4B)
- new net IN12_0: U306.12 (5B)
- new net IN12_1: U306.11 (6B)
- new net IN12_2: U306.10 (7B)
- new net IN12_3: U306.9 (8B)
- new net IN13_0: U307.16 (1B)
- new net IN13_1: U307.15 (2B)
- new net IN13_2: U307.14 (3B)
- new net IN13_3: U307.13 (4B)
- new net IN14_0: U307.12 (5B)
- new net IN14_1: U307.11 (6B)
- new net IN14_2: U307.10 (7B)
- new net IN14_3: U307.9 (8B)
- new net IN15_0: U308.16 (1B)
- new net IN15_1: U308.15 (2B)
- new net IN15_2: U308.14 (3B)
- new net IN15_3: U308.13 (4B)
- new net IN16_0: U308.12 (5B)
- new net IN16_1: U308.11 (6B)
- new net IN16_2: U308.10 (7B)
- new net IN16_3: U308.9 (8B)
- new net IN1_0: U301.16 (1B)
- new net IN1_1: U301.15 (2B)
- new net IN1_2: U301.14 (3B)
- new net IN1_3: U301.13 (4B)
- new net IN2_0: U301.12 (5B)
- new net IN2_1: U301.11 (6B)
- new net IN2_2: U301.10 (7B)
- new net IN2_3: U301.9 (8B)
- new net IN3_0: U302.16 (1B)
- new net IN3_1: U302.15 (2B)
- new net IN3_2: U302.14 (3B)
- new net IN3_3: U302.13 (4B)
- new net IN4_0: U302.12 (5B)
- new net IN4_1: U302.11 (6B)
- new net IN4_2: U302.10 (7B)
- new net IN4_3: U302.9 (8B)
- new net IN5_0: U304.16 (1B)
- new net IN5_1: U304.15 (2B)
- new net IN5_2: U304.14 (3B)
- new net IN5_3: U304.13 (4B)
- new net IN6_0: U304.12 (5B)
- new net IN6_1: U304.11 (6B)
- new net IN6_2: U304.10 (7B)
- new net IN6_3: U304.9 (8B)
- new net IN7_0: U303.16 (1B)
- new net IN7_1: U303.15 (2B)
- new net IN7_2: U303.14 (3B)
- new net IN7_3: U303.13 (4B)
- new net IN8_0: U303.12 (5B)
- new net IN8_1: U303.11 (6B)
- new net IN8_2: U303.10 (7B)
- new net IN8_3: U303.9 (8B)
- new net IN9_0: U305.16 (1B)
- new net IN9_1: U305.15 (2B)
- new net IN9_2: U305.14 (3B)
- new net IN9_3: U305.13 (4B)
Other:
- moved on the sheet: J101A, J101B, J101C, J101D, J101E, J101F, J101G, J101H, J101I, J101J, J101K, J101L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
